File: pcb/pcb.sch (KiCad schematic (older format))
At the start: 33 parts

Commit message: Add files via upload
Parts:
- added BZ?: Buzzer, symbol Device:Buzzer
- added R? (x7): R, symbol Device:R
- added U?: openMV_M7_R2, symbol openmv_m7_r2:openMV_M7_R2
- added set_goal_color: SW_DIP_x01, symbol Switch:SW_DIP_x01
- added settings: SW_DIP_x06, symbol Switch:SW_DIP_x06
- renumbered i2converter to i2converter1
Connections:
- wire segments 426 -> 539

Commit message: Add files via upload
Parts:
- added BT1: Battery, Connector_AMASS:AMASS_XT60-F_1x02_P7.20mm_Vertical, symbol Device:Battery
- added BT2: Battery, Connector_AMASS:AMASS_XT30U-F_1x02_P5.0mm_Vertical, symbol Device:Battery
- BZ1: renamed from BZ?; footprint (none) -> custom:buzer
- R1, R2, R3, R4, R5, R6, R7: renamed from R?; footprint (none) -> custom:resistor
- collor_sensor_1, collor_sensor_2, collor_sensor_3, collor_sensor_4, collor_sensor_5, collor_sensor_6: footprint (none) -> custom:tcs3472
- controllboard1: footprint (none) -> custom:teensy4.1; symbol teensy:Teensy4.1 -> pcb-rescue:Teensy4.1-teensy
- ir_sensor_1, ir_sensor_10, ir_sensor_11, ir_sensor_12, ir_sensor_13, ir_sensor_14, ir_sensor_15, ir_sensor_16, ir_sensor_2, ir_sensor_3, ir_sensor_4, ir_sensor_5, ir_sensor_6, ir_sensor_7, ir_sensor_8, ir_sensor_9: footprint (none) -> custom:tssp4038
- motor1, motor2, motor3: footprint (none) -> custom:pololu_motor
- motor_driver1, motor_driver2: footprint (none) -> custom:l298n
- openmvcam1: renamed from U?; footprint (none) -> custom:openmv_m7_r2
- set_goal_color1: renamed from set_goal_color; footprint (none) -> custom:dipswitch1
- settings1: renamed from settings; footprint (none) -> custom:dipswitch6
Connections:
- wire segments 539 -> 544

Commit message: Add files via upload
Parts:
- added U?: miniIMU-9_v6, symbol miniimu-9_v6:miniIMU-9_v6
Connections:
- wire segments 544 -> 560
Changed lines of the file:
@@
 tijdelijke plaatsing tot goede gevonden
-Wire Wire Line
-	3450 5600 3575 5600
 Wire Wire Line
 	3450 5400 3700 5400
@@
 $EndComp
 Wire Wire Line
-	3500 2100 4600 2100
-Wire Wire Line
-	3500 2200 4600 2200
+	3500 2100 3900 2100
+Wire Wire Line
+	3500 2200 3875 2200
 Wire Wire Line
 	4350 1900 5000 1900
@@
 	3700 5400 3700 12325
 Wire Wire Line
-	3700 12325 16575 12325
+	3700 12325 6375 12325
 Connection ~ 3700 5400
 Wire Wire Line
@@
 	16875 11850 16875 12900
 Wire Wire Line
-	3575 12425 17025 12425
+	3575 12425 6400 12425
 Wire Wire Line
 	12100 12900 12100 10650
@@
 	600  6900 850  6900
 Connection ~ 850  7800
+$Comp
+L miniimu-9_v6:miniIMU-9_v6 U?
+U 1 1 6641AB3C
+P 5075 13425
+F 0 "U?" H 5553 13313 50  0000 L CNN
+F 1 "miniIMU-9_v6" H 5553 13222 50  0000 L CNN
+F 2 "" H 5075 13875 50  0001 C CNN
+F 3 "" H 5075 13875 50  0001 C CNN
+	1    5075 13425
+	1    0    0    -1
+$EndComp
+Wire Wire Line
+	4975 14025 4975 14200
+Wire Wire Line
+	5075 14025 5075 14225
+Wire Wire Line
+	3900 14200 3900 2100
+Wire Wire Line
+	3900 14200 4975 14200
+Connection ~ 3900 2100
+Wire Wire Line
+	3900 2100 4600 2100
+Wire Wire Line
+	3875 2200 3875 14225
+Wire Wire Line
+	3875 14225 5075 14225
+Connection ~ 3875 2200
+Wire Wire Line
+	3875 2200 4600 2200
+Wire Wire Line
+	3450 5600 3575 5600
+Wire Wire Line
+	5175 14025 5175 14325
+Wire Wire Line
+	5175 14325 6400 14325
+Wire Wire Line
+	6400 14325 6400 12425
+Connection ~ 6400 12425
+Wire Wire Line
+	6400 12425 17025 12425
+Wire Wire Line
+	5275 14025 5275 14300
+Wire Wire Line
+	5275 14300 6375 14300
+Wire Wire Line
+	6375 14300 6375 12325
+Connection ~ 6375 12325
+Wire Wire Line
+	6375 12325 16575 12325
 $EndSCHEMATC

Commit message: Commit message
Parts:
- removed 3.3vconverter1: ATA00F18S-L, Converter_DCDC:Converter_DCDC_Artesyn_ATA_SMD, symbol Converter_DCDC:ATA00F18S-L
- removed 5Vconverter1: ATA00A18S-L, Converter_DCDC:Converter_DCDC_Artesyn_ATA_SMD, symbol Converter_DCDC:ATA00A18S-L
- added 3.3vconverter: CC6-1203SR-E, custom:CC60512SRE, symbol CC6-1203SR-E:CC6-1203SR-E
- added 5vconverter: CC6-1205SF-E, CC6_SF, symbol cc6-1205sf-e:CC6-1205SF-E
Connections:
- wire segments 560 -> 561
Other:
- note added: "xt60 en xt30 connector"
- note removed: "tijdelijke plaatsing tot goede gevonden"
Changed lines of the file:
@@
 Text GLabel 1800 6250 0    50   Input ~ 0
 12v
-Wire Wire Line
-	4050 4950 4050 5400
-Wire Wire Line
-	4150 5600 4150 4900
 $Comp
 L pcb-rescue:Teensy4.1-teensy controllboard1
@@
 $EndComp
 Connection ~ 850  6900
-Connection ~ 1800 6500
-Wire Wire Line
-	1800 6500 1800 7350
-Wire Wire Line
-	1800 5400 1800 6500
 Wire Wire Line
 	850  6900 850  7150
-Wire Wire Line
-	850  5800 850  6900
-Text Notes 2200 6200 0    50   ~ 0
-tijdelijke plaatsing tot goede gevonden
-Text Notes 2350 5100 0    50   ~ 0
-tijdelijke plaatsing tot goede gevonden
-Wire Wire Line
-	3450 5400 3700 5400
-Wire Wire Line
-	2450 6500 1800 6500
-Wire Wire Line
-	2450 6900 1950 6900
-Wire Wire Line
-	850  5800 2450 5800
-Wire Wire Line
-	1800 5400 2450 5400
-$Comp
-L Converter_DCDC:ATA00F18S-L 3.3vconverter1
-U 1 1 6631FEBC
-P 2950 6700
-F 0 "3.3vconverter1" H 2950 7167 50  0000 C CNN
-F 1 "ATA00F18S-L" H 2950 7076 50  0000 C CNN
-F 2 "Converter_DCDC:Converter_DCDC_Artesyn_ATA_SMD" H 2950 6350 50  0001 C CIN
-F 3 "https://www.artesyn.com/power/assets/ata_series_ds_01apr2015_79c25814fd.pdf" H 2950 6250 50  0001 C CNN
-	1    2950 6700
-	1    0    0    -1
-$EndComp
-$Comp
-L Converter_DCDC:ATA00A18S-L 5Vconverter1
-U 1 1 6631ECD9
-P 2950 5600
-F 0 "5Vconverter1" H 2950 6067 50  0000 C CNN
-F 1 "ATA00A18S-L" H 2950 5976 50  0000 C CNN
-F 2 "Converter_DCDC:Converter_DCDC_Artesyn_ATA_SMD" H 2950 5250 50  0001 C CIN
-F 3 "https://www.artesyn.com/power/assets/ata_series_ds_01apr2015_79c25814fd.pdf" H 2950 5150 50  0001 C CNN
-	1    2950 5600
-	1    0    0    -1
-$EndComp
-Wire Wire Line
-	3450 6500 4350 6500
 Wire Wire Line
 	4350 6500 4350 6250
@@
 	4100 11050 4100 8450
 Connection ~ 4100 6700
-Wire Wire Line
-	4100 6700 3450 6700
 Wire Wire Line
 	6600 8450 4100 8450
@@
 Connection ~ 18275 12325
 Wire Wire Line
-	3700 5400 3700 12325
-Wire Wire Line
 	3700 12325 6375 12325
-Connection ~ 3700 5400
-Wire Wire Line
-	3700 5400 4050 5400
 Connection ~ 16575 12325
-Wire Wire Line
-	3575 5600 3575 12425
-Connection ~ 3575 5600
-Wire Wire Line
-	3575 5600 4150 5600
 Connection ~ 18725 12425
 Wire Wire Line
@@
 Wire Wire Line
 	16700 8325 16700 8175
-Connection ~ 1950 6900
 Wire Wire Line
 	1950 6900 850  6900
@@
 	3875 2200 4600 2200
 Wire Wire Line
-	3450 5600 3575 5600
-Wire Wire Line
 	5175 14025 5175 14325
 Wire Wire Line
@@
 Wire Wire Line
 	6375 12325 16575 12325
+Text Notes 675  7900 0    50   ~ 0
+xt60 en xt30 connector
+$Comp
+L CC6-1203SR-E:CC6-1203SR-E 3.3vconverter
+U 1 1 66758C94
+P 2025 6500
+F 0 "3.3vconverter" H 2725 6765 50  0000 C CNN
+F 1 "CC6-1203SR-E" H 2725 6674 50  0000 C CNN
+F 2 "custom:CC60512SRE" H 3275 6600 50  0001 L CNN
+F 3 "https://product.tdk.com/system/files/dam/doc/product/power/switching-power/dc-dc-converter/catalog/cc-e_e.pdf" H 3275 6500 50  0001 L CNN
+F 4 "DC-DC Converters, On-board type, Output: 3.96W, 3.3V, Isolated type, Option: SMD type" H 3275 6400 50  0001 L CNN "Description"
+F 5 "8.8" H 3275 6300 50  0001 L CNN "Height"
+F 6 "TDK" H 3275 6200 50  0001 L CNN "Manufacturer_Name"
+F 7 "CC6-1203SR-E" H 3275 6100 50  0001 L CNN "Manufacturer_Part_Number"
+F 8 "967-CC6-1203SR-E" H 3275 6000 50  0001 L CNN "Mouser Part Number"
+F 9 "https://www.mouser.co.uk/ProductDetail/TDK-Lambda/CC6-1203SR-E?qs=Vwh6e7toGLi4J%2FzloL2n3g%3D%3D" H 3275 5900 50  0001 L CNN "Mouser Price/Stock"
+F 10 "CC6-1203SR-E" H 3275 5800 50  0001 L CNN "Arrow Part Number"
+F 11 "https://www.arrow.com/en/products/cc6-1203sr-e/tdk-lambda-americas?region=nac" H 3275 5700 50  0001 L CNN "Arrow Price/Stock"
+	1    2025 6500
+	1    0    0    -1
+$EndComp
+Wire Wire Line
+	1800 5400 1800 6500
+Wire Wire Line
+	3425 6500 4350 6500
+Wire Wire Line
+	3425 6700 4100 6700
+Wire Wire Line
+	1800 6500 2025 6500
+Connection ~ 1800 6500
+Wire Wire Line
+	1800 6500 1800 7350
+Wire Wire Line
+	2025 6700 850  6700
+Connection ~ 850  6700
+Wire Wire Line
+	850  6700 850  6900
+$Comp
+L cc6-1205sf-e:CC6-1205SF-E 5vconverter
+U 1 1 66A897F1
+P 2250 5400
+F 0 "5vconverter" H 2850 5665 50  0000 C CNN
+F 1 "CC6-1205SF-E" H 2850 5574 50  0000 C CNN
+F 2 "CC6_SF" H 3300 5500 50  0001 L CNN
+F 3 "https://product.tdk.com/system/files/dam/doc/product/power/switching-power/dc-dc-converter/catalog/cc-e_e.pdf" H 3300 5400 50  0001 L CNN
+F 4 "dcdc,convertor TDK-Lambda Through Hole Isolated DC-DC Converter, I/O isolation 500V ac, Vout 5V dc" H 3300 5300 50  0001 L CNN "Description"
+F 5 "TDK" H 3300 5100 50  0001 L CNN "Manufacturer_Name"
+F 6 "CC6-1205SF-E" H 3300 5000 50  0001 L CNN "Manufacturer_Part_Number"
+F 7 "967-CC6-1205SF-E" H 3300 4900 50  0001 L CNN "Mouser Part Number"
+F 8 "https://www.mouser.co.uk/ProductDetail/TDK-Lambda/CC6-1205SF-E?qs=Vwh6e7toGLhaPHzXVKmH%252BA%3D%3D" H 3300 4800 50  0001 L CNN "Mouser Price/Stock"
+F 9 "CC6-1205SF-E" H 3300 4700 50  0001 L CNN "Arrow Part Number"
+F 10 "https://www.arrow.com/en/products/cc6-1205sf-e/tdk-lambda-americas?region=nac" H 3300 4600 50  0001 L CNN "Arrow Price/Stock"
+	1    2250 5400
+	1    0    0    -1
+$EndComp
+Wire Wire Line
+	2250 5400 1800 5400
+Wire Wire Line
+	2250 5600 850  5600
+Wire Wire Line
+	850  5600 850  6700
+Wire Wire Line
+	3450 5400 3575 5400
+Wire Wire Line
+	4150 5400 4150 4900
+Wire Wire Line
+	3575 5400 3575 12425
+Connection ~ 3575 5400
+Wire Wire Line
+	3575 5400 4150 5400
+Wire Wire Line
+	3450 5600 3700 5600
+Wire Wire Line
+	4050 5600 4050 4950
+Wire Wire Line
+	3700 12325 3700 5600
+Connection ~ 3700 5600
+Wire Wire Line
+	3700 5600 4050 5600
 $EndSCHEMATC

Commit message: Commit message
Parts:
- 3.3vconverter: symbol CC6-1203SR-E:CC6-1203SR-E -> pcb-rescue:CC6-1203SR-E-CC6-1203SR-E
Changed lines of the file:
@@
 xt60 en xt30 connector
 $Comp
-L CC6-1203SR-E:CC6-1203SR-E 3.3vconverter
+L pcb-rescue:CC6-1203SR-E-CC6-1203SR-E 3.3vconverter
 U 1 1 66758C94
 P 2025 6500

Commit message: Commit message
Parts:
- removed motor_driver1, motor_driver2: l298n, custom:l298n, symbol l298n:l298n
- added Motor_driver2, motor_driver1, motor_driver3: TB9051FTG, custom:TB9051FTG, symbol tb9051ftg:TB9051FTG
- kompas1: renamed from U?; footprint (none) -> custom:miniIMU-9_v6
- renumbered 3.3vconverter to 3.3vconverter1, 5vconverter to 5vconverter1
Connections:
- net +12V: now also Motor_driver2.1 (vin), motor_driver1.1 (vin), motor_driver3.1 (vin)
- net Earth: now also Motor_driver2.2 (gnd), motor_driver1.2 (gnd), motor_driver3.2 (gnd)
- net at controllboard1.44 (22_A8_CTX1): now also motor_driver3.11 (pwm2)
- net at controllboard1.45 (23_A9_CRX1_MCLK1): now also motor_driver3.12 (pwm)
- net at 5vconverter1.5 (-VOUT), BZ1.2 (+), R2.2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: now also Motor_driver2.6 (gnd), motor_driver1.6 (gnd), motor_driver3.6 (gnd)
- net at 5vconverter1.7 (+VOUT), controllboard1.48 (VIN), kompas1.3 (vin(2.5-5v))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: now also Motor_driver2.7 (vcc), motor_driver1.7 (vcc), motor_driver3.7 (vcc)
- net at io_expender2.1 (GPB0): now also motor_driver3.9 (en)
- net at io_expender2.2 (GPB1): now also Motor_driver2.12 (pwm)
- net at io_expender2.21 (GPA0): now also motor_driver1.9 (en)
- net at io_expender2.24 (GPA3): now also motor_driver3.10 (enB)
- net at io_expender2.3 (GPB2): now also Motor_driver2.11 (pwm2)
- net at io_expender2.4 (GPB3): now also Motor_driver2.10 (enB)
- net at io_expender2.5 (GPB4): now also Motor_driver2.9 (en)
- net at io_expender2.6 (GPB5): now also motor_driver1.12 (pwm)
- net at io_expender2.7 (GPB6): now also motor_driver1.11 (pwm2)
- net at io_expender2.8 (GPB7): now also motor_driver1.10 (enB)
- net at motor1.~ (-): now also motor_driver1.4 (out1)
- net at motor2.~ (-): now also Motor_driver2.4 (out1)
- net at motor3.~ (-): now also motor_driver3.4 (out1)
- new net: motor1.~ (-), motor_driver1.3 (out2)
- new net: Motor_driver2.3 (out2), motor2.~ (-)
- new net: motor3.~ (-), motor_driver3.3 (out2)

Commit message: Commit message
Parts:
- removed 5vconverter1: CC6-1205SF-E, CC6_SF, symbol cc6-1205sf-e:CC6-1205SF-E
- added PS1: SFTN01M-05N, custom:SFTN01M05N, symbol sftn01m-05n:SFTN01M-05N
Connections:
- net +12V: now also PS1.2 (+VIN)
- net Earth: now also PS1.1 (-VIN)
- net at BZ1.2 (+), Motor_driver2.6 (gnd), R2.2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: now also PS1.5 (-VOUT)
- net at Motor_driver2.7 (vcc), controllboard1.48 (VIN), kompas1.3 (vin(2.5-5v))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: now also PS1.8 (+VOUT)
- net at motor_driver1.12 (pwm): now also io_expender2.6 (GPB5)
- net at Motor_driver2.12 (pwm): now also io_expender2.2 (GPB1)
Changed lines of the file:
@@
 $EndComp
-Wire Wire Line
-	1800 5400 1800 6500
 Wire Wire Line
 	3425 6500 4350 6500
@@
 Wire Wire Line
 	1800 6500 2025 6500
-Connection ~ 1800 6500
 Wire Wire Line
 	1800 6500 1800 7350
@@
 Wire Wire Line
 	850  6700 850  6900
-$Comp
-L cc6-1205sf-e:CC6-1205SF-E 5vconverter1
-U 1 1 66A897F1
-P 2250 5400
-F 0 "5vconverter1" H 2850 5665 50  0000 C CNN
-F 1 "CC6-1205SF-E" H 2850 5574 50  0000 C CNN
-F 2 "CC6_SF" H 3300 5500 50  0001 L CNN
-F 3 "https://product.tdk.com/system/files/dam/doc/product/power/switching-power/dc-dc-converter/catalog/cc-e_e.pdf" H 3300 5400 50  0001 L CNN
-F 4 "dcdc,convertor TDK-Lambda Through Hole Isolated DC-DC Converter, I/O isolation 500V ac, Vout 5V dc" H 3300 5300 50  0001 L CNN "Description"
-F 5 "TDK" H 3300 5100 50  0001 L CNN "Manufacturer_Name"
-F 6 "CC6-1205SF-E" H 3300 5000 50  0001 L CNN "Manufacturer_Part_Number"
-F 7 "967-CC6-1205SF-E" H 3300 4900 50  0001 L CNN "Mouser Part Number"
-F 8 "https://www.mouser.co.uk/ProductDetail/TDK-Lambda/CC6-1205SF-E?qs=Vwh6e7toGLhaPHzXVKmH%252BA%3D%3D" H 3300 4800 50  0001 L CNN "Mouser Price/Stock"
-F 9 "CC6-1205SF-E" H 3300 4700 50  0001 L CNN "Arrow Part Number"
-F 10 "https://www.arrow.com/en/products/cc6-1205sf-e/tdk-lambda-americas?region=nac" H 3300 4600 50  0001 L CNN "Arrow Price/Stock"
-	1    2250 5400
-	1    0    0    -1
-$EndComp
-Wire Wire Line
-	2250 5400 1800 5400
-Wire Wire Line
-	2250 5600 850  5600
-Wire Wire Line
-	850  5600 850  6700
-Wire Wire Line
-	3450 5400 3575 5400
 Wire Wire Line
 	4150 5400 4150 4900
 Wire Wire Line
-	3575 5400 3575 12425
-Connection ~ 3575 5400
-Wire Wire Line
 	3575 5400 4150 5400
 Wire Wire Line
-	3450 5600 3700 5600
-Wire Wire Line
-	4050 5600 4050 4950
-Wire Wire Line
-	3700 12325 3700 5600
-Connection ~ 3700 5600
-Wire Wire Line
-	3700 5600 4050 5600
+	3700 12325 3700 5700
 $Comp
 L tb9051ftg:TB9051FTG motor_driver1
@@
 Connection ~ 19100 7900
 Connection ~ 20475 12425
+$Comp
+L sftn01m-05n:SFTN01M-05N PS1
+U 1 1 66490BE8
+P 1975 5400
+F 0 "PS1" H 2625 5665 50  0000 C CNN
+F 1 "SFTN01M-05N" H 2625 5574 50  0000 C CNN
+F 2 "custom:SFTN01M05N" H 3125 5500 50  0001 L CNN
+F 3 "https://www.meanwell.com/webapp/product/search.aspx?prod=SFTN01-N" H 3125 5400 50  0001 L CNN
+F 4 "Isolated DC/DC Converters - SMD 1W 12Vin 5Vout 20-200mA SMT Unregulated" H 3125 5300 50  0001 L CNN "Description"
+F 5 "7.6" H 3125 5200 50  0001 L CNN "Height"
+F 6 "Mean Well" H 3125 5100 50  0001 L CNN "Manufacturer_Name"
+F 7 "SFTN01M-05N" H 3125 5000 50  0001 L CNN "Manufacturer_Part_Number"
+F 8 "709-SFTN01M-05N" H 3125 4900 50  0001 L CNN "Mouser Part Number"
+F 9 "https://www.mouser.co.uk/ProductDetail/MEAN-WELL/SFTN01M-05N?qs=A6eO%252BMLsxmQLvWwJN5Fn%252BQ%3D%3D" H 3125 4800 50  0001 L CNN "Mouser Price/Stock"
+	1    1975 5400
+	1    0    0    -1
+$EndComp
+Wire Wire Line
+	1800 6500 1800 5500
+Wire Wire Line
+	1800 5500 1975 5500
+Connection ~ 1800 6500
+Wire Wire Line
+	1975 5400 850  5400
+Wire Wire Line
+	850  5400 850  6700
+Wire Wire Line
+	1975 5700 1900 5700
+Wire Wire Line
+	1900 5700 1900 5975
+Wire Wire Line
+	3275 5700 3700 5700
+Connection ~ 3700 5700
+Wire Wire Line
+	4050 5700 3700 5700
+Wire Wire Line
+	4050 4950 4050 5700
+Wire Wire Line
+	1900 5975 3575 5975
+Wire Wire Line
+	3575 5400 3575 5975
+Connection ~ 3575 5975
+Wire Wire Line
+	3575 5975 3575 12425
 $EndSCHEMATC

Commit message: pcb onder gemaakt
Connections:
- net at motor_driver1.12 (pwm): now also io_expender2.6 (GPB5)
- net at Motor_driver2.12 (pwm): now also io_expender2.2 (GPB1)
Changed lines of the file:
@@
 Connection ~ 10850 2300
-$Comp
-L Device:R R2
-U 1 1 675AF867
-P 11500 2725
-F 0 "R2" H 11570 2771 50  0000 L CNN
-F 1 "R" H 11570 2680 50  0000 L CNN
-F 2 "custom:resistor" V 11430 2725 50  0001 C CNN
-F 3 "~" H 11500 2725 50  0001 C CNN
-	1    11500 2725
-	1    0    0    -1
-$EndComp
 $Comp
 L Device:R R3
@@
 Wire Wire Line
 	3575 5975 3575 12425
+$Comp
+L Device:R R2
+U 1 1 675AF867
+P 11500 2725
+F 0 "R2" H 11570 2771 50  0000 L CNN
+F 1 "R" H 11570 2680 50  0000 L CNN
+F 2 "custom:resistor" V 11430 2725 50  0001 C CNN
+F 3 "~" H 11500 2725 50  0001 C CNN
+	1    11500 2725
+	1    0    0    -1
+$EndComp
 $EndSCHEMATC
