File: pcb_onder/pcb_onder.sch (KiCad schematic (older format))
At the start: 0 parts

Commit message: pcb onder gemaakt
Parts:
- added 3.3v_converter1: CC6-1203SR-E, custom:CC60512SRE, symbol cc6-1203sr-e:CC6-1203SR-E
- added 5v_converter1: SFTN01M-05N, custom:SFTN01M05N, symbol sftn01m-05n:SFTN01M-05N
- added i2c_multiplexer1: PCA9548ADB, Package_SO:SSOP-24_5.3x8.2mm_P0.65mm, symbol Interface_Expansion:PCA9548ADB
- added kleur_sensor_1, kleur_sensor_2, kleur_sensor_3, kleur_sensor_4, kleur_sensor_5, kleur_sensor_6: tcs3472_color_sensor, custom:tcs3472, symbol tcs3472_color_sensor:tcs3472_color_sensor
- added motor1, motor2, motor3: pololu_motor, custom:pololu_motor, symbol pololu_motor:pololu_motor
- added motor_driver1, motor_driver2, motor_driver3: TB9051FTG, custom:TB9051FTG, symbol tb9051ftg:TB9051FTG
- added port_multiplexer_2: MCP23017_SP, Package_DIP:DIP-28_W7.62mm, symbol Interface_Expansion:MCP23017_SP
- added xt30: Battery, Connector_AMASS:AMASS_XT30U-F_1x02_P5.0mm_Vertical, symbol Device:Battery
- added xt60: Battery, Connector_AMASS:AMASS_XT60-F_1x02_P7.20mm_Vertical, symbol Device:Battery
Connections:
- net labels added: +12v, 3.3v, 5v, A, B, gnd, sc6, scl, sd6, sda
- wire segments 0 -> 232
Other:
- note added: "omgedraaid omdat xt connectors \nvekeerd zitten in pcb ondwerp"
