File: pcb_onder/pcb_onder.kicad_pcb (KiCad board)
At the start: 2 copper layers, 147.7 x 147.7 mm, 22 parts, among them J1 Conn_01x10_Female, U1 screw_hole, U2 screw_hole, U3 screw_hole, U4 screw_hole, U5 screw_hole, U6 screw_hole

Commit message: pcb
Other:
- board size 147.7 x 147.7 mm -> 132.2 x 150.9 mm
