File: pcb_boven/pcb_boven.sch (KiCad schematic (older format))
At the start: 36 parts, among them U1 miniIMU-9_v6, U2 openMV_M7_R2

Commit message: i2c
Parts:
- added extrapins1: Conn_01x10_Female, custom:10connect, symbol Connector:Conn_01x10_Female
- added pwr_sw1: SW_DIP_x01, custom:dipswitch1, symbol Switch:SW_DIP_x01
Connections:
- net 3.3v: now also extrapins1.6 (Pin_6)
- net 5v: now also extrapins1.4 (Pin_4)
- net gnd: now also 3V3_converter1.3 (-VIN), 5V_converter1.1 (-VIN), xt30.2 (-), xt60.2 (-), extrapins1.5 (Pin_5), pwr_sw1.2
- net sc6: no longer Portmultiplexer1.12 (SCK), pcb_conn1.5 (Pin_5)
- net scl: now also Portmultiplexer1.12 (SCK), extrapins1.10 (Pin_10)
- net sd6: no longer Portmultiplexer1.13 (SDA), pcb_conn1.6 (Pin_6)
- net sda: now also Portmultiplexer1.13 (SDA), extrapins1.9 (Pin_9)
- net 25: now reaches control_board1.17 (25_A11_RX6_SDA2)
- net 25: now also extrapins1.8 (Pin_8)
- net 26: now reaches control_board1.18 (26_A12_MOSI1)
- net 26: now also extrapins1.7 (Pin_7)
- net 27: now reaches control_board1.19 (27_A13_SCK1)
- net 27: now also extrapins1.2 (Pin_2)
- net 28: now reaches control_board1.20 (28_RX7)
- net 28: now also extrapins1.1 (Pin_1)
- net 12V: now reaches 3V3_converter1.1 (+VIN), 5V_converter1.2 (+VIN), xt30.1 (+), xt60.1 (+)
- net 12V: now also pcb_conn1.7 (Pin_7), extrapins1.3 (Pin_3)
- net at 3V3_converter1.2 (RC): now also pwr_sw1.1
Changed lines of the file:
@@
 	8100 7300 8100 10775
 Wire Wire Line
-	8100 10775 950  10775
+	8100 10775 3450 10775
 Text GLabel 1300 10775 0    50   Input ~ 0
 scl
@@
 	8075 7400 8075 10675
 Wire Wire Line
-	8075 10675 950  10675
+	8075 10675 3400 10675
 Text GLabel 1300 10675 0    50   Input ~ 0
 sda
@@
 Wire Wire Line
 	8125 6700 8125 10875
-Wire Wire Line
-	8125 10875 950  10875
 Text GLabel 1300 10875 0    50   Input ~ 0
 gnd
@@
 	8150 6600 8150 10975
 Wire Wire Line
-	8150 10975 950  10975
+	8150 10975 2600 10975
 Text GLabel 1300 10975 0    50   Input ~ 0
 5v
 Text Notes 975  11100 0    50   ~ 0
 naar pcb onder
-Wire Wire Line
-	9150 7200 9150 10575
-Wire Wire Line
-	9150 10575 950  10575
-Wire Wire Line
-	9150 7200 10325 7200
-Wire Wire Line
-	10325 7100 9125 7100
-Wire Wire Line
-	9125 7100 9125 10475
-Wire Wire Line
-	9125 10475 950  10475
 Text GLabel 1300 10475 0    50   Input ~ 0
 sd6
@@
 	8700 5825 8750 5825
 Wire Wire Line
-	950  10275 9075 10275
+	950  10275 2775 10275
 Text GLabel 1300 10275 0    50   Input ~ 0
 3.3v
@@
 $EndComp
 Wire Wire Line
-	1600 4925 1975 4925
-Wire Wire Line
 	1975 5325 1600 5325
 Wire Wire Line
@@
 Wire Wire Line
 	2625 5125 2525 5125
-Wire Wire Line
-	2525 5125 2525 5625
 Wire Wire Line
 	2525 5625 3750 5625
@@
 	5150 4500 5150 4475
 Connection ~ 4125 4500
+$Comp
+L Connector:Conn_01x10_Female extrapins1
+U 1 1 66687DFB
+P 1950 8950
+F 0 "extrapins1" H 1842 8225 50  0000 C CNN
+F 1 "Conn_01x10_Female" H 1842 8316 50  0000 C CNN
+F 2 "custom:10connect" H 1950 8950 50  0001 C CNN
+F 3 "~" H 1950 8950 50  0001 C CNN
+	1    1950 8950
+	-1   0    0    1
+$EndComp
+Wire Wire Line
+	3450 10775 3450 8700
+Wire Wire Line
+	3450 8700 2725 8700
+Wire Wire Line
+	2725 8700 2725 8450
+Wire Wire Line
+	2725 8450 2150 8450
+Connection ~ 3450 10775
+Wire Wire Line
+	3450 10775 950  10775
+Wire Wire Line
+	3400 10675 3400 8725
+Wire Wire Line
+	3400 8725 2700 8725
+Wire Wire Line
+	2700 8725 2700 8550
+Wire Wire Line
+	2700 8550 2150 8550
+Connection ~ 3400 10675
+Wire Wire Line
+	3400 10675 950  10675
+Wire Wire Line
+	5025 8200 4600 8200
+Wire Wire Line
+	4600 8200 4600 8750
+Wire Wire Line
+	4600 8750 2675 8750
+Wire Wire Line
+	2675 8750 2675 8650
+Wire Wire Line
+	2675 8650 2150 8650
+Wire Wire Line
+	5025 8300 4625 8300
+Wire Wire Line
+	2150 8775 2150 8750
+Wire Wire Line
+	4625 8300 4625 8775
+Wire Wire Line
+	2150 8775 4625 8775
+Wire Wire Line
+	2150 8850 2775 8850
+Wire Wire Line
+	2775 8850 2775 10275
+Connection ~ 2775 10275
+Wire Wire Line
+	2775 10275 9075 10275
+Wire Wire Line
+	2150 8950 2675 8950
+Wire Wire Line
+	2675 8950 2675 10875
+Wire Wire Line
+	950  10875 2675 10875
+Connection ~ 2675 10875
+Wire Wire Line
+	2675 10875 8125 10875
+Wire Wire Line
+	2150 9050 2600 9050
+Wire Wire Line
+	2600 9050 2600 10975
+Connection ~ 2600 10975
+Wire Wire Line
+	2600 10975 950  10975
+Wire Wire Line
+	950  10375 2525 10375
+Wire Wire Line
+	3800 10375 3800 8600
+Wire Wire Line
+	3800 8600 2825 8600
+Wire Wire Line
+	2825 8600 2825 5725
+Wire Wire Line
+	2825 5725 1325 5725
+Wire Wire Line
+	1325 5725 1325 4925
+Wire Wire Line
+	1325 4925 1600 4925
+Connection ~ 1600 4925
+Wire Wire Line
+	1600 4925 1975 4925
+Wire Wire Line
+	2300 5325 2525 5325
+Wire Wire Line
+	2525 5125 2525 5325
+Connection ~ 2300 5325
+Connection ~ 2525 5325
+Wire Wire Line
+	2525 5325 2525 5625
+Text GLabel 1300 10375 0    50   Input ~ 0
+12V
+Wire Wire Line
+	2525 10375 2525 9150
+Wire Wire Line
+	2525 9150 2150 9150
+Connection ~ 2525 10375
+Wire Wire Line
+	2525 10375 3800 10375
+Text GLabel 2325 8450 0    50   Input ~ 0
+scl
+Text GLabel 2350 8550 0    50   Input ~ 0
+sda
+Text GLabel 2325 8650 0    50   Input ~ 0
+25
+Text GLabel 2325 8775 0    50   Input ~ 0
+26
+Text GLabel 2350 8850 0    50   Input ~ 0
+3v3
+Text GLabel 2350 8950 0    50   Input ~ 0
+gnd
+Text GLabel 2350 9050 0    50   Input ~ 0
+5v
+Text GLabel 2350 9150 0    50   Input ~ 0
+12v
+Wire Wire Line
+	2150 9250 4650 9250
+Wire Wire Line
+	4650 9250 4650 8400
+Wire Wire Line
+	4650 8400 5025 8400
+Wire Wire Line
+	5025 8500 4675 8500
+Wire Wire Line
+	4675 8500 4675 9275
+Wire Wire Line
+	4675 9275 2450 9275
+Wire Wire Line
+	2450 9275 2450 9350
+Wire Wire Line
+	2450 9350 2150 9350
+Text GLabel 2350 9250 0    50   Input ~ 0
+27
+Text GLabel 2350 9350 0    50   Input ~ 0
+28
+$Comp
+L Switch:SW_DIP_x01 pwr_sw1
+U 1 1 66829A54
+P 2400 3850
+F 0 "pwr_sw1" H 2400 3583 50  0000 C CNN
+F 1 "SW_DIP_x01" H 2400 3674 50  0000 C CNN
+F 2 "custom:dipswitch1" H 2400 3850 50  0001 C CNN
+F 3 "~" H 2400 3850 50  0001 C CNN
+	1    2400 3850
+	-1   0    0    1
+$EndComp
+Wire Wire Line
+	2300 4500 2100 4500
+Wire Wire Line
+	2100 4500 2100 3850
+Connection ~ 2300 4500
+Wire Wire Line
+	2600 4400 2525 4400
+Wire Wire Line
+	2525 4400 2525 4050
+Wire Wire Line
+	2525 4050 2700 4050
+Wire Wire Line
+	2700 4050 2700 3850
+Wire Wire Line
+	8075 7400 8825 7400
+Wire Wire Line
+	8825 7400 8825 7100
+Connection ~ 8075 7400
+Wire Wire Line
+	8275 7200 8275 7300
+Wire Wire Line
+	8275 7300 8100 7300
+Connection ~ 8100 7300
+Wire Wire Line
+	8275 7200 10325 7200
+Wire Wire Line
+	8825 7100 10325 7100
 $EndSCHEMATC

Commit message: 4dip
Parts:
- removed R6, R7: R, custom:resistor, symbol Device:R
- removed dip_swith_instellinen1: SW_DIP_x06, custom:dipswitch6, symbol Switch:SW_DIP_x06
- added SW1: SW_DIP_x04, custom:dipswitch4, symbol Switch:SW_DIP_x04
Connections:
- net at R2.2, control_board1.4 (2_OUT2): now also SW1.8
- net at control_board1.46 (3V3): now also SW1.1, SW1.2, SW1.3, SW1.4
- net at R3.2, control_board1.5 (3_LRCLK2): now also SW1.7
- net at R4.2, control_board1.6 (4_BCLK2): now also SW1.6
- net at R5.2, control_board1.7 (5_IN2): now also SW1.5
Changed lines of the file:
@@
-$EndComp
-$Comp
-L Switch:SW_DIP_x06 dip_swith_instellinen1
-U 1 1 66364D70
-P 3575 7200
-F 0 "dip_swith_instellinen1" H 3575 7767 50  0000 C CNN
-F 1 "SW_DIP_x06" H 3575 7676 50  0000 C CNN
-F 2 "custom:dipswitch6" H 3575 7200 50  0001 C CNN
-F 3 "~" H 3575 7200 50  0001 C CNN
-	1    3575 7200
-	1    0    0    -1
 $EndComp
 $Comp
@@
 $EndComp
 $Comp
-L Device:R R6
-U 1 1 66553C02
-P 4650 6175
-F 0 "R6" V 4443 6175 50  0000 C CNN
-F 1 "R" V 4534 6175 50  0000 C CNN
-F 2 "custom:resistor" V 4580 6175 50  0001 C CNN
-F 3 "~" H 4650 6175 50  0001 C CNN
-	1    4650 6175
-	1    0    0    -1
-$EndComp
-$Comp
-L Device:R R7
-U 1 1 6655A960
-P 4800 6175
-F 0 "R7" V 4593 6175 50  0000 C CNN
-F 1 "R" V 4684 6175 50  0000 C CNN
-F 2 "custom:resistor" V 4730 6175 50  0001 C CNN
-F 3 "~" H 4800 6175 50  0001 C CNN
-	1    4800 6175
-	1    0    0    -1
-$EndComp
-$Comp
 L Device:R R1
 U 1 1 665A1C89
@@
 	5025 7200 4500 7200
 Wire Wire Line
-	3875 7300 4650 7300
-Wire Wire Line
 	4050 6325 4050 6900
 Connection ~ 4050 6900
@@
 	4500 7200 3875 7200
 Wire Wire Line
-	4650 6325 4650 7300
-Connection ~ 4650 7300
-Wire Wire Line
-	4650 7300 5025 7300
-Wire Wire Line
-	4800 6325 4800 7400
-Wire Wire Line
-	3875 7400 4800 7400
-Connection ~ 4800 7400
-Wire Wire Line
-	4800 7400 5025 7400
-Wire Wire Line
-	3275 7400 3275 7300
-Wire Wire Line
-	3275 7300 3275 7200
-Connection ~ 3275 7300
-Wire Wire Line
 	3275 7200 3275 7100
-Connection ~ 3275 7200
 Wire Wire Line
 	3275 7000 3275 6900
@@
 Wire Wire Line
 	4350 6025 4500 6025
-Wire Wire Line
-	4650 6025 4800 6025
-Wire Wire Line
-	4650 6025 4500 6025
-Connection ~ 4650 6025
 Connection ~ 4500 6025
 Wire Wire Line
@@
 Connection ~ 4200 6025
 Wire Wire Line
-	4800 6025 7275 6025
-Wire Wire Line
 	7550 6025 7550 6700
-Connection ~ 4800 6025
 Connection ~ 7550 6700
 Wire Wire Line
@@
 Wire Wire Line
 	8825 7100 10325 7100
+$Comp
+L Switch:SW_DIP_x04 SW1
+U 1 1 666FC3F3
+P 3575 7100
+F 0 "SW1" H 3575 7567 50  0000 C CNN
+F 1 "SW_DIP_x04" H 3575 7476 50  0000 C CNN
+F 2 "custom:dipswitch4" H 3575 7100 50  0001 C CNN
+F 3 "~" H 3575 7100 50  0001 C CNN
+	1    3575 7100
+	1    0    0    -1
+$EndComp
+Wire Wire Line
+	4500 6025 7275 6025
 $EndSCHEMATC

Commit message: code
Connections:
- net at U2.2 (p0): no longer control_board1.13 (11_MOSI_CTX1)
- net at U2.3 (p1): no longer control_board1.14 (12_MISO_MQSL)
- net at U2.4 (p2): no longer control_board1.28 (36_CS)
- net at U2.5 (p3): no longer control_board1.12 (10_CS_MQSR)
- net at U2.6 (p4): now also control_board1.2 (0_RX1_CRX2_CS1)
- net at U2.7 (p5): now also control_board1.3 (1_TX1_CTX2_MISO1)
Changed lines of the file:
@@
 Connection ~ 8700 5825
 Wire Wire Line
-	8750 5425 4975 5425
-Wire Wire Line
-	4975 5425 4975 7700
-Wire Wire Line
-	4975 7700 5025 7700
-Wire Wire Line
 	5025 8100 4800 8100
-Wire Wire Line
-	5025 7800 4950 7800
-Wire Wire Line
-	4950 7800 4950 5300
-Wire Wire Line
-	4950 5300 8275 5300
-Wire Wire Line
-	8275 5300 8275 5125
-Wire Wire Line
-	8275 5125 8750 5125
-Wire Wire Line
-	8750 5225 8325 5225
-Wire Wire Line
-	8325 5225 8325 5350
-Wire Wire Line
-	8325 5350 4925 5350
-Wire Wire Line
-	4925 5350 4925 7900
-Wire Wire Line
-	4925 7900 5025 7900
-Wire Wire Line
-	7225 8600 8475 8600
-Wire Wire Line
-	8475 8600 8475 5325
-Wire Wire Line
-	8475 5325 8750 5325
 Wire Wire Line
 	7350 7300 8100 7300
@@
 Wire Wire Line
 	4500 6025 7275 6025
+Wire Wire Line
+	4925 6700 4925 5350
+Wire Wire Line
+	4925 5350 8550 5350
+Wire Wire Line
+	8550 5350 8550 5525
+Wire Wire Line
+	8550 5525 8750 5525
+Wire Wire Line
+	4925 6700 5025 6700
+Wire Wire Line
+	8750 5625 8525 5625
+Wire Wire Line
+	8525 5625 8525 5375
+Wire Wire Line
+	8525 5375 4950 5375
+Wire Wire Line
+	4950 5375 4950 6800
+Wire Wire Line
+	4950 6800 5025 6800
 $EndSCHEMATC
