File: pcb_boven/pcb_boven.kicad_pcb (KiCad board)
At the start: 2 copper layers, 30 parts, among them U1 miniIMU-9_v6, U2 openMV_M7_R2

Commit message: pcb onder gemaakt
Parts:
- moved R1 23.4 mm to (145.3, 104.2)
- moved R2 23.4 mm to (174.7, 76.4)
- moved R3 23.4 mm to (152.9, 96.7)
- moved R6 23.4 mm to (160.5, 91.6)
- moved R7 23.4 mm to (138.4, 113.1)
- moved control_board1 23.4 mm to (108.0, 79.0)
- moved goal_kleur1 23.4 mm to (130.8, 113.1)
- moved ir_sensor_1 23.4 mm to (152.9, 91.6)
- moved ir_sensor_10 23.4 mm to (130.8, 115.6)
- moved ir_sensor_11 23.4 mm to (167.1, 71.3)
- moved ir_sensor_12 23.4 mm to (145.3, 91.6)
- moved ir_sensor_13 23.4 mm to (167.1, 81.4)
- moved ir_sensor_14 23.4 mm to (145.3, 101.7)
- moved ir_sensor_15 23.4 mm to (174.7, 73.8)
- moved ir_sensor_16 23.4 mm to (152.9, 94.2)
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Connections:
- ir_sensor_1 pad 1: Net-(ir_sensor_1-Pad1) -> 3.3v
- ir_sensor_1 pad 2: Net-(ir_sensor_1-Pad2) -> gnd
- ir_sensor_10 pad 1: Net-(ir_sensor_1-Pad1) -> 3.3v
- ir_sensor_10 pad 2: Net-(ir_sensor_1-Pad2) -> gnd
- ir_sensor_11 pad 1: Net-(ir_sensor_1-Pad1) -> 3.3v
- ir_sensor_11 pad 2: Net-(ir_sensor_1-Pad2) -> gnd
- ir_sensor_12 pad 1: Net-(ir_sensor_1-Pad1) -> 3.3v
- ir_sensor_12 pad 2: Net-(ir_sensor_1-Pad2) -> gnd
- ir_sensor_13 pad 1: Net-(ir_sensor_1-Pad1) -> 3.3v
- ir_sensor_13 pad 2: Net-(ir_sensor_1-Pad2) -> gnd
- ir_sensor_14 pad 1: Net-(ir_sensor_1-Pad1) -> 3.3v
- ir_sensor_14 pad 2: Net-(ir_sensor_1-Pad2) -> gnd
- ir_sensor_15 pad 1: Net-(ir_sensor_1-Pad1) -> 3.3v
- ir_sensor_15 pad 2: Net-(ir_sensor_1-Pad2) -> gnd
- ir_sensor_16 pad 1: Net-(ir_sensor_1-Pad1) -> 3.3v
- ir_sensor_16 pad 2: Net-(ir_sensor_1-Pad2) -> gnd
- ir_sensor_2 pad 1: Net-(ir_sensor_1-Pad1) -> 3.3v
- ir_sensor_2 pad 2: Net-(ir_sensor_1-Pad2) -> gnd
- ir_sensor_3 pad 1: Net-(ir_sensor_1-Pad1) -> 3.3v
- ir_sensor_3 pad 2: Net-(ir_sensor_1-Pad2) -> gnd
- ir_sensor_4 pad 1: Net-(ir_sensor_1-Pad1) -> 3.3v
- ir_sensor_4 pad 2: Net-(ir_sensor_1-Pad2) -> gnd
- ir_sensor_5 pad 1: Net-(ir_sensor_1-Pad1) -> 3.3v
- ir_sensor_5 pad 2: Net-(ir_sensor_1-Pad2) -> gnd
- ir_sensor_6 pad 1: Net-(ir_sensor_1-Pad1) -> 3.3v
- ir_sensor_6 pad 2: Net-(ir_sensor_1-Pad2) -> gnd
- ir_sensor_7 pad 1: Net-(ir_sensor_1-Pad1) -> 3.3v
- ir_sensor_7 pad 2: Net-(ir_sensor_1-Pad2) -> gnd
- ir_sensor_8 pad 1: Net-(ir_sensor_1-Pad1) -> 3.3v
- ir_sensor_8 pad 2: Net-(ir_sensor_1-Pad2) -> gnd
- ir_sensor_9 pad 1: Net-(ir_sensor_1-Pad1) -> 3.3v
- ir_sensor_9 pad 2: Net-(ir_sensor_1-Pad2) -> gnd

Commit message: pcb
Parts:
- added 3V3_converter1: CC6-1203SR-E, custom:CC60512SRE, F.Cu at (91.4, 53.3)
- added 5V_converter1: SFTN01M-05N, custom:SFTN01M05N, F.Cu at (152.4, 77.5)
- added xt30: Battery, Connector_AMASS:AMASS_XT30U-F_1x02_P5.0mm_Vertical, F.Cu at (147.3, 49.5)
- added xt60: Battery, Connector_AMASS:AMASS_XT60-F_1x02_P7.20mm_Vertical, F.Cu at (143.5, 58.4)
- moved ir_sensor_7 158.9 mm to (41.9, 158.8), turned to 135 degrees
- moved ir_sensor_5 151.2 mm to (17.8, 100.3), turned to 90 degrees
- moved ir_sensor_3 129.2 mm to (41.9, 41.9), turned to 45 degrees
- moved ir_sensor_6 126.3 mm to (24.1, 132.1), turned to 112.5 degrees
- moved ir_sensor_9 123.6 mm to (100.3, 182.9), turned to 180 degrees
- moved ir_sensor_4 112.3 mm to (22.9, 68.6), turned to 67.5 degrees
- moved ir_sensor_8 109.0 mm to (68.6, 176.5), turned to 157.5 degrees
- moved ir_sensor_2 103.9 mm to (68.6, 24.1), turned to 22.5 degrees
- moved ir_sensor_1 90.7 mm to (100.3, 17.8)
- moved ir_sensor_11 87.8 mm to (158.8, 158.8), turned to 225 degrees
- moved ir_sensor_16 73.1 mm to (132.1, 24.1), turned to 337.5 degrees
- moved Portmultiplexer1 70.3 mm to (50.8, 53.3)
- moved R2 66.1 mm to (143.5, 134.6)
- moved ir_sensor_10 62.2 mm to (132.1, 177.8), turned to 202.5 degrees
- moved U2 58.1 mm to (100.3, 114.3)
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Connections:
- Portmultiplexer1 pad 15: Net-(Portmultiplexer1-Pad15) -> gnd
- Portmultiplexer1 pad 16: Net-(Portmultiplexer1-Pad16) -> gnd
- Portmultiplexer1 pad 17: Net-(Portmultiplexer1-Pad17) -> gnd
- control_board1 pad 12: A -> Net-(U2-Pad5)
- control_board1 pad 13: Net-(control_board1-Pad13) -> Net-(U2-Pad2)
- control_board1 pad 14: Net-(control_board1-Pad14) -> Net-(U2-Pad3)
- control_board1 pad 16: Net-(control_board1-Pad16) -> A
- control_board1 pad 2: Net-(control_board1-Pad2) -> scl
- control_board1 pad 28: Net-(control_board1-Pad28) -> Net-(U2-Pad4)
- control_board1 pad 3: Net-(control_board1-Pad3) -> sda
Routing:
- net gnd: track 0.00 -> 657.0 mm
- net 3.3v: track 0.00 -> 626.8 mm, vias 0 -> 2
- net Net-(Portmultiplexer1-Pad3): track 0.00 -> 236.4 mm, vias 0 -> 1
- net Net-(Portmultiplexer1-Pad4): track 0.00 -> 225.1 mm
- net Net-(Portmultiplexer1-Pad1): track 0.00 -> 219.2 mm
- net Net-(Portmultiplexer1-Pad2): track 0.00 -> 207.9 mm, vias 0 -> 1
- net Net-(Portmultiplexer1-Pad8): track 0.00 -> 171.8 mm, vias 0 -> 2
- net Net-(Portmultiplexer1-Pad5): track 0.00 -> 155.1 mm
- net Net-(Portmultiplexer1-Pad6): track 0.00 -> 133.2 mm
- net Net-(Portmultiplexer1-Pad28): track 0.00 -> 128.6 mm
- net Net-(3V3_converter1-Pad1): track 0.00 -> 126.0 mm
- net Net-(Portmultiplexer1-Pad27): track 0.00 -> 121.9 mm
- net Net-(Portmultiplexer1-Pad7): track 0.00 -> 121.0 mm
- net Net-(Portmultiplexer1-Pad26): track 0.00 -> 114.5 mm
- net Net-(3V3_converter1-Pad3): track 0.00 -> 109.3 mm
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Other:
- board outline added: 170.4 x 170.4 mm

Commit message: upd pcb
Parts:
- added pcb_conn1: Conn_01x10_Female, custom:10connect, F.Cu at (99.1, 74.9)
- control_board1: footprint custom:teensy4.1 -> teensy:Teensy41
- moved control_board1 20.5 mm to (68.6, 127.0), turned to 270 degrees
Connections:
- U2 pad 17: (no net) -> gnd
- U2 pad 6: scl -> Net-(U2-Pad6)
- U2 pad 7: sda -> Net-(U2-Pad7)
- U2 pad screw: Net-(U2-Padscrew) -> gnd
- control_board1 pad 2: scl -> Net-(control_board1-Pad2)
- control_board1 pad 3: sda -> Net-(control_board1-Pad3)
Routing:
- net gnd: track 657.0 -> 1020.8 mm
- net 3.3v: track 626.8 -> 821.4 mm, vias 2 -> 4
- net Net-(R5-Pad2): track 7.62 -> 137.8 mm
- net 5v: track 0.00 -> 128.6 mm
- net Net-(R6-Pad2): track 7.62 -> 124.6 mm
- net Net-(R4-Pad2): track 7.62 -> 123.9 mm
- net Net-(R3-Pad2): track 7.62 -> 120.7 mm
- net scl: track 0.00 -> 110.7 mm, vias 0 -> 1
- net A: track 0.00 -> 110.5 mm, vias 0 -> 1
- net Net-(R2-Pad2): track 7.62 -> 115.0 mm
- net Net-(control_board1-Pad46): track 0.00 -> 105.7 mm
- net sda: track 0.00 -> 104.6 mm, vias 0 -> 1
- net B: track 0.00 -> 79.7 mm, vias 0 -> 2
- net sd6: track 0.00 -> 71.8 mm, vias 0 -> 1
- net sc6: track 0.00 -> 56.6 mm, vias 0 -> 2
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
Commit message: f
Other:
- outline, holes or cut-outs redrawn
Changed lines of the file:
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@@
   (general
     (thickness 1.6)
-    (drawings 19)
+    (drawings 88)
     (tracks 572)
     (zones 0)
@@
       (net 2 "Net-(BZ1-Pad1)"))
   )
+  (gr_line (start 109.22 63.5) (end 127 63.5) (layer Edge.Cuts) (width 0.05))
+  (gr_line (start 109.22 66.04) (end 109.22 63.5) (layer Edge.Cuts) (width 0.05))
+  (gr_line (start 101.6 66.04) (end 109.22 66.04) (layer Edge.Cuts) (width 0.05))
+  (gr_line (start 101.6 68.58) (end 101.6 66.04) (layer Edge.Cuts) (width 0.05))
+  (gr_line (start 121.92 68.58) (end 101.6 68.58) (layer Edge.Cuts) (width 0.05))
+  (gr_line (start 127 63.5) (end 121.92 68.58) (layer Edge.Cuts) (width 0.05))
+  (gr_line (start 146.05 63.5) (end 130.81 63.5) (layer Edge.Cuts) (width 0.05))
+  (gr_line (start 146.05 69.85) (end 146.05 63.5) (layer Edge.Cuts) (width 0.05))
+  (gr_line (start 124.46 69.85) (end 146.05 69.85) (layer Edge.Cuts) (width 0.05))
+  (gr_line (start 130.81 63.5) (end 124.46 69.85) (layer Edge.Cuts) (width 0.05))
+  (gr_line (start 101.6 26.67) (end 90.17 26.67) (layer Edge.Cuts) (width 0.05))
+  (gr_line (start 101.6 40.64) (end 101.6 26.67) (layer Edge.Cuts) (width 0.05))
+  (gr_line (start 78.74 39.37) (end 101.6 40.64) (layer Edge.Cuts) (width 0.05))
+  (gr_line (start 90.17 26.67) (end 78.74 39.37) (layer Edge.Cuts) (width 0.05))
+  (gr_line (start 88.9 81.28) (end 67.31 80.01) (layer Edge.Cuts) (width 0.05))
+  (gr_line (start 73.66 93.98) (end 88.9 81.28) (layer Edge.Cuts) (width 0.05))
+  (gr_line (start 63.5 85.09) (end 73.66 93.98) (layer Edge.Cuts) (width 0.05))
+  (gr_line (start 67.31 80.01) (end 63.5 85.09) (layer Edge.Cuts) (width 0.05))
+  (gr_line (start 46.99 66.04) (end 31.75 80.01) (layer Edge.Cuts) (width 0.05))
+  (gr_line (start 46.99 88.9) (end 46.99 66.04) (layer Edge.Cuts) (width 0.05))
+  (gr_line (start 50.8 90.17) (end 46.99 88.9) (layer Edge.Cuts) (width 0.05))
+  (gr_line (start 50.8 99.06) (end 50.8 90.17) (layer Edge.Cuts) (width 0.05))
+  (gr_line (start 36.83 99.06) (end 50.8 99.06) (layer Edge.Cuts) (width 0.05))
+  (gr_line (start 31.75 102.87) (end 36.83 99.06) (layer Edge.Cuts) (width 0.05))
+  (gr_line (start 31.75 80.01) (end 31.75 102.87) (layer Edge.Cuts) (width 0.05))
+  (gr_line (start 146.05 41.91) (end 133.35 31.75) (layer Edge.Cuts) (width 0.05))
+  (gr_line (start 140.97 48.26) (end 146.05 41.91) (layer Edge.Cuts) (width 0.05))
+  (gr_line (start 118.11 45.72) (end 140.97 48.26) (layer Edge.Cuts) (width 0.05))
+  (gr_line (start 133.35 31.75) (end 118.11 45.72) (layer Edge.Cuts) (width 0.05))
+  (gr_line (start 171.45 93.98) (end 153.67 86.36) (layer Edge.Cuts) (width 0.05))
+  (gr_line (start 171.45 113.03) (end 171.45 93.98) (layer Edge.Cuts) (width 0.05))
+  (gr_line (start 163.83 120.65) (end 171.45 113.03) (layer Edge.Cuts) (width 0.05))
+  (gr_line (start 142.24 99.06) (end 163.83 120.65) (layer Edge.Cuts) (width 0.05))
+  (gr_line (start 153.67 86.36) (end 142.24 99.06) (layer Edge.Cuts) (width 0.05))
+  (gr_line (start 3.81 100.33) (end 207.01 100.33) (layer Dwgs.User) (width 0.15))
+  (gr_line (start 52.07 128.27) (end 41.91 132.08) (layer Edge.Cuts) (width 0.05))
+  (gr_line (start 53.34 148.59) (end 52.07 128.27) (layer Edge.Cuts) (width 0.05))
+  (gr_line (start 50.8 149.86) (end 53.34 148.59) (layer Edge.Cuts) (width 0.05))
+  (gr_line (start 41.91 140.97) (end 50.8 149.86) (layer Edge.Cuts) (width 0.05))
+  (gr_line (start 41.91 132.08) (end 41.91 140.97) (layer Edge.Cuts) (width 0.05))
+  (gr_line (start 50.8 105.41) (end 31.75 107.95) (layer Edge.Cuts) (width 0.05))
+  (gr_line (start 50.8 121.92) (end 50.8 105.41) (layer Edge.Cuts) (width 0.05))
+  (gr_line (start 44.45 128.27) (end 50.8 121.92) (layer Edge.Cuts) (width 0.05))
+  (gr_line (start 31.75 127) (end 44.45 128.27) (layer Edge.Cuts) (width 0.05))
+  (gr_line (start 31.75 107.95) (end 31.75 127) (layer Edge.Cuts) (width 0.05))
+  (gr_line (start 119.38 115.57) (end 119.38 129.54) (layer Edge.Cuts) (width 0.05))
+  (gr_line (start 132.08 114.3) (end 119.38 115.57) (layer Edge.Cuts) (width 0.05))
+  (gr_line (start 138.43 121.92) (end 132.08 114.3) (layer Edge.Cuts) (width 0.05))
+  (gr_line (start 138.43 135.89) (end 138.43 121.92) (layer Edge.Cuts) (width 0.05))
+  (gr_line (start 132.08 140.97) (end 138.43 135.89) (layer Edge.Cuts) (width 0.05))
+  (gr_line (start 119.38 129.54) (end 132.08 140.97) (layer Edge.Cuts) (width 0.05))
+  (gr_line (start 135.89 160.02) (end 130.81 167.64) (layer Edge.Cuts) (width 0.05))
+  (gr_line (start 151.13 154.94) (end 135.89 160.02) (layer Edge.Cuts) (width 0.05))
+  (gr_line (start 157.48 153.67) (end 151.13 154.94) (layer Edge.Cuts) (width 0.05))
+  (gr_line (start 154.94 148.59) (end 157.48 153.67) (layer Edge.Cuts) (width 0.05))
+  (gr_line (start 140.97 138.43) (end 154.94 148.59) (layer Edge.Cuts) (width 0.05))
+  (gr_line (start 132.08 148.59) (end 140.97 138.43) (layer Edge.Cuts) (width 0.05))
+  (gr_line (start 125.73 148.59) (end 132.08 148.59) (layer Edge.Cuts) (width 0.05))
+  (gr_line (start 125.73 161.29) (end 125.73 148.59) (layer Edge.Cuts) (width 0.05))
+  (gr_line (start 130.81 167.64) (end 125.73 161.29) (layer Edge.Cuts) (width 0.05))
+  (gr_circle (center 111.76 34.29) (end 118.11 31.75) (layer Edge.Cuts) (width 0.05))
+  (gr_line (start 81.28 158.75) (end 83.82 152.4) (layer Edge.Cuts) (width 0.05))
+  (gr_line (start 73.66 161.29) (end 81.28 158.75) (layer Edge.Cuts) (width 0.05))
+  (gr_line (start 73.66 165.1) (end 73.66 161.29) (layer Edge.Cuts) (width 0.05))
+  (gr_line (start 81.28 173.99) (end 73.66 165.1) (layer Edge.Cuts) (width 0.05))
+  (gr_line (start 124.46 172.72) (end 81.28 173.99) (layer Edge.Cuts) (width 0.05))
+  (gr_line (start 123.19 168.91) (end 124.46 172.72) (layer Edge.Cuts) (width 0.05))
+  (gr_line (start 121.92 152.4) (end 123.19 168.91) (layer Edge.Cuts) (width 0.05))
+  (gr_line (start 83.82 152.4) (end 121.92 152.4) (layer Edge.Cuts) (width 0.05))
+  (gr_circle (center 168.91 82.55) (end 171.45 81.28) (layer Edge.Cuts) (width 0.05))
   (gr_line (start 100.33 100.33) (end 177.8 177.8) (layer Dwgs.User) (width 0.15))
   (gr_line (start 100.33 100.33) (end 12.7 187.96) (layer Dwgs.User) (width 0.15))
@@
   (gr_line (start 100.33 100.33) (end 62.23 8.89) (layer Dwgs.User) (width 0.15))
   (gr_line (start 100.33 100.33) (end 33.02 33.02) (layer Dwgs.User) (width 0.15))
-  (gr_line (start 3.81 100.33) (end 207.01 100.33) (layer Dwgs.User) (width 0.15))
   (gr_line (start 100.33 5.08) (end 100.33 194.31) (layer Dwgs.User) (width 0.15))
   (gr_circle (center 100.33 100.33) (end 185.42 104.14) (layer Edge.Cuts) (width 0.05))

Commit message: pcb
Parts:
- added screwhoel1: screw_hole, custom:screwhole, F.Cu at (185.6, 220.5)
- added screwhoel1: screw_hole, custom:screwhole, F.Cu at (113.0, 178.5)
- added screwhoel1 (x2): screw_hole, custom:screwhole, F.Cu at (185.7, 52.8)
- added screwhoel1: screw_hole, custom:screwhole, F.Cu at (258.3, 178.5)
- added screwhoel1: screw_hole, custom:screwhole, F.Cu at (258.3, 94.6)
- added screwhoel1: screw_hole, custom:screwhole, F.Cu at (113.0, 94.6)
- moved ir_sensor_12 108.7 mm to (276.7, 174.1)
- moved ir_sensor_11 107.6 mm to (255.3, 206.2)
- moved ir_sensor_13 107.5 mm to (284.1, 136.7)
- moved Portmultiplexer1 107.2 mm to (150.4, 93.0)
- moved ir_sensor_14 104.6 mm to (276.6, 99.1)
- moved ir_sensor_10 104.0 mm to (223.4, 227.6)
- moved ir_sensor_9 100.0 mm to (185.7, 234.9)
- moved ir_sensor_15 99.7 mm to (255.3, 67.1)
- moved ir_sensor_8 94.3 mm to (147.8, 227.6)
- moved ir_sensor_16 94.0 mm to (223.5, 45.7)
- moved R2 92.8 mm to (228.9, 170.9)
- moved R4 92.8 mm to (228.9, 165.9)
- moved R5 92.8 mm to (228.9, 163.3)
- moved R6 92.8 mm to (228.9, 160.8)
- moved R7 92.8 mm to (228.9, 158.2)
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Routing:
- net Net-(Portmultiplexer1-Pad24): track 57.0 -> 391.2 mm
- net Net-(Portmultiplexer1-Pad25): track 106.1 -> 351.7 mm
- net Net-(Portmultiplexer1-Pad26): track 114.5 -> 309.4 mm
- net Net-(Portmultiplexer1-Pad27): track 121.9 -> 265.1 mm
- net gnd: track 1020.8 -> 1153.2 mm, vias 0 -> 5
- net Net-(Portmultiplexer1-Pad28): track 128.6 -> 218.5 mm
- net Net-(Portmultiplexer1-Pad21): track 76.6 -> 129.7 mm
- net 3.3v: track 821.4 -> 871.0 mm, vias 4 -> 3
- net Net-(Portmultiplexer1-Pad22): track 50.6 -> 93.0 mm
- net Net-(Portmultiplexer1-Pad3): track 236.4 -> 277.2 mm
- net Net-(Portmultiplexer1-Pad23): track 37.8 -> 74.4 mm
- net Net-(Portmultiplexer1-Pad5): track 155.1 -> 191.2 mm, vias 0 -> 1
- net Net-(Portmultiplexer1-Pad1): track 219.2 -> 187.2 mm, vias 0 -> 1
- net Net-(Portmultiplexer1-Pad7): track 121.0 -> 150.4 mm, vias 0 -> 1
- net sd6: track 71.8 -> 44.2 mm
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Other:
- board size 170.4 x 170.4 mm -> 200 x 200 mm

Commit message: i2c
Parts:
- added extrapins1: Conn_01x10_Female, custom:10connect, F.Cu at (245.7, 140.5)
- added pwr_sw1: SW_DIP_x01, custom:dipswitch1, F.Cu at (200.9, 89.4)
Connections:
- 3V3_converter1 pad 1: Net-(3V3_converter1-Pad1) -> 12V
- 3V3_converter1 pad 3: Net-(3V3_converter1-Pad3) -> gnd
- 5V_converter1 pad 1: Net-(3V3_converter1-Pad3) -> gnd
- 5V_converter1 pad 2: Net-(3V3_converter1-Pad1) -> 12V
- Portmultiplexer1 pad 12: sc6 -> scl
- Portmultiplexer1 pad 13: sd6 -> sda
- control_board1 pad 17: Net-(control_board1-Pad17) -> 25
- control_board1 pad 18: Net-(control_board1-Pad18) -> 26
- control_board1 pad 19: Net-(control_board1-Pad19) -> 27
- control_board1 pad 20: Net-(control_board1-Pad20) -> 28
- pcb_conn1 pad 5: sc6 -> Net-(pcb_conn1-Pad5)
- pcb_conn1 pad 6: sd6 -> Net-(pcb_conn1-Pad6)
- pcb_conn1 pad 7: Net-(pcb_conn1-Pad7) -> 12V
- screwhoel1 pad 1: (no net) -> gnd (x6)
- xt30 pad 1: Net-(3V3_converter1-Pad1) -> 12V
- xt30 pad 2: Net-(3V3_converter1-Pad3) -> gnd
- xt60 pad 1: Net-(3V3_converter1-Pad1) -> 12V
- xt60 pad 2: Net-(3V3_converter1-Pad3) -> gnd
Routing:
- net 12V: track 0.00 -> 216.0 mm, vias 0 -> 2
- net gnd: track 1153.2 -> 1320.9 mm
- net 3.3v: track 871.0 -> 1020.2 mm
- net 25: track 0.00 -> 134.5 mm, vias 0 -> 2
- net 28: track 0.00 -> 133.2 mm
- net 27: track 0.00 -> 131.4 mm, vias 0 -> 1
- net Net-(3V3_converter1-Pad1): track 126.2 -> 0.00 mm, vias 1 -> 0
- net 26: track 0.00 -> 122.2 mm, vias 0 -> 1
- net Net-(3V3_converter1-Pad3): track 118.6 -> 0.00 mm
- net scl: track 110.7 -> 228.5 mm, vias 1 -> 4
- net Net-(R7-Pad2): track 7.62 -> 107.1 mm, vias 0 -> 5
- net sda: track 104.6 -> 179.9 mm, vias 1 -> 2
- net sd6: track 44.2 -> 0.00 mm, vias 1 -> 0
- net Net-(3V3_converter1-Pad2): track 0.00 -> 43.0 mm, vias 0 -> 1
- net sc6: track 40.9 -> 0.00 mm, vias 1 -> 0
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Other:
- outline, holes or cut-outs redrawn

Commit message: 3d file pcb
Parts:
- removed the screwhoel1 at (185.6, 220.5)
- removed the screwhoel1 at (113.0, 178.5)
- removed the screwhoel1 at (185.7, 52.8) (x2)
- removed the screwhoel1 at (258.3, 178.5)
- removed the screwhoel1 at (258.3, 94.6)
- removed the screwhoel1 at (113.0, 94.6)
- added screwhoel1: screw_hole, custom:screwhole, F.Cu at (185.6, 219.1)
- added screwhoel1: screw_hole, custom:screwhole, F.Cu at (114.2, 177.8)
- added screwhoel1: screw_hole, custom:screwhole, F.Cu at (185.6, 54.1)
- added screwhoel1: screw_hole, custom:screwhole, F.Cu at (257.1, 95.3)
- added screwhoel1: screw_hole, custom:screwhole, F.Cu at (257.1, 177.8)
- added screwhoel1: screw_hole, custom:screwhole, F.Cu at (114.2, 95.3)
Routing:
- net gnd: track 1320.9 -> 1569.8 mm, vias 5 -> 7

Commit message: add_3d
Parts:
- moved xt60 11.2 mm to (237.7, 87.9)
- renumbered Portmultiplexer1 to mcpmc
Routing:
- net gnd: track 1569.8 -> 1598.7 mm
- net 12V: track 216.0 -> 236.0 mm
Other:
- outline, holes or cut-outs redrawn
