File: pcb_boven/pcb_boven.kicad_pcb (KiCad board)
At the start: 2 copper layers, 200 x 200 mm, 43 parts, among them U1 miniIMU-9_v6, U2 openMV_M7_R2

Commit message: dfas
Parts:
- moved ir_sensor_15 2.49 mm to (256.7, 69.1)
- moved R2 0.76 mm to (229.6, 170.9)
- moved R3 0.76 mm to (229.6, 168.4)
- moved R4 0.76 mm to (229.6, 165.9)
- moved R5 0.76 mm to (229.6, 163.3)
- moved R6 0.76 mm to (229.6, 160.8)
- moved R7 0.76 mm to (229.6, 158.2)
- moved ir_sensor_12 0.58 mm to (276.2, 174.1)
- moved ir_sensor_10 0.53 mm to (223.1, 227.1)
- moved ir_sensor_8 0.53 mm to (148.1, 227.1)
- moved ir_sensor_16 0.52 mm to (223.1, 46.0)
- moved ir_sensor_11 0.51 mm to (254.9, 205.9)
- moved R1 0.51 mm to (212.9, 177.3)
- moved ir_sensor_13 0.49 mm to (283.6, 136.6)
- moved ir_sensor_2 0.43 mm to (148.1, 46.0)
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Routing:
- net gnd: track 1598.7 -> 1661.0 mm, vias 7 -> 6
- net 3.3v: track 1020.2 -> 972.1 mm
- net Net-(Portmultiplexer1-Pad24): track 391.2 -> 373.0 mm
- net Net-(Portmultiplexer1-Pad3): track 277.2 -> 263.6 mm
- net Net-(Portmultiplexer1-Pad4): track 230.8 -> 224.3 mm
- net Net-(R7-Pad2): track 107.1 -> 112.7 mm
- net Net-(R6-Pad2): track 124.6 -> 130.1 mm, vias 0 -> 1
- net Net-(R5-Pad2): track 137.8 -> 143.4 mm
- net Net-(R4-Pad2): track 123.9 -> 129.5 mm
- net Net-(R3-Pad2): track 120.7 -> 126.2 mm
- net Net-(R2-Pad2): track 115.0 -> 120.6 mm, vias 0 -> 1
- net Net-(Portmultiplexer1-Pad25): track 351.7 -> 346.5 mm
- net Net-(Portmultiplexer1-Pad2): track 216.8 -> 214.3 mm
- net Net-(Portmultiplexer1-Pad26): track 309.4 -> 307.0 mm
- net Net-(Portmultiplexer1-Pad7): track 150.4 -> 148.0 mm
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Other:
- board size 200 x 200 mm -> 199.8 x 199.8 mm

Commit message: 4dip
Parts:
- removed R6, R7: R, custom:resistor
- removed dip_swith_instellinen1: SW_DIP_x06, custom:dipswitch6
- added SW1: SW_DIP_x04, custom:dipswitch4, F.Cu at (240.3, 167.3)
- renumbered mcpmc to Portmultiplexer1
Routing:
- net Net-(control_board1-Pad8): track 130.1 -> 0.00 mm, vias 1 -> 0
- net Net-(control_board1-Pad9): track 112.7 -> 1.84 mm, vias 5 -> 0
- net Net-(SW1-Pad1): track 105.7 -> 118.8 mm
- net Net-(R2-Pad2): track 120.6 -> 127.5 mm
- net gnd: track 1661.0 -> 1657.1 mm
- net Net-(R5-Pad2): track 143.4 -> 142.3 mm
- net Net-(R4-Pad2): track 129.5 -> 128.6 mm
- net Net-(R3-Pad2): track 126.2 -> 125.5 mm

Commit message: code
Connections:
- control_board1 pad 12: Net-(U2-Pad5) -> Net-(control_board1-Pad12)
- control_board1 pad 13: Net-(U2-Pad2) -> Net-(control_board1-Pad13)
- control_board1 pad 14: Net-(U2-Pad3) -> Net-(control_board1-Pad14)
- control_board1 pad 2: Net-(control_board1-Pad2) -> Net-(U2-Pad6)
- control_board1 pad 28: Net-(U2-Pad4) -> Net-(control_board1-Pad28)
- control_board1 pad 3: Net-(control_board1-Pad3) -> Net-(U2-Pad7)
Routing:
- net Net-(U2-Pad6): track 0.00 -> 46.0 mm, vias 0 -> 1
- net Net-(U2-Pad7): track 0.00 -> 42.9 mm, vias 0 -> 1
- net Net-(U2-Pad5): track 33.6 -> 0.00 mm
- net Net-(U2-Pad2): track 27.8 -> 0.00 mm
- net Net-(U2-Pad3): track 27.8 -> 0.00 mm
- net 26: track 122.2 -> 124.4 mm
