File: pcb_boven/pcb_boven_backup.kicad_pcb (KiCad board)
At the start: 2 copper layers, 170.4 x 170.4 mm, 35 parts, among them U1 miniIMU-9_v6, U2 openMV_M7_R2

Commit message: dfas
Parts:
- added extrapins1: Conn_01x10_Female, custom:10connect, F.Cu at (245.7, 140.5)
- added pwr_sw1: SW_DIP_x01, custom:dipswitch1, F.Cu at (200.9, 89.4)
- added screwhoel1: screw_hole, custom:screwhole, F.Cu at (185.6, 219.1)
- added screwhoel1: screw_hole, custom:screwhole, F.Cu at (114.2, 177.8)
- added screwhoel1: screw_hole, custom:screwhole, F.Cu at (185.6, 54.1)
- added screwhoel1: screw_hole, custom:screwhole, F.Cu at (257.1, 95.3)
- added screwhoel1: screw_hole, custom:screwhole, F.Cu at (257.1, 177.8)
- added screwhoel1: screw_hole, custom:screwhole, F.Cu at (114.2, 95.3)
- moved ir_sensor_12 108.7 mm to (276.7, 174.1)
- moved ir_sensor_11 107.6 mm to (255.3, 206.2)
- moved ir_sensor_13 107.5 mm to (284.1, 136.7)
- moved mcpmc 107.2 mm to (150.4, 93.0)
- moved ir_sensor_14 104.6 mm to (276.6, 99.1)
- moved ir_sensor_10 104.0 mm to (223.4, 227.6)
- moved ir_sensor_9 100.0 mm to (185.7, 234.9)
- moved ir_sensor_15 99.7 mm to (255.3, 67.1)
- moved xt60 98.7 mm to (237.7, 87.9)
- moved ir_sensor_8 94.3 mm to (147.8, 227.6)
- moved ir_sensor_16 94.0 mm to (223.5, 45.7)
- moved R2 92.8 mm to (228.9, 170.9)
- moved R4 92.8 mm to (228.9, 165.9)
- moved R5 92.8 mm to (228.9, 163.3)
- moved R6 92.8 mm to (228.9, 160.8)
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- renumbered Portmultiplexer1 to mcpmc
Connections:
- 3V3_converter1 pad 1: Net-(3V3_converter1-Pad1) -> 12V
- 3V3_converter1 pad 3: Net-(3V3_converter1-Pad3) -> gnd
- 5V_converter1 pad 1: Net-(3V3_converter1-Pad3) -> gnd
- 5V_converter1 pad 2: Net-(3V3_converter1-Pad1) -> 12V
- control_board1 pad 17: Net-(control_board1-Pad17) -> 25
- control_board1 pad 18: Net-(control_board1-Pad18) -> 26
- control_board1 pad 19: Net-(control_board1-Pad19) -> 27
- control_board1 pad 20: Net-(control_board1-Pad20) -> 28
- mcpmc pad 12: sc6 -> scl
- mcpmc pad 13: sd6 -> sda
- pcb_conn1 pad 5: sc6 -> Net-(pcb_conn1-Pad5)
- pcb_conn1 pad 6: sd6 -> Net-(pcb_conn1-Pad6)
- pcb_conn1 pad 7: Net-(pcb_conn1-Pad7) -> 12V
- xt30 pad 1: Net-(3V3_converter1-Pad1) -> 12V
- xt30 pad 2: Net-(3V3_converter1-Pad3) -> gnd
- xt60 pad 1: Net-(3V3_converter1-Pad1) -> 12V
- xt60 pad 2: Net-(3V3_converter1-Pad3) -> gnd
Routing:
- net gnd: track 1020.8 -> 1598.7 mm, vias 0 -> 7
- net Net-(Portmultiplexer1-Pad24): track 57.0 -> 391.2 mm
- net Net-(Portmultiplexer1-Pad25): track 106.1 -> 351.7 mm
- net 12V: track 0.00 -> 236.0 mm, vias 0 -> 2
- net 3.3v: track 821.4 -> 1020.2 mm, vias 4 -> 3
- net Net-(Portmultiplexer1-Pad26): track 114.5 -> 309.4 mm
- net Net-(Portmultiplexer1-Pad27): track 121.9 -> 265.1 mm
- net 25: track 0.00 -> 134.5 mm, vias 0 -> 2
- net 28: track 0.00 -> 133.2 mm
- net 27: track 0.00 -> 131.4 mm, vias 0 -> 1
- net Net-(3V3_converter1-Pad1): track 126.0 -> 0.00 mm
- net 26: track 0.00 -> 122.2 mm, vias 0 -> 1
- net scl: track 110.7 -> 228.5 mm, vias 1 -> 4
- net Net-(3V3_converter1-Pad3): track 109.3 -> 0.00 mm
- net Net-(R7-Pad2): track 7.62 -> 107.1 mm, vias 0 -> 5
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Other:
- board size 170.4 x 170.4 mm -> 200 x 200 mm
