File: PCBs/midden/midden.kicad_sch (KiCad schematic)
At the start: 25 parts, among them J1 Conn_01x14_Pin, J2 Conn_01x14_Pin, J3 Conn_01x04_Pin, SW1 SW_SPDT_312

Commit message: PCB
Parts:
- added F1: Fuse, symbol Device:Fuse
Connections:
- net at 3V3_conv1.3 (VIN), 5V_conv1.3 (VIN), DR1.1 (VIN)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: now also F1.1; no longer D5.1 (K)
- new net: D5.1 (K), F1.2
Changed lines of the file:
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@@
-	)
-	(junction
-		(at 33.02 82.55)
-		(diameter 0)
-		(color 0 0 0 0)
 	)
 	(junction
@@
 	)
 	(junction
+		(at 33.02 71.12)
+		(diameter 0)
+		(color 0 0 0 0)
+	)
+	(junction
 		(at 121.92 149.86)
 		(diameter 0)
@@
 	(wire
 		(pts
-			(xy 50.8 82.55) (xy 50.8 105.41)
+			(xy 50.8 71.12) (xy 50.8 105.41)
 		)
 		(stroke
@@
 	(wire
 		(pts
-			(xy 33.02 82.55) (xy 50.8 82.55)
+			(xy 33.02 71.12) (xy 50.8 71.12)
 		)
 		(stroke
@@
 	(wire
 		(pts
-			(xy 33.02 45.72) (xy 33.02 82.55)
+			(xy 33.02 45.72) (xy 33.02 71.12)
 		)
 		(stroke
@@
 		(pts
 			(xy 223.52 80.01) (xy 255.27 80.01)
+		)
+		(stroke
+			(width 0)
+			(type default)
+		)
+	)
+	(wire
+		(pts
+			(xy 33.02 71.12) (xy 33.02 74.93)
 		)
 		(stroke
@@
 					(unit 1)
 				)
+			)
+		)
+	)
+	(symbol
+		(lib_id "Device:Fuse")
+		(at 33.02 78.74 0)
+		(unit 1)
+		(exclude_from_sim no)
+		(in_bom yes)
+		(on_board yes)
+		(dnp no)
+		(fields_autoplaced yes)
+		(property "Reference" "F1"
+			(at 35.56 77.4699 0)
+			(effects
+				(font
+					(size 1.27 1.27)
+				)
+				(justify left)
+			)
+		)
+		(property "Value" "Fuse"
+			(at 35.56 80.0099 0)
+			(effects
+				(font
+					(size 1.27 1.27)
+				)
+				(justify left)
+			)
+		)
+		(property "Footprint" ""
+			(at 31.242 78.74 90)
+			(effects
+				(font
+					(size 1.27 1.27)
+				)
+				(hide yes)
+			)
+		)
+		(property "Datasheet" "~"
+			(at 33.02 78.74 0)
+			(effects
+				(font
+					(size 1.27 1.27)
+				)
+				(hide yes)
+			)
+		)
+		(property "Description" "Fuse"
+			(at 33.02 78.74 0)
+			(effects
+				(font
+					(size 1.27 1.27)
+				)
+				(hide yes)
+			)
+		)
+		(pin "1"
+		)
+		(pin "2"
+		)
+		(instances
+			(project ""
+				(path "/1db6a830-bef0-4b5d-9df3-c3637fd891d4"
+					(reference "F1")
+					(unit 1)
+				)

Commit message: dfg
Parts:
- added xt60: Battery, Connector_AMASS:AMASS_XT60-F_1x02_P7.20mm_Vertical, symbol Device:Battery
- 3V3_conv1, 5V_conv1: footprint (none) -> cust_footpr:pololu_power_converter
- DR1, DR2, DR3: footprint (none) -> cust_footpr:TB9051FTG
- F1: footprint (none) -> Fuse:Fuseholder_TR5_Littelfuse_No560_No460
- Jst1: renamed from J1; footprint (none) -> Connector_JST:JST_EH_B14B-EH-A_1x14_P2.50mm_Vertical
- M1, M2, M3: footprint (none) -> cust_footpr:pololu_4.41 Metal Gearmotor 25Dx63L mm MP 12V with 48 CPR Encoder
- grove1: renamed from J3; footprint (none) -> Connector:NS-Tech_Grove_1x04_P2mm_Vertical
- jst2: renamed from J2; footprint (none) -> Connector_JST:JST_EH_S14B-EH_1x14_P2.50mm_Horizontal
- teensy1: renamed from teensy; footprint (none) -> cust_footpr:TEENSY41
- xt30: renamed from BT1; footprint (none) -> Connector_AMASS:AMASS_XT30U-M_1x02_P5.0mm_Vertical
- renumbered solenoid to solenoid1
Connections:
- net at D6.1 (K): now also xt30.1 (+), xt60.1 (+); no longer xt30.2 (-)
- net at D10.1 (K), D6.2 (A), D7.1 (K)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: now also DR1.0 (screw), DR2.0 (screw), DR3.0 (screw); no longer D2.1 (K), D8.2 (A)
- net at DR1.1 (VIN), DR2.1 (VIN), DR3.1 (VIN)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: now also D8.2 (A); no longer 3V3_conv1.3 (VIN), 5V_conv1.3 (VIN)
- net at 3V3_conv1.4 (GND), 3V3_conv1.5 (GND), D7.2 (A): now also 5V_conv1.4 (GND), 5V_conv1.5 (GND), D2.1 (K)
- net at D5.2 (A): now also xt30.2 (-), xt60.2 (-); no longer xt30.1 (+)
- new net: 3V3_conv1.3 (VIN), 5V_conv1.3 (VIN), D8.1 (K)
Other:
- moved on the sheet: xt30
