File: PCB/aparte_pcb/midden/_autosave-midden.kicad_sch (KiCad schematic)
At the start: 31 parts, among them J1 Conn_01x13_Socket, J2 Conn_01x13_Socket

Commit message: alleen solinoid nog
Parts:
- added SW1: SW_Reed_SPDT, Connector_PinHeader_1.27mm:PinHeader_1x03_P1.27mm_Vertical, symbol Switch:SW_Reed_SPDT
Connections:
- net groundd: now also SW1.1
- net at teensy1.44 (22_A8_CTX1): now also SW1.2
Changed lines of the file:
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@@
 	)
 	(junction
+		(at 259.08 74.93)
+		(diameter 0)
+		(color 0 0 0 0)
+	)
+	(junction
 		(at 199.39 20.32)
 		(diameter 0)
@@
 	(wire
 		(pts
+			(xy 243.84 77.47) (xy 237.49 77.47)
+		)
+		(stroke
+			(width 0)
+			(type default)
+		)
+	)
+	(wire
+		(pts
 			(xy 63.5 80.01) (xy 63.5 113.03)
 		)
@@
 	(wire
 		(pts
-			(xy 259.08 69.85) (xy 259.08 133.35)
+			(xy 259.08 69.85) (xy 259.08 74.93)
 		)
 		(stroke
@@
 	(wire
 		(pts
+			(xy 256.54 74.93) (xy 259.08 74.93)
+		)
+		(stroke
+			(width 0)
+			(type default)
+		)
+	)
+	(wire
+		(pts
 			(xy 45.72 76.2) (xy 45.72 110.49)
 		)
@@
 	(wire
 		(pts
+			(xy 259.08 74.93) (xy 259.08 133.35)
+		)
+		(stroke
+			(width 0)
+			(type default)
+		)
+	)
+	(wire
+		(pts
 			(xy 127 52.07) (xy 127 53.34)
 		)
@@
 					(unit 1)
 				)
+			)
+		)
+	)
+	(symbol
+		(lib_id "Switch:SW_Reed_SPDT")
+		(at 248.92 77.47 0)
+		(unit 1)
+		(exclude_from_sim no)
+		(in_bom yes)
+		(on_board yes)
+		(dnp no)
+		(fields_autoplaced yes)
+		(property "Reference" "SW1"
+			(at 249.6215 69.85 0)
+			(effects
+				(font
+					(size 1.27 1.27)
+				)
+				(hide yes)
+			)
+		)
+		(property "Value" "SW_Reed_SPDT"
+			(at 249.6215 72.39 0)
+			(effects
+				(font
+					(size 1.27 1.27)
+				)
+				(hide yes)
+			)
+		)
+		(property "Footprint" "Connector_PinHeader_1.27mm:PinHeader_1x03_P1.27mm_Vertical"
+			(at 248.92 77.47 0)
+			(effects
+				(font
+					(size 1.27 1.27)
+				)
+				(hide yes)
+			)
+		)
+		(property "Datasheet" "~"
+			(at 248.92 77.47 0)
+			(effects
+				(font
+					(size 1.27 1.27)
+				)
+				(hide yes)
+			)
+		)
+		(property "Description" "SPDT reed switch"
+			(at 248.92 77.47 0)
+			(effects
+				(font
+					(size 1.27 1.27)
+				)
+				(hide yes)
+			)
+		)
+		(pin "3"
+		)
+		(pin "1"
+		)
+		(pin "2"
+		)
+		(instances
+			(project ""
+				(path "/e189b955-7e7c-46c1-a031-b30377455d70"
+					(reference "SW1")
+					(unit 1)
+				)
