File: PCB/aparte_pcb/midden/midden.kicad_pcb (KiCad board)
At the start: 2 copper layers, 211 x 207.2 mm, 30 parts, among them J1 Conn_01x13_Socket, J2 Conn_01x13_Socket

Commit message: midden bijna klaar
Parts:
- moved D16 113.8 mm to (162.8, 193.8), turned to -90 degrees
- moved D15 104.7 mm to (169.8, 193.8), turned to 90 degrees
- moved J2 77.9 mm to (224.5, 183.2), turned to 180 degrees
- moved J1 74.2 mm to (189.0, 182.7), turned to 180 degrees
- moved D11 63.5 mm to (204.2, 195.2)
- moved D10 62.8 mm to (210.5, 195.2)
- moved D12 60.1 mm to (198.0, 195.2)
- moved D13 51.4 mm to (220.8, 156.5), turned to -90 degrees
- moved teensy1 43.0 mm to (205.4, 133.4), turned to 180 degrees
- moved D14 27.9 mm to (206.8, 170.0)
- moved D4 18.0 mm to (153.2, 211.2)
- moved D5 16.7 mm to (144.2, 211.0)
Routing:
- net Net-(D12-A): track 41.7 -> 465.5 mm, vias 0 -> 2
- net groundd: track 20.1 -> 347.5 mm
- net Net-(D11-A): track 0.00 -> 263.6 mm
- net Net-(D4-A): track 0.00 -> 250.9 mm
- net Net-(M1-A_out): track 42.6 -> 264.8 mm, vias 0 -> 2
- net Net-(M1-B_out): track 40.9 -> 256.0 mm
- net Net-(M2-B_out): track 25.2 -> 236.5 mm, vias 0 -> 2
- net Net-(M2-A_out): track 27.5 -> 238.7 mm, vias 0 -> 2
- net Net-(M3-B_out): track 8.19 -> 207.6 mm
- net Net-(M3-A_out): track 10.6 -> 208.3 mm
- net Net-(DR3-PWM1): track 0.00 -> 170.1 mm, vias 0 -> 2
- net Net-(DR3-PWM2): track 0.00 -> 169.1 mm, vias 0 -> 2
- net Net-(DR3-ENB): track 0.00 -> 167.6 mm, vias 0 -> 2
- net Net-(DR3-EN): track 0.00 -> 166.4 mm, vias 0 -> 2
- net Net-(DR2-PWM1): track 0.00 -> 134.5 mm
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
Commit message: alleen solinoid nog
Parts:
- added SW1: SW_Reed_SPDT, Connector_PinHeader_1.27mm:PinHeader_1x03_P1.27mm_Vertical, F.Cu at (214.0, 159.0)
Connections:
- teensy1 pad 44: unconnected-(teensy1-22_A8_CTX1-Pad44) -> Net-(teensy1-22_A8_CTX1)
Routing:
- net Net-(D4-A): track 250.9 -> 348.6 mm, vias 0 -> 2
- net Net-(D2-A): track 255.6 -> 349.4 mm, vias 0 -> 1
- net Net-(teensy1-22_A8_CTX1): track 0.00 -> 23.1 mm
- net groundd: track 347.5 -> 364.3 mm
- net Net-(M1-A_out): track 264.8 -> 263.4 mm
Other:
- outline, holes or cut-outs redrawn
- board text removed: "kicker"

Commit message: pxb
Parts:
- removed J2: Conn_01x13_Socket, Connector_JST:JST_PH_S15B-PH-K_1x15_P2.00mm_Horizontal
- added D17: D, Diode_SMD:D_MELF-RM10_Universal_Handsoldering, F.Cu at (139.0, 194.0)
- added D18: D, Diode_SMD:D_MELF-RM10_Universal_Handsoldering, F.Cu at (123.0, 193.8)
- added J4: Conn_01x10_Socket, Connector_JST:JST_EH_S10B-EH_1x10_P2.50mm_Horizontal, F.Cu at (188.0, 175.0)
- added J5: Conn_01x04_Socket, Connector_JST:JST_EH_S4B-EH_1x04_P2.50mm_Horizontal, F.Cu at (154.5, 190.5)
- added SW2: SW_DIP_x01, dpdsd:R1966ABLKBLKEF, F.Cu at (200.0, 98.9)
- added U1: ~, Library:miniIMU, F.Cu at (130.0, 184.1)
- J1: value Conn_01x13_Socket -> Conn_01x10_Socket; footprint Connector_JST:JST_PH_S15B-PH-K_1x15_P2.00mm_Horizontal -> Connector_JST:JST_EH_S10B-EH_1x10_P2.50mm_Horizontal
- moved J1 33.9 mm to (222.8, 179.8)
- moved D16 9.95 mm to (167.0, 184.8), turned to 0 degrees
- moved D15 5.15 mm to (167.8, 189.0), turned to 180 degrees
Connections:
- F1 pad 2: Net-(D1-K) -> Net-(F1-Pad2)
- J1 pad 1: pr1 -> soft_power_sw
- J1 pad 10: GROEN -> 5v
- J1 pad 2: pr2 -> rx3
- J1 pad 3: pr3 -> tx3
- J1 pad 4: pr4 -> rx2
- J1 pad 5: pr5 -> tx2
- J1 pad 6: pr6 -> rx1
- J1 pad 7: pr7 -> tx1
- J1 pad 8: pr8 -> gnd
- J1 pad 9: ROOD -> 3v3
- teensy1 pad 40: unconnected-(teensy1-18_A4_SDA-Pad40) -> Net-(U1-sda)
- teensy1 pad 41: unconnected-(teensy1-19_A5_SCL-Pad41) -> Net-(U1-scl)
Routing:
- net Net-(U1-sda): track 0.00 -> 176.0 mm
- net Net-(U1-scl): track 0.00 -> 168.5 mm
- net groundd: track 364.3 -> 439.8 mm, vias 0 -> 1
- net Net-(D12-A): track 465.1 -> 514.4 mm, vias 2 -> 3
- net BLAUW: track 78.3 -> 114.2 mm, vias 1 -> 2
- net Net-(F1-Pad2): track 0.00 -> 20.8 mm
- net Net-(D1-K): track 7.12 -> 16.2 mm
- net Net-(D17-K): track 0.00 -> 7.96 mm
- net Net-(D18-A): track 0.00 -> 7.94 mm
- net pr1: track 46.9 -> 39.6 mm
- net pr2: track 45.6 -> 38.6 mm
- net pr3: track 45.4 -> 38.5 mm
- net pr4: track 45.2 -> 38.5 mm
- net pr5: track 45.0 -> 38.5 mm
- net pr6: track 44.8 -> 38.5 mm
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
Commit message: kicker
Parts:
- added C1: C, Capacitor_THT:CP_Radial_D8.0mm_P3.50mm, F.Cu at (162.1, 218.0)
- added K1: G5Q-1A, Relay_THT:Relay_SPST_Omron-G5Q-1A, F.Cu at (178.4, 214.6)
- added solenoid1: Re, TerminalBlock_Altech:Altech_AK100_1x02_P5.00mm, F.Cu at (153.9, 226.2)
Connections:
- D4 pad 1: unconnected-(D4-K-Pad1) -> Net-(D4-K)
- D5 pad 2: unconnected-(D5-A-Pad2) -> Net-(D5-A)
- teensy1 pad 39: unconnected-(teensy1-17_A3_TX4_SDA1-Pad39) -> Net-(teensy1-17_A3_TX4_SDA1)
- teensy1 pad 42: unconnected-(teensy1-20_A6_TX5_LRCLK1-Pad42) -> Net-(teensy1-20_A6_TX5_LRCLK1)
Routing:
- net Net-(teensy1-17_A3_TX4_SDA1): track 0.00 -> 164.7 mm, vias 0 -> 1
- net Net-(teensy1-20_A6_TX5_LRCLK1): track 0.00 -> 157.9 mm, vias 0 -> 1
- net Net-(solenoid1-+): track 0.00 -> 25.1 mm
- net Net-(C1-Pad2): track 0.00 -> 19.7 mm
- net Net-(D5-A): track 0.00 -> 12.1 mm
- net Net-(D4-K): track 0.00 -> 9.57 mm
- net Net-(U1-sda): track 176.0 -> 178.4 mm
- net Net-(U1-scl): track 168.5 -> 170.1 mm
