File: PCB/aparte_pcb/onder/onder.kicad_sch (KiCad schematic)
At the start: 73 parts, among them J1 Conn_01x13_Socket, Q1 NPN, Q2 NPN, Q3 NPN

Commit message: pxb
Parts:
- D1, D10, D11, D12, D2, D3, D4, D5, D6, D7, D8, D9: footprint (none) -> LED_SMD:LED_RGB_5050-6
Changed lines of the file:
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@@
 			)
 		)
-		(property "Footprint" ""
+		(property "Footprint" "LED_SMD:LED_RGB_5050-6"
 			(at 62.23 66.04 0)
 			(effects
@@
 			)
 		)
-		(property "Footprint" ""
+		(property "Footprint" "LED_SMD:LED_RGB_5050-6"
 			(at 43.18 66.04 0)
 			(effects
@@
 			)
 		)
-		(property "Footprint" ""
+		(property "Footprint" "LED_SMD:LED_RGB_5050-6"
 			(at 119.38 66.04 0)
 			(effects
@@
 			)
 		)
-		(property "Footprint" ""
+		(property "Footprint" "LED_SMD:LED_RGB_5050-6"
 			(at 138.43 66.04 0)
 			(effects
@@
 			)
 		)
-		(property "Footprint" ""
+		(property "Footprint" "LED_SMD:LED_RGB_5050-6"
 			(at 81.28 66.04 0)
 			(effects
@@
 			)
 		)
-		(property "Footprint" ""
+		(property "Footprint" "LED_SMD:LED_RGB_5050-6"
 			(at 176.53 66.04 0)
 			(effects
@@
 			)
 		)
-		(property "Footprint" ""
+		(property "Footprint" "LED_SMD:LED_RGB_5050-6"
 			(at 157.48 66.04 0)
 			(effects
@@
 			)
 		)
-		(property "Footprint" ""
+		(property "Footprint" "LED_SMD:LED_RGB_5050-6"
 			(at 24.13 66.04 0)
 			(effects
@@
 			)
 		)
-		(property "Footprint" ""
+		(property "Footprint" "LED_SMD:LED_RGB_5050-6"
 			(at 214.63 66.04 0)
 			(effects
@@
 			)
 		)
-		(property "Footprint" ""
+		(property "Footprint" "LED_SMD:LED_RGB_5050-6"
 			(at 100.33 66.04 0)
 			(effects
@@
 			)
 		)
-		(property "Footprint" ""
+		(property "Footprint" "LED_SMD:LED_RGB_5050-6"
 			(at 233.68 66.04 0)
 			(effects
@@
 			)
 		)
-		(property "Footprint" ""
+		(property "Footprint" "LED_SMD:LED_RGB_5050-6"
 			(at 195.58 66.04 0)
 			(effects

Commit message: \x
Connections:
- net at 220Ω_1.2, 220Ω_10.2, 220Ω_13.2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: no longer Q3.1 (C)
- net at 220Ω_11.2, 220Ω_14.2, 220Ω_17.2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: no longer Q2.1 (C)
- net at D14.1 (K), PR1.1, PR2.1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: now also Q2.1 (C), Q3.1 (C)
Changed lines of the file:
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@@
+	)
+	(junction
+		(at 196.85 121.92)
+		(diameter 0)
+		(color 0 0 0 0)
 	)
 	(junction
@@
 	)
 	(junction
+		(at 212.09 121.92)
+		(diameter 0)
+		(color 0 0 0 0)
+	)
+	(junction
 		(at 58.42 81.28)
 		(diameter 0)
@@
 	)
 	(junction
-		(at 234.95 82.55)
-		(diameter 0)
-		(color 0 0 0 0)
-	)
-	(junction
 		(at 186.69 82.55)
 		(diameter 0)
@@
 	)
 	(junction
-		(at 229.87 81.28)
-		(diameter 0)
-		(color 0 0 0 0)
-	)
-	(junction
 		(at 163.83 83.82)
 		(diameter 0)
@@
 	(wire
 		(pts
-			(xy 182.88 121.92) (xy 247.65 121.92)
+			(xy 182.88 121.92) (xy 196.85 121.92)
 		)
 		(stroke
@@
 	(wire
 		(pts
+			(xy 212.09 121.92) (xy 247.65 121.92)
+		)
+		(stroke
+			(width 0)
+			(type default)
+		)
+	)
+	(wire
+		(pts
 			(xy 110.49 129.54) (xy 266.7 129.54)
 		)
@@
 	(wire
 		(pts
-			(xy 196.85 113.03) (xy 234.95 113.03)
-		)
-		(stroke
-			(width 0)
-			(type default)
-		)
-	)
-	(wire
-		(pts
 			(xy 153.67 81.28) (xy 153.67 78.74)
 		)
@@
 	(wire
 		(pts
-			(xy 229.87 109.22) (xy 212.09 109.22)
-		)
-		(stroke
-			(width 0)
-			(type default)
-		)
-	)
-	(wire
-		(pts
 			(xy 186.69 82.55) (xy 196.85 82.55)
 		)
@@
 	(wire
 		(pts
-			(xy 196.85 109.22) (xy 196.85 113.03)
+			(xy 196.85 109.22) (xy 196.85 121.92)
 		)
 		(stroke
@@
 	(wire
 		(pts
-			(xy 234.95 113.03) (xy 234.95 82.55)
-		)
-		(stroke
-			(width 0)
-			(type default)
-		)
-	)
-	(wire
-		(pts
 			(xy 55.88 121.92) (xy 71.12 121.92)
 		)
@@
 	(wire
 		(pts
+			(xy 212.09 109.22) (xy 212.09 121.92)
+		)
+		(stroke
+			(width 0)
+			(type default)
+		)
+	)
+	(wire
+		(pts
 			(xy 158.75 82.55) (xy 139.7 82.55)
 		)
@@
 	(wire
 		(pts
+			(xy 196.85 121.92) (xy 212.09 121.92)
+		)
+		(stroke
+			(width 0)
+			(type default)
+		)
+	)
+	(wire
+		(pts
 			(xy 269.24 50.8) (xy 278.13 50.8)
 		)
@@
 		)
 		(stroke
-			(width 0)
-			(type default)
-		)
-	)
-	(wire
-		(pts
-			(xy 229.87 81.28) (xy 229.87 109.22)
-		)
-		(stroke
