File: PCB/aparte_pcb/onder/onder.kicad_sch (KiCad schematic)
At the start: 73 parts, among them J1 Conn_01x13_Socket, Q1 NPN, Q2 NPN, Q3 NPN

Commit message: Add files via upload
Parts:
- removed J1: Conn_01x13_Socket, symbol Connector:Conn_01x13_Socket
- added J1: Conn_01x04_Socket, Connector_JST:JST_EH_S4B-EH_1x04_P2.50mm_Horizontal, symbol Connector:Conn_01x04_Socket
- added J2: Conn_01x10_Socket, Connector_JST:JST_EH_S10B-EH_1x10_P2.50mm_Horizontal, symbol Connector:Conn_01x10_Socket
- PR1, PR2, PR3, PR4, PR5, PR6, PR7, PR8: footprint Library:FOTORES -> Library:FOTORESist
- Q1, Q2, Q3: footprint (none) -> Library:NPN
Connections:
- net 5V: now also J2.1 (Pin_1)
- net BLAUW: now also J2.3 (Pin_3)
- net GND: now also J2.2 (Pin_2)
- net GROEN: now also J2.4 (Pin_4)
- net ROOD: now also J2.5 (Pin_5)
- net pr1: now also J1.3 (Pin_3)
- net pr2: now also J1.2 (Pin_2)
- net pr3: now also J1.1 (Pin_1)
- net pr4: now also J2.10 (Pin_10)
- net pr5: now also J2.9 (Pin_9)
- net pr6: now also J2.8 (Pin_8)
- net pr7: now also J2.7 (Pin_7)
- net pr8: now also J2.6 (Pin_6)
- net at 220Ω_1.2, 220Ω_10.2, 220Ω_13.2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: no longer Q3.1 (C)
- net at 220Ω_11.2, 220Ω_14.2, 220Ω_17.2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: no longer Q2.1 (C)
- net at D14.1 (K), PR1.1, PR2.1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: now also Q2.1 (C), Q3.1 (C)
Changed lines of the file:
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@@
 	)
 	(junction
+		(at 212.09 121.92)
+		(diameter 0)
+		(color 0 0 0 0)
+	)
+	(junction
 		(at 125.73 60.96)
 		(diameter 0)
@@
 	)
 	(junction
-		(at 234.95 82.55)
-		(diameter 0)
-		(color 0 0 0 0)
-	)
-	(junction
 		(at 186.69 82.55)
 		(diameter 0)
@@
 	)
 	(junction
+		(at 196.85 121.92)
+		(diameter 0)
+		(color 0 0 0 0)
+	)
+	(junction
 		(at 63.5 82.55)
 		(diameter 0)
@@
 	)
 	(junction
-		(at 229.87 81.28)
-		(diameter 0)
-		(color 0 0 0 0)
-	)
-	(junction
 		(at 163.83 83.82)
 		(diameter 0)
@@
 	(wire
 		(pts
-			(xy 182.88 121.92) (xy 247.65 121.92)
+			(xy 182.88 121.92) (xy 196.85 121.92)
 		)
 		(stroke
@@
 	(wire
 		(pts
-			(xy 63.5 82.55) (xy 44.45 82.55)
+			(xy 196.85 121.92) (xy 212.09 121.92)
 		)
 		(stroke
@@
 	(wire
 		(pts
-			(xy 196.85 113.03) (xy 234.95 113.03)
+			(xy 63.5 82.55) (xy 44.45 82.55)
 		)
 		(stroke
@@
 	(wire
 		(pts
-			(xy 229.87 109.22) (xy 212.09 109.22)
-		)
-		(stroke
-			(width 0)
-			(type default)
-		)
-	)
-	(wire
-		(pts
 			(xy 186.69 82.55) (xy 196.85 82.55)
 		)
@@
 	(wire
 		(pts
-			(xy 196.85 109.22) (xy 196.85 113.03)
+			(xy 196.85 109.22) (xy 196.85 121.92)
 		)
 		(stroke
@@
 	(wire
 		(pts
-			(xy 234.95 113.03) (xy 234.95 82.55)
+			(xy 212.09 121.92) (xy 247.65 121.92)
 		)
 		(stroke
@@
 	(wire
 		(pts
-			(xy 260.35 33.02) (xy 260.35 86.36)
+			(xy 212.09 109.22) (xy 212.09 121.92)
 		)
 		(stroke
@@
 	(wire
 		(pts
-			(xy 95.25 113.03) (xy 95.25 130.81)
+			(xy 260.35 33.02) (xy 260.35 86.36)
 		)
 		(stroke
@@
 	(wire
 		(pts
-			(xy 229.87 81.28) (xy 229.87 109.22)
+			(xy 95.25 113.03) (xy 95.25 130.81)
 		)
 		(stroke
@@
 			)
 		)
-		(property "Footprint" "Library:FOTORES"
+		(property "Footprint" "Library:FOTORESist"
 			(at 44.45 108.585 90)
 			(effects
@@
 			)
 		)
-		(property "Footprint" "Library:FOTORES"
+		(property "Footprint" "Library:FOTORESist"
 			(at 120.65 108.585 90)
 			(effects
@@
 			)
 		)
-		(property "Footprint" "Library:FOTORES"
+		(property "Footprint" "Library:FOTORESist"
 			(at 106.68 108.585 90)
 			(effects
@@
 			)
 		)
-		(property "Footprint" "Library:FOTORES"
+		(property "Footprint" "Library:FOTORESist"
 			(at 137.16 108.585 90)
 			(effects
@@
 	)
 	(symbol
+		(lib_id "Connector:Conn_01x10_Socket")
+		(at 283.21 38.1 0)
+		(unit 1)
+		(exclude_from_sim no)
+		(in_bom yes)
+		(on_board yes)
+		(dnp no)
+		(fields_autoplaced yes)
+		(property "Reference" "J2"
+			(at 284.48 38.0999 0)
+			(effects
+				(font
+					(size 1.27 1.27)
+				)
+				(justify left)
+			)
+		)
+		(property "Value" "Conn_01x10_Socket"
+			(at 284.48 40.6399 0)
+			(effects
+				(font
+					(size 1.27 1.27)
+				)
+				(justify left)
+			)
+		)
+		(property "Footprint" "Connector_JST:JST_EH_S10B-EH_1x10_P2.50mm_Horizontal"
+			(at 283.21 38.1 0)
+			(effects
+				(font
+					(size 1.27 1.27)
+				)
+				(hide yes)
+			)
+		)
+		(property "Datasheet" "~"
+			(at 283.21 38.1 0)
+			(effects
+				(font
+					(size 1.27 1.27)
+				)
+				(hide yes)
+			)
+		)
+		(property "Description" "Generic connector, single row, 01x10, script generated"
+			(at 283.21 38.1 0)
+			(effects
+				(font
+					(size 1.27 1.27)
+				)
+				(hide yes)
+			)
+		)
+		(pin "10"
+		)
+		(pin "9"
+		)
+		(pin "6"
+		)
+		(pin "3"
+		)
+		(pin "7"
+		)
+		(pin "2"
+		)
+		(pin "4"
+		)
+		(pin "8"
+		)
+		(pin "5"
+		)
+		(pin "1"
+		)
+		(instances
+			(project ""
+				(path "/ad4887b8-c911-42f3-ba06-5ec84621d2a6"
+					(reference "J2")
+					(unit 1)
+				)
+			)
+		)
+	)
+	(symbol
 		(lib_id "Library:R_US")
 		(at 20.32 74.93 0)
@@
 			)
 		)
-		(property "Footprint" ""
+		(property "Footprint" "Library:NPN"
 			(at 177.8 170.18 0)
 			(effects
@@
 	)
 	(symbol
+		(lib_id "Connector:Conn_01x04_Socket")
+		(at 283.21 55.88 0)
+		(unit 1)
+		(exclude_from_sim no)
+		(in_bom yes)
+		(on_board yes)
+		(dnp no)
+		(fields_autoplaced yes)
+		(property "Reference" "J1"
+			(at 284.48 55.8799 0)
+			(effects
+				(font
+					(size 1.27 1.27)
+				)
+				(justify left)
+			)
+		)
+		(property "Value" "Conn_01x04_Socket"
+			(at 284.48 58.4199 0)
+			(effects
+				(font
+					(size 1.27 1.27)
+				)
+				(justify left)
+			)
+		)
+		(property "Footprint" "Connector_JST:JST_EH_S4B-EH_1x04_P2.50mm_Horizontal"
+			(at 283.21 55.88 0)
+			(effects
+				(font
+					(size 1.27 1.27)
+				)
+				(hide yes)
+			)
+		)
+		(property "Datasheet" "~"
+			(at 283.21 55.88 0)
+			(effects
+				(font
+					(size 1.27 1.27)
+				)
+				(hide yes)
+			)
+		)
+		(property "Description" "Generic connector, single row, 01x04, script generated"
+			(at 283.21 55.88 0)
+			(effects
+				(font
+					(size 1.27 1.27)
+				)
+				(hide yes)
+			)
+		)
+		(pin "1"
+		)
+		(pin "2"
+		)
+		(pin "3"
+		)
+		(pin "4"
+		)
+		(instances
+			(project ""
+				(path "/ad4887b8-c911-42f3-ba06-5ec84621d2a6"
+					(reference "J1")
+					(unit 1)
+				)
+			)
+		)
+	)
+	(symbol
 		(lib_id "Library:A1050")
 		(at 91.44 113.03 90)
@@
 			)
 		)
-		(property "Footprint" "Library:FOTORES"
+		(property "Footprint" "Library:FOTORESist"
 			(at 91.44 108.585 90)
 			(effects
@@
 			)
 		)
-		(property "Footprint" ""
+		(property "Footprint" "Library:NPN"
 			(at 207.01 170.18 0)
 			(effects
@@
 			)
 		)
-		(property "Footprint" "Library:FOTORES"
+		(property "Footprint" "Library:FOTORESist"
 			(at 59.69 108.585 90)
 			(effects
@@
 			)
 		)
-		(property "Footprint" ""
+		(property "Footprint" "Library:NPN"
 			(at 191.77 170.18 0)
 			(effects
@@
 	)
 	(symbol
-		(lib_id "Connector:Conn_01x13_Socket")
-		(at 283.21 43.18 0)
-		(unit 1)
-		(exclude_from_sim no)
-		(in_bom yes)
-		(on_board yes)
-		(dnp no)
-		(fields_autoplaced yes)
-		(property "Reference" "J1"
-			(at 284.48 41.9099 0)
-			(effects
-				(font
-					(size 1.27 1.27)
-				)
-				(justify left)
-				(hide yes)
-			)
-		)
-		(property "Value" "Conn_01x13_Socket"
-			(at 284.48 44.4499 0)
-			(effects
-				(font
-					(size 1.27 1.27)
-				)
-				(justify left)
-				(hide yes)
-			)
-		)
-		(property "Footprint" ""
-			(at 283.21 43.18 0)
-			(effects
-				(font
-					(size 1.27 1.27)
-				)
-				(hide yes)
-			)
-		)
-		(property "Datasheet" "~"
-			(at 283.21 43.18 0)
-			(effects
-				(font
-					(size 1.27 1.27)
-				)
-				(hide yes)
-			)
-		)
-		(property "Description" "Generic connector, single row, 01x13, script generated"
-			(at 283.21 43.18 0)
-			(effects
-				(font
-					(size 1.27 1.27)
-				)
-				(hide yes)
-			)
-		)
-		(pin "9"
-		)
-		(pin "7"
-		)
-		(pin "8"
-		)
-		(pin "11"
-		)
-		(pin "3"
-		)
-		(pin "2"
-		)
-		(pin "4"
-		)
-		(pin "5"
-		)
-		(pin "13"
-		)
-		(pin "6"
-		)
-		(pin "1"
-		)
-		(pin "10"
-		)
-		(pin "12"
-		)
-		(instances
-			(project ""
-				(path "/ad4887b8-c911-42f3-ba06-5ec84621d2a6"
-					(reference "J1")
-					(unit 1)
-				)
-			)
-		)
-	)
-	(symbol
 		(lib_id "Library:R_US")
 		(at 120.65 74.93 0)
@@
 			)
 		)
-		(property "Footprint" "Library:FOTORES"
+		(property "Footprint" "Library:FOTORESist"
 			(at 27.94 108.585 90)
 			(effects
@@
 			)
 		)
-		(property "Footprint" "Library:FOTORES"
+		(property "Footprint" "Library:FOTORESist"
 			(at 74.93 108.585 90)
 			(effects
