File: PCB/next-pcb/total/total.kicad_sch (KiCad schematic)
At the start: 259 parts, among them J1 progam, K1 TE_PCH-1xxx2M, K2 DIPxx-1Cxx-51x, SW2 SW_Push, U1 P8X32A-D40, U2 24LC256, U4 TCA9548APWR, U5 ATmega8-16P, U6 TCA9548APWR, U7 ATmega8-16P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

Commit message: V1.01
Connections:
- net LED: no longer names the net of D1.4 (DIN)
Changed lines of the file:
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@@
 	(wire
 		(pts
+			(xy 27.94 443.23) (xy 27.94 459.74)
+		)
+		(stroke
+			(width 0)
+			(type default)
+		)
+	)
+	(wire
+		(pts
 			(xy 261.62 111.76) (xy 261.62 115.57)
 		)
@@
 	(wire
 		(pts
+			(xy 27.94 459.74) (xy 31.75 459.74)
+		)
+		(stroke
+			(width 0)
+			(type default)
+		)
+	)
+	(wire
+		(pts
 			(xy 303.53 439.42) (xy 297.18 439.42)
 		)
@@
 			(effects
 				(font
-					(size 1.27 1.27)
-				)
-				(justify right)
-				(hide yes)
-			)
-		)
-	)
-	(global_label "LED"
-		(shape input)
-		(at 31.75 459.74 180)
-		(fields_autoplaced yes)
-		(effects
-			(font
-				(size 1.27 1.27)
-			)
-			(justify right)
-		)
-		(property "Intersheetrefs" "${INTERSHEET_REFS}"
-			(at 25.3177 459.74 0)
-			(effects
-				(font
