File: PCB/next-pcb/total 14-11/total 14-11.kicad_sch (KiCad schematic)
At the start: 35 parts

Commit message: power toegevoegd
Parts:
- added 3V3_conv1: ~, symbol TSSP4038:3V3_conv1
- added 5V1: ~, symbol TSSP4038:L7805CV
- added 5V_conv1: ~, symbol TSSP4038:5V_conv
- added BT1, BT2: Battery, symbol Device:Battery
- added M1, M2, M3, M4: ~, symbol TSSP4038:M1
- added R3, R4, R5, R6, R7, R8: 100, symbol Device:R
- added SW1, SW2: tacticle push button, 1825910-6:SW_1825910-6-4, symbol button:1825910-6
- added TB9051FTG1: 1, symbol TSSP4038:TB9051FTG
- added TB9051FTG2: 2, symbol TSSP4038:TB9051FTG
- added TB9051FTG3: 3, symbol TSSP4038:TB9051FTG
- added TB9051FTG4: 4, symbol TSSP4038:TB9051FTG
Connections:
- net 3V3: now also R3.2, R4.2, R5.2, R6.2, R7.2, R8.2; no longer C3.1, C4.1, C5.1, C6.1, C7.1, C8.1, IR3.3 (VS), IR4.3 (VS), IR5.3 (VS), IR6.3 (VS), IR7.3 (VS), IR8.3 (VS)
- net GND: now also 3V3_conv1.4 (GND), 3V3_conv1.5 (GND), 5V1.2 (GND), 5V_conv1.4 (GND), 5V_conv1.5 (GND), BT1.2 (-), BT2.2 (-), M1.3 (GND), M2.3 (GND), M3.3 (GND), M4.3 (GND), TB9051FTG1.2 (GND), TB9051FTG2.2 (GND), TB9051FTG3.2 (GND), TB9051FTG4.2 (GND)
- new net: C3.1, IR3.3 (VS), R3.1
- new net: 3V3_conv1.3 (VIN), 5V1.3 (VCC), 5V_conv1.3 (VIN), BT1.1 (+), BT2.1 (+)
- new net: M3.1 (MotorPW), TB9051FTG3.4 (OUT1)
- new net: M3.2 (MotorPW), TB9051FTG3.3 (OUT2)
- new net: M3.4 (VCC), TB9051FTG3.1 (Vin)
- new net: C5.1, IR5.3 (VS), R5.1
- new net: M4.1 (MotorPW), TB9051FTG4.4 (OUT1)
- new net: M4.2 (MotorPW), TB9051FTG4.3 (OUT2)
- new net: M4.4 (VCC), TB9051FTG4.1 (Vin)
- new net: C4.1, IR4.3 (VS), R4.1
- new net: M1.1 (MotorPW), TB9051FTG1.4 (OUT1)
- new net: M1.2 (MotorPW), TB9051FTG1.3 (OUT2)
- new net: M1.4 (VCC), TB9051FTG1.1 (Vin)
- new net: C7.1, IR7.3 (VS), R7.1
- new net: C6.1, IR6.3 (VS), R6.1
- new net: C8.1, IR8.3 (VS), R8.1
- new net: M2.4 (VCC), TB9051FTG2.1 (Vin)
- new net: M2.2 (MotorPW), TB9051FTG2.3 (OUT2)
- new net: M2.1 (MotorPW), TB9051FTG2.4 (OUT1)
Other:
- moved on the sheet: C10, C11, C12, C13, C14, C15, C16, C9, IR10, IR11, IR12, IR13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

Commit message: V1.01
Parts:
- added 3V3: ~, symbol TSSP4038:3V3_Converter_
- added C17, C19, C20, C21, C22, C37, C38, C39, C40, C41, C42, C43, C44, C45, C46, C47, C48, C49, C50, C51, C52, C53, C54, C55, C56, C57, C58, C77, C78, C79, C80: 100nF, symbol Device:C
- added C18: 100NF, symbol Device:C
- added C23, C24, C25, C26, C27, C28, C29, C30, C61, C62, C63, C64, C65, C66, C67, C68: 0.1uF, symbol Device:C
- added C31, C32, C33, C34, C35, C36, C59, C60, C69, C70, C71, C72, C73, C74, C75, C76: 1uF, symbol Device:C_Polarized
- added CS17, CS18, CS19, CS20, CS21, CS22, CS23, CS24, CS25, CS26, CS27, CS28, CS29, CS30, CS31, CS32: ~, Lib:ISL29125, symbol lib:ISL29125
- added D1, D10, D11, D12, D13, D14, D15, D16, D17, D18, D19, D2, D20, D21, D22, D23, D24, D25, D26, D27, D28, D29, D3, D30, D31, D32, D4, D5, D6, D7, D8, D9: WS2812B, LED_SMD:LED_WS2812B_PLCC4_5.0x5.0mm_P3.2mm, symbol LED:WS2812B
- added Esp1: 38 pin, symbol ESP32-38pin:Esp32
- added JP17, JP18, JP19, JP20, JP21, JP22, JP23, JP24, JP25, JP26, JP27, JP28, JP29, JP30, JP31, JP32: SolderJumper_3_Bridged123, symbol Jumper:SolderJumper_3_Bridged123
- added R10, R11, R111, R112, R113, R114, R115, R116, R117, R118, R12, R13, R14, R15, R16, R9: 100, symbol Device:R_US
- added R104, R105, R106, R107, R108, R109, R120, R121, R122, R123, R124, R125, R126, R127, R128, R129, R130, R131, R132, R133, R134, R135, R136, R137, R138, R139, R140, R141, R142, R143, R51, R73, R74, R75, R76, R77, R78, R79, R80, R81, R82, R83, R84, R85, R86, R87, R88, R89: 10K, symbol Device:R_US
- added R110, R144: PULL-UP, symbol Device:R_US
- added R119, R17: 100K, symbol Device:R_US
- added SW3: SW_DIP_x03, symbol Switch:SW_DIP_x03
- added SW4: tacticle push button, 1825910-6:SW_1825910-6-4, symbol button:1825910-6
- added U1: ~, Library:miniIMU, symbol TSSP4038:miniIMU
- added U10: 74AHCT125, symbol 74xx:74AHCT125
- added U3, U5: TCA9548APWR, Package_SO:TSSOP-24_4.4x7.8mm_P0.65mm, symbol Interface_Expansion:TCA9548APWR
- added U6: ~, Lib:openMV_H7, symbol lib:openMV_H7
- added teensy1: Teensy4.1, Library:Teensy41, symbol TSSP4038:Teensy4.1
Connections:
- net 3V3: now also 3V3_conv1.6 (VOUT), 3V3.1 (VOUT), Esp1.1 (3.3v)
- net GND: now also Esp32.14 (GND), Esp32.32 (GND), Esp32.38 (GND), SW1.3, SW1.4, SW2.3, SW2.4, 3V3.2 (GND), C17.2, C18.2, C19.2, C20.2, C21.2, C22.2, C23.2, C24.2, C25.2, C26.2, C27.2, C28.2, C29.2, C30.2, C31.2, C32.2, C33.2, C34.2, C35.2, C36.2, C37.2, C38.2, C39.2, C40.2, C41.2, C42.2, C43.2, C44.2, C45.2, C46.2, C47.2, C48.2, C49.2, C50.2, C51.2, C52.2, C53.2, C54.2, C55.2, C56.2, C57.2, C58.2, C59.2, C60.2, C61.2, C62.2, C63.2, C64.2, C65.2, C66.2, C67.2, C68.2, C69.2, C70.2, C71.2, C72.2, C73.2, C74.2, C75.2, C76.2, C77.2, C78.2, C79.2, C80.2, CS17.2 (NC), CS17.3 (GND), CS18.2 (NC), CS18.3 (GND), CS19.2 (NC), CS19.3 (GND), CS20.2 (NC), CS20.3 (GND), CS21.2 (NC), CS21.3 (GND), CS22.2 (NC), CS22.3 (GND), CS23.2 (NC), CS23.3 (GND), CS24.2 (NC), CS24.3 (GND), CS25.2 (NC), CS25.3 (GND), CS26.2 (NC), CS26.3 (GND), CS27.2 (NC), CS27.3 (GND), CS28.2 (NC), CS28.3 (GND), CS29.2 (NC), CS29.3 (GND), CS30.2 (NC), CS30.3 (GND), CS31.2 (NC), CS31.3 (GND), CS32.2 (NC), CS32.3 (GND), D1.3 (VSS), D10.3 (VSS), D11.3 (VSS), D12.3 (VSS), D13.3 (VSS), D14.3 (VSS), D15.3 (VSS), D16.3 (VSS), D17.3 (VSS), D18.3 (VSS), D19.3 (VSS), D2.3 (VSS), D20.3 (VSS), D21.3 (VSS), D22.3 (VSS), D23.3 (VSS), D24.3 (VSS), D25.3 (VSS), D26.3 (VSS), D27.3 (VSS), D28.3 (VSS), D3.3 (VSS), D30.3 (VSS), D31.3 (VSS), D32.3 (VSS), D4.3 (VSS), D5.3 (VSS), D6.3 (VSS), D7.3 (VSS), D8.3 (VSS), D9.3 (VSS), Esp1.38 (GND), SW3.4, SW3.5, SW3.6, SW4.3, SW4.4, U10.1, U3.1 (A0), U3.12 (GND), U3.2 (A1), U3.21 (A2), U5.1 (A0), U5.12 (GND), U5.2 (A1), U5.21 (A2), U6.0 (SCREW), U6.16 (GND)
- net 12V: now reaches 3V3_conv1.3 (VIN), 5V1.3 (VCC), 5V_conv1.3 (VIN), BT1.1 (+), BT2.1 (+)
- net 12V: now also TB9051FTG1.1 (Vin), TB9051FTG2.1 (Vin), TB9051FTG3.1 (Vin), TB9051FTG4.1 (Vin), 3V3.3 (VCC)
- net 5V: now reaches M3.4 (VCC)
- net 5V: now also 5V1.1 (VOUT), 5V_conv1.6 (VOUT), M1.4 (VCC), M2.4 (VCC), M4.4 (VCC), C17.1, C18.1, C19.1, C20.1, C21.1, C22.1, C37.1, C38.1, C39.1, C40.1, C41.1, C42.1, C43.1, C44.1, C45.1, C46.1, C47.1, C48.1, C49.1, C50.1, C51.1, C52.1, C53.1, C54.1, C55.1, C56.1, C57.1, C58.1, C77.1, C78.1, C79.1, C80.1, D1.1 (VDD), D10.1 (VDD), D11.1 (VDD), D12.1 (VDD), D13.1 (VDD), D14.1 (VDD), D15.1 (VDD), D16.1 (VDD), D17.1 (VDD), D18.1 (VDD), D19.1 (VDD), D2.1 (VDD), D20.1 (VDD), D21.1 (VDD), D22.1 (VDD), D23.1 (VDD), D24.1 (VDD), D25.1 (VDD), D26.1 (VDD), D27.1 (VDD), D28.1 (VDD), D29.1 (VDD), D3.1 (VDD), D30.1 (VDD), D31.1 (VDD), D32.1 (VDD), D4.1 (VDD), D5.1 (VDD), D6.1 (VDD), D7.1 (VDD), D8.1 (VDD), D9.1 (VDD), Esp1.19 (5V); no longer TB9051FTG3.1 (Vin)
- net at Esp32.29 (GPIO5): now also SW4.1
- net at Esp32.30 (GPIO18): now also SW2.1
- net at Esp32.31 (GPIO19): now also SW1.1
- net SDA Boven: now reaches Esp32.33 (GPIO21)
- net RX_CAM: now reaches Esp32.34 (GPIO3)
- net RX_CAM: now also U6.6 (P5)
- net TX_CAM: now reaches Esp32.35 (GPIO1)
- net TX_CAM: now also U6.5 (P4)
- net SCL Boven: now reaches Esp32.36 (GPIO22)
- new net: CS22.5 (INT), R107.2
- new net: C27.1, C35.1, CS21.1 (VDD), R13.2
- new net: CS21.4 (SDA), R76.2, U3.10 (SD3)
- new net: CS21.5 (INT), R106.2
- new net: CS21.6 (SCL), R84.2, U3.11 (SC3)
- new net: CS30.5 (INT), R141.2
- new net: C67.1, C75.1, CS31.1 (VDD), R117.2
- new net: C26.1, C34.1, CS20.1 (VDD), R12.2
- new net: JP26.1 (A), R129.1
- new net: CS26.6 (SCL), R129.2, U5.18 (SC6)
- new net: C62.1, C70.1, CS26.1 (VDD), R112.2
- new net: JP21.1 (A), R84.1
- new net: JP31.1 (A), R134.1
- new net: CS31.6 (SCL), R134.2, U5.7 (SC1)
- new net: D21.2 (DOUT), D23.4 (DIN)
- new net: D19.2 (DOUT), D21.4 (DIN)
- new net: JP23.1 (A), R86.1
- new net: CS23.6 (SCL), R86.2, U3.7 (SC1)
- new net: JP28.1 (A), R131.1
- new net: JP28.3 (B), R123.1
- new net: Esp1.29 (GPIO5), SW3.1
- new net: Esp1.30 (GPIO18), SW3.2
- new net: Esp1.31 (GPIO19), SW3.3
- new net: JP24.3 (B), R79.1
- new net: CS24.4 (SDA), R79.2, U3.4 (SD0)
- new net: JP24.1 (A), R87.1
- new net: CS24.6 (SCL), R87.2, U3.5 (SC0)
- new net: CS28.4 (SDA), R123.2, U5.13 (SD4)
- new net: C23.1, C31.1, CS17.1 (VDD), R9.2
- new net: JP30.1 (A), R133.1
- new net: CS30.6 (SCL), R133.2, U5.9 (SC2)
- new net: C63.1, C71.1, CS27.1 (VDD), R113.2
- new net: JP17.3 (B), R17.1, R51.1
- new net: CS17.4 (SDA), R17.2, R51.2, U3.19 (SD7)
- new net: C25.1, C33.1, CS19.1 (VDD), R11.2
- new net: CS19.4 (SDA), R74.2, U3.15 (SD5)
- new net: CS19.5 (INT), R104.2
- new net: CS19.6 (SCL), R82.2, U3.16 (SC5)
- new net: D13.2 (DOUT), D14.4 (DIN)
- new net: D12.2 (DOUT), D13.4 (DIN)
- new net: C30.1, C60.1, CS24.1 (VDD), R16.2
- new net: D27.2 (DOUT), D29.4 (DIN)
- new net: D25.2 (DOUT), D27.4 (DIN)
- new net: C61.1, C69.1, CS25.1 (VDD), R111.2
- new net: JP26.3 (B), R121.1
- new net: CS26.4 (SDA), R121.2, U5.17 (SD6)
- new net: C64.1, C72.1, CS28.1 (VDD), R114.2
- new net: CS28.5 (INT), R139.2
- new net: CS28.6 (SCL), R131.2, U5.14 (SC4)
- new net: JP21.3 (B), R76.1
- new net: JP29.1 (A), R132.1
- new net: JP29.3 (B), R124.1
- new net: C24.1, C32.1, CS18.1 (VDD), R10.2
- new net: JP23.3 (B), R78.1
- new net: CS23.4 (SDA), R78.2, U3.6 (SD1)
- new net: D26.2 (DOUT), D28.4 (DIN)
- new net: D24.2 (DOUT), D26.4 (DIN)
- new net: CS27.5 (INT), R138.2
- new net: D4.2 (DOUT), D5.4 (DIN)
- new net: D3.2 (DOUT), D4.4 (DIN)
- new net: R110.1, U3.3 (~{RESET})
- new net: C65.1, C73.1, CS29.1 (VDD), R115.2
- new net: D7.2 (DOUT), D8.4 (DIN)
- new net: D6.2 (DOUT), D7.4 (DIN)
- new net: JP32.1 (A), R135.1
- new net: JP32.3 (B), R127.1
- new net: CS17.5 (INT), R88.2
- new net: CS17.6 (SCL), R80.2, U3.20 (SC7)
- new net: D1.4 (DIN), U10.3
- new net: D18.4 (DIN), D31.2 (DOUT)
- new net: D29.2 (DOUT), D31.4 (DIN)
- new net: C68.1, C76.1, CS32.1 (VDD), R118.2
- new net: CS26.5 (INT), R137.2
- new net: D16.2 (DOUT), D17.4 (DIN)
- new net: D15.2 (DOUT), D16.4 (DIN)
- new net: JP20.3 (B), R75.1
- new net: CS20.4 (SDA), R75.2, U3.13 (SD4)
- new net: C29.1, C59.1, CS23.1 (VDD), R15.2
- new net: D22.2 (DOUT), D24.4 (DIN)
- new net: CS31.4 (SDA), R126.2, U5.6 (SD1)
- new net: CS31.5 (INT), R142.2
- new net: D1.2 (DOUT), D2.4 (DIN)
- new net: CS29.4 (SDA), R124.2, U5.10 (SD3)
- new net: CS29.6 (SCL), R132.2, U5.11 (SC3)
- new net: CS27.4 (SDA), R122.2, U5.15 (SD5)
- new net: CS27.6 (SCL), R130.2, U5.16 (SC5)
- new net: CS25.4 (SDA), R119.2, R120.2, U5.19 (SD7)
- new net: CS25.6 (SCL), R128.2, U5.20 (SC7)
- new net: R144.1, U5.3 (~{RESET})
- new net: CS32.4 (SDA), R127.2, U5.4 (SD0)
- new net: CS32.6 (SCL), R135.2, U5.5 (SC0)
- new net: CS30.4 (SDA), R125.2, U5.8 (SD2)
- new net: D2.2 (DOUT), D3.4 (DIN)
- new net: CS20.5 (INT), R105.2
- new net: JP19.3 (B), R74.1
- new net: C28.1, C36.1, CS22.1 (VDD), R14.2
- new net: D10.2 (DOUT), D11.4 (DIN)
- new net: D10.4 (DIN), D9.2 (DOUT)
- new net: JP27.1 (A), R130.1
- new net: JP22.1 (A), R85.1
- new net: JP22.3 (B), R77.1
- new net: JP31.3 (B), R126.1
- new net: D30.2 (DOUT), D32.4 (DIN)
- new net: JP19.1 (A), R82.1
- new net: JP18.3 (B), R73.1
- new net: CS18.4 (SDA), R73.2, U3.17 (SD6)
- new net: D23.2 (DOUT), D25.4 (DIN)
- new net: CS29.5 (INT), R140.2
- new net: C66.1, C74.1, CS30.1 (VDD), R116.2
- new net: D11.2 (DOUT), D12.4 (DIN)
- new net: CS24.5 (INT), R109.2
- new net: JP25.1 (A), R128.1
- new net: JP25.3 (B), R119.1, R120.1
- new net: JP20.1 (A), R83.1
- new net: JP18.1 (A), R81.1
- new net: CS18.6 (SCL), R81.2, U3.18 (SC6)
- new net: CS20.6 (SCL), R83.2, U3.14 (SC4)
- new net: CS22.4 (SDA), R77.2, U3.8 (SD2)
- new net: CS22.6 (SCL), R85.2, U3.9 (SC2)
- new net: JP27.3 (B), R122.1
- new net: JP30.3 (B), R125.1
- new net: JP17.1 (A), R80.1
- new net: D28.2 (DOUT), D30.4 (DIN)
- new net: D5.2 (DOUT), D6.4 (DIN)
- new net: CS25.5 (INT), R136.2
- new net: CS23.5 (INT), R108.2
- new net: D17.2 (DOUT), D19.4 (DIN)
- new net: D20.2 (DOUT), D22.4 (DIN)
- new net: D18.2 (DOUT), D20.4 (DIN)
- new net: CS18.5 (INT), R89.2
- new net: CS32.5 (INT), R143.2
- new net: D14.2 (DOUT), D15.4 (DIN)
- new net: D8.2 (DOUT), D9.4 (DIN)
- new net +3.3V: JP18.2 (C), JP19.2 (C), JP20.2 (C), JP21.2 (C), JP22.2 (C), JP23.2 (C), JP24.2 (C), JP25.2 (C), JP26.2 (C), JP27.2 (C), JP28.2 (C), JP29.2 (C), JP30.2 (C), JP31.2 (C), JP32.2 (C), R10.1, R104.1, R105.1, R106.1, R107.1, R108.1, R109.1, R11.1, R110.2, R111.1, R112.1, R113.1, R114.1, R115.1, R116.1, R117.1, R118.1, R12.1, R13.1, R136.1, R137.1, R138.1, R139.1, R14.1, R140.1, R141.1, R142.1, R143.1, R144.2, R15.1, R16.1, R88.1, R89.1, R9.1, U3.24 (VCC), U5.24 (VCC)
- new net +5V: U6.15 (VIN)
- new net LED: Esp1.3 (GPI36), U10.2
- new net SCL Onder: Esp1.36 (GPIO22), U3.22 (SCL), U5.22 (SCL)
- new net SDA Onder: Esp1.33 (GPIO21), U3.23 (SDA), U5.23 (SDA)
- no-connect marks 0 -> 12
Other:
- note added: "https://www.renesas.com/en/document/dst/isl29125-datasheet"
- moved on the sheet: 3V3_conv1, 5V1, 5V_conv1, BT1, BT2, Esp32, SW1, SW2
