File: PCB/Electronics/Electronics.kicad_sch (KiCad schematic)
At the start: 366 parts, among them IC1 TB9051FTG, IC2 TB9051FTG, IC3 TB9051FTG, IC4 TB9051FTG, Q1 Q_PMOS_DGS, Q2 Q_PMOS_DGS, Q3 Q_PMOS_DGS, Q4 Q_PMOS_DGS, SW1 tacticle push button, SW2 tacticle push button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

Commit message: Update Electronics.kicad_sch
Parts:
- removed U13: ESP32-S3-DEVKITM-1-N8, ESP32-S3-DEVKITM-1-N8:MODULE_ESP32-S3-DEVKITM-1-N8, symbol ESP32-S3-DEVKITM-1-N8:ESP32-S3-DEVKITM-1-N8
- added J1, J4, J6: Conn_01x08_Socket, symbol Connector:Conn_01x08_Socket
- added J2, J3, J5: Conn_01x08_Pin, symbol Connector:Conn_01x08_Pin
- added J7: Conn_01x03_Pin, symbol Connector:Conn_01x03_Pin
- added J8: Conn_01x03_Socket, symbol Connector:Conn_01x03_Socket
Connections:
- net 3V3: now also J1.1 (Pin_1), J2.1 (Pin_1), J3.1 (Pin_1), J4.1 (Pin_1), J7.3 (Pin_3), J8.1 (Pin_1)
- net 5V: now also U11.J1_21 (5V0), U5.4 (vin), J1.3 (Pin_3), J2.3 (Pin_3), J3.3 (Pin_3), J4.3 (Pin_3), J7.1 (Pin_1), J8.3 (Pin_3)
- net GND: now also U11.J1_22 (GND_J1_22), J1.2 (Pin_2), J2.2 (Pin_2), J3.2 (Pin_2), J4.2 (Pin_2), J7.2 (Pin_2), J8.2 (Pin_2)
- net LED: now also J1.4 (Pin_4), J2.4 (Pin_4), J3.4 (Pin_4), J4.4 (Pin_4)
- net SCL: now also J3.6 (Pin_6), J4.6 (Pin_6)
- net SDA: now also J3.5 (Pin_5), J4.5 (Pin_5)
- net esp-rx: now also J1.6 (Pin_6), J2.6 (Pin_6)
- net esp-tx: now also J1.5 (Pin_5), J2.5 (Pin_5)
- net rx-cam: now also J1.7 (Pin_7), J2.7 (Pin_7)
- net rx-m1: now also J5.2 (Pin_2), J6.2 (Pin_2)
- net rx-m2: now also J5.4 (Pin_4), J6.4 (Pin_4)
- net rx-m3: now also J5.6 (Pin_6), J6.6 (Pin_6)
- net rx-m4: now also J5.8 (Pin_8), J6.8 (Pin_8)
- net tx-cam: now also J1.8 (Pin_8), J2.8 (Pin_8)
- net tx-m1: now also J5.1 (Pin_1), J6.1 (Pin_1)
- net tx-m2: now also J5.3 (Pin_3), J6.3 (Pin_3)
- net tx-m3: now also J5.5 (Pin_5), J6.5 (Pin_5)
- net tx-m4: now also J5.7 (Pin_7), J6.7 (Pin_7)
Other:
- moved on the sheet: 3V3_conv1, C10, C11, C17, C23, C24, C25, C26, C27, C28, C29, C30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
