File: PCB/Electronics/Electronics.kicad_sch (KiCad schematic)
At the start: 207 parts, among them U4 TCA9548APWR, U6 TCA9548APWR

Commit message: pcb changes
-file now in electronics
-motordriver integraded
-etc
Parts:
- removed D1, D10, D11, D12, D13, D14, D15, D16, D17, D18, D19, D2, D20, D21, D22, D23, D24, D25, D26, D27, D28, D29, D3, D30, D31, D32, D4, D5, D6, D7, D8, D9: WS2812B, LED_SMD:LED_WS2812B_PLCC4_5.0x5.0mm_P3.2mm, symbol LED:WS2812B
- removed DR1, DR2, DR3, DR4: ~, Lib:TB9051FTG, symbol lib:TB9051FTG
- added 3V3: ~, symbol TSSP4038:3V3_Converter_
- added 3V3_conv1: ~, symbol TSSP4038:3V3_conv1
- added 5V1: ~, symbol TSSP4038:L7805CV
- added 5V_conv1: ~, symbol TSSP4038:5V_conv
- added BT1, BT2: Battery, symbol Device:Battery
- added C1, C10, C11, C17, C2, C23, C24, C25, C26, C27, C28, C29, C3, C30, C31, C32, C33, C34, C35, C36, C4, C5, C59, C6, C60, C61, C62, C63, C64, C65, C7, C77, C78, C79, C8, C80, C81, C82, C83, C84, C85, C86, C87, C88, C89, C9, C90, C91: 100nF, symbol Device:C
- added C100, C101, C102, C107, C108, C69, C70, C71, C73, C93, C94, C95: 0.1uF, symbol Device:C
- added C103, C72, C74, C96: 4.7uF, symbol Device:C
- added C104, C66, C75, C97: 0.47uF, symbol Device:C
- added C105, C67, C76, C98: NP, symbol Device:C
- added C106, C68, C92, C99: 47uF, symbol Device:C
- added D1, D2, D3, D4: 16.2v, symbol Device:D_Zener
- added D33, D34, D35, D36, D37, D38, D39, D40, D41, D42, D43, D44, D45, D46, D47, D48, D49, D50, D51, D52, D53, D54, D55, D56, D57, D58, D59, D60, D61, D62, D63, D64: WS2812B, LED_SMD:LED_WS2812B_PLCC4_5.0x5.0mm_P3.2mm, symbol LED:WS2812B
- added IC1, IC2, IC3, IC4: TB9051FTG, TB9051FTG, symbol SamacSys_Parts:TB9051FTG
- added JP17, JP18, JP19, JP20, JP21, JP22, JP24: SolderJumper_3_Bridged12, symbol Jumper:SolderJumper_3_Bridged12
- added JP23: SolderJumper_3_Bridged123, symbol Jumper:SolderJumper_3_Bridged123
- added Q1, Q2, Q3, Q4: Q_PMOS_DGS, symbol Transistor_FET:Q_PMOS_DGS
- added R104, R113, R80, R81: 1, symbol Device:R_US
- added R105, R108, R109, R110, R114, R117, R118, R119, R51, R73, R74, R78, R82, R85, R86, R87: 1K, symbol Device:R_US
- added R106, R115, R122, R123, R124, R125, R126, R79, R83: 100K, symbol Device:R_US
- added R107, R112, R116, R121, R75, R77, R84, R89: 220, symbol Device:R_US
- added R111, R120, R127, R128, R76, R88: 10K, symbol Device:R_US
- added SW1, SW2, SW4: tacticle push button, 1825910-6:SW_1825910-6-4, symbol button:1825910-6
- added SW3: SW_DIP_x03, symbol Switch:SW_DIP_x03
- added U1: ~, Lib:openMV_H7, symbol lib:openMV_H7
- added U10, U12: 74AHCT125, symbol 74xx:74AHCT125
- added U11: ESP32-S3-DEVKITM-1-N8, ESP32-S3-DEVKITM-1-N8:MODULE_ESP32-S3-DEVKITM-1-N8, symbol ESP32-S3-DEVKITM-1-N8:ESP32-S3-DEVKITM-1-N8
- added U2: ~, teensy.pretty-master:protoboard, symbol New_Library:extra-pins
- added U3, U7, U8, U9: ATtiny85V-10P, Package_DIP:DIP-8_W7.62mm, symbol MCU_Microchip_ATtiny:ATtiny85V-10P
- added U5: ~, Library:miniIMU, symbol TSSP4038:miniIMU
- added teensy1: Teensy4.1, Library:Teensy41, symbol TSSP4038:Teensy4.1
- R1, R50, R72: value PULL-UP -> 100K
- R10, R11, R12, R13, R14, R15, R16, R17, R2, R3, R4, R5, R6, R7, R8, R9: value R_US -> 100
Connections:
- net +12V: now also Q1.1 (D), Q2.1 (D), Q3.1 (D), Q4.1 (D), U2.8 (12v)
- net +3.3V: now also R122.2, R123.2, R124.2, R125.2, R126.2
- net +5V: now also C102.1, C71.1, C73.1, C95.1, IC1.2 (VCC), IC2.2 (VCC), IC3.2 (VCC), IC4.2 (VCC), JP24.3 (B), R104.2, R111.1, R113.2, R120.1, R76.1, R80.2, R81.2, R88.1, U1.15 (VIN), U10.14 (VCC), U2.5 (5v), U3.8 (VCC), U7.8 (VCC), U8.8 (VCC), U9.8 (VCC), teensy1.48 (VIN)
- net GND: now also IR1.2 (GND), IR10.2 (GND), IR11.2 (GND), IR12.2 (GND), IR13.2 (GND), IR14.2 (GND), IR15.2 (GND), IR16.2 (GND), IR2.2 (GND), IR3.2 (GND), IR4.2 (GND), IR5.2 (GND), IR6.2 (GND), IR7.2 (GND), IR8.2 (GND), IR9.2 (GND), 3V3.2 (GND), 3V3_conv1.4 (GND), 3V3_conv1.5 (GND), 5V1.2 (GND), 5V_conv1.4 (GND), 5V_conv1.5 (GND), BT1.2 (-), BT2.2 (-), C1.2, C10.2, C100.2, C101.2, C102.2, C103.2, C104.1, C105.2, C106.2, C107.2, C108.2, C11.2, C17.2, C2.2, C23.2, C24.2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; no longer U4.1 (A0), U4.2 (A1), U4.21 (A2), U6.2 (A1), U6.21 (A2)
- net LED: now also U12.2, teensy1.4 (2_OUT2)
- net SCL: now also R128.2, U2.1 (SCL), U5.1 (scl), teensy1.41 (19_A5_SCL)
- net SDA: now also R127.2, U2.1 (SCL), U5.2 (sda), teensy1.40 (18_A4_SDA)
- net at IR11.3 (Vs), R12.1: now also C86.1
- net +3V3: now reaches R12.2
- net +3V3: now also R10.2, R11.2, R13.2, R14.2, R15.2, R16.2, R17.2, R2.2, R3.2, R4.2, R5.2, R6.2, R7.2, R8.2, R9.2, JP24.1 (A), U11.J1_1 (3V3), U2.6 (3.3v)
- net at IR12.3 (Vs), R13.1: now also C87.1
- net at IR14.3 (Vs), R15.1: now also C89.1
- net at IR10.1 (OUT): now also U11.J1_11 (GPIO9)
- net at IR10.3 (Vs), R11.1: now also C85.1
- net at IR9.1 (OUT): now also U11.J1_10 (GPIO8)
- net at IR9.3 (Vs), R10.1: now also C84.1
- net at IR11.1 (OUT): now also U11.J1_12 (GPIO10)
- net at IR6.3 (Vs), R7.1: now also C5.1
- net at IR16.3 (Vs), R17.1: now also C91.1
- net at IR3.3 (Vs), R4.1: now also C2.1
- net out1-m4: now reaches M3.1 (+)
- net out1-m4: now also IC4.13 (OUT1_1), IC4.14 (OUT1_2)
- net out2-m4: now reaches M3.2 (-)
- net out2-m4: now also IC4.22 (OUT2_1), IC4.23 (OUT2_2)
- net at IR6.1 (OUT): now also U11.J1_7 (GPIO5)
- net at IR14.1 (OUT): now also U11.J1_15 (GPIO13)
- net at IR16.1 (OUT): now also U11.J1_17 (GPIO15)
- net at IR4.3 (Vs), R5.1: now also C3.1
- net out1-m2: now reaches M1.1 (+)
- net out1-m2: now also IC2.13 (OUT1_1), IC2.14 (OUT1_2)
- net out2-m2: now reaches M1.2 (-)
- net out2-m2: now also IC2.22 (OUT2_1), IC2.23 (OUT2_2)
- net out2-m3: now reaches M2.2 (-)
- net out2-m3: now also IC3.22 (OUT2_1), IC3.23 (OUT2_2)
- net out1-m3: now reaches M2.1 (+)
- net out1-m3: now also IC3.13 (OUT1_1), IC3.14 (OUT1_2)
- net at IR3.1 (OUT): now also U11.J1_4 (GPIO2)
- net at IR13.1 (OUT): now also U11.J1_14 (GPIO12)
- net at IR13.3 (Vs), R14.1: now also C88.1
- net at IR5.3 (Vs), R6.1: now also C4.1
- net at IR8.3 (Vs), R9.1: now also C83.1
- net at IR15.3 (Vs), R16.1: now also C90.1
- net out1-m1: now reaches M4.1 (+)
- net out1-m1: now also IC1.13 (OUT1_1), IC1.14 (OUT1_2)
- net out2-m1: now reaches M4.2 (-)
- net out2-m1: now also IC1.22 (OUT2_1), IC1.23 (OUT2_2)
- net at IR1.1 (OUT): now also U11.J1_2 (GPIO0)
- net at IR1.3 (Vs), R2.1: now also C81.1
- net at IR7.1 (OUT): now also U11.J1_8 (GPIO6)
- net at IR7.3 (Vs), R8.1: now also C82.1
- net at U6.1 (A0): now also JP17.2 (C); no longer R1.1
- net at IR4.1 (OUT): now also U11.J1_5 (GPIO3)
- net at IR2.1 (OUT): now also U11.J1_3 (GPIO1)
- net at IR2.3 (Vs), R3.1: now also C1.1
- net at IR8.1 (OUT): now also U11.J1_9 (GPIO7)
- net at IR15.1 (OUT): now also U11.J1_16 (GPIO14)
- net at IR5.1 (OUT): now also U11.J1_6 (GPIO4)
- net at IR12.1 (OUT): now also U11.J1_13 (GPIO11)
- new net: C74.1, R81.1
- new net: IC3.7 (OCM), R105.2, R107.2
- new net: D4.2 (A), Q4.2 (G), R115.2
- new net: D55.2 (DOUT), D59.4 (DIN)
- new net: D51.2 (DOUT), D55.4 (DIN)
- new net: IC2.7 (OCM), R82.2, R84.2
- new net: D3.2 (A), Q3.2 (G), R106.2
- new net: JP19.1 (A), R123.1
- new net: IC1.18 (DIAG), R76.2, R77.2
- new net: D42.2 (DOUT), D46.4 (DIN)
- new net: D38.2 (DOUT), D42.4 (DIN)
- new net: U2.10 (P1), teensy1.18 (26_A12_MOSI1)
- new net: U2.9 (P0), teensy1.19 (27_A13_SCK1)
- new net: SW3.1, teensy1.5 (3_LRCLK2)
- new net: SW3.2, teensy1.6 (4_BCLK2)
- new net: SW3.3, teensy1.7 (5_IN2)
- new net: JP21.3 (B), R126.1
- new net: D39.2 (DOUT), D43.4 (DIN)
- new net: D35.2 (DOUT), D39.4 (DIN)
- new net: IC4.7 (OCM), R114.2, R116.2
- new net: D1.2 (A), Q1.2 (G), R79.2
- new net: IC3.1 (OCC), R108.2
- new net: IC1.1 (OCC), R78.2
- new net: D56.2 (DOUT), D60.4 (DIN)
- new net: D52.2 (DOUT), D56.4 (DIN)
- new net: D36.4 (DIN), D63.2 (DOUT)
- new net: D59.2 (DOUT), D63.4 (DIN)
- new net: D60.2 (DOUT), D64.4 (DIN)
- new net: D48.2 (DOUT), D52.4 (DIN)
- new net: D44.2 (DOUT), D48.4 (DIN)
- new net: D33.4 (DIN), U12.3
- new net: IC2.1 (OCC), R85.2
- new net: JP22.3 (B), R125.1
- new net: JP22.2 (C), U4.1 (A0)
- new net: JP21.2 (C), U4.2 (A1)
- new net: JP20.2 (C), U4.21 (A2)
- new net: R73.1, U3.2 (XTAL1/PB3)
- new net: IC1.8 (PWM1), U3.5 (AREF/PB0)
- new net: IC1.9 (PWM2), U3.6 (PB1)
- new net: R51.1, U3.7 (PB2)
- new net: R118.1, U9.7 (PB2)
- new net: IC4.3 (ENB), R118.2
- new net: IC3.18 (DIAG), R111.2, R112.2
- new net: D53.2 (DOUT), D57.4 (DIN)
- new net: D49.2 (DOUT), D53.4 (DIN)
- new net: D35.4 (DIN), D62.2 (DOUT)
- new net: D58.2 (DOUT), D62.4 (DIN)
- new net: SW2.1, U11.J3_21 (GPIO48)
- new net: SW4.1, U11.J3_22 (GPIO47)
- new net: IC2.18 (DIAG), R88.2, R89.2
- new net: IC1.7 (OCM), R74.2, R75.2
- new net: D46.2 (DOUT), D50.4 (DIN)
- new net: IC4.18 (DIAG), R120.2, R121.2
- new net: C72.1, R80.1
- new net: JP17.3 (B), R1.1
- new net: D34.2 (DOUT), D38.4 (DIN)
- new net: R109.1, U8.7 (PB2)
- new net: IC3.3 (ENB), R109.2
- new net: IC4.1 (OCC), R117.2
- new net: JP20.3 (B), R124.1
- new net: D54.2 (DOUT), D58.4 (DIN)
- new net: R119.1, U9.2 (XTAL1/PB3)
- new net: IC4.5 (EN), R119.2
- new net: IC4.8 (PWM1), U9.5 (AREF/PB0)
- new net: IC4.9 (PWM2), U9.6 (PB1)
- new net: IC3.5 (EN), R110.2
- new net: IC3.8 (PWM1), U8.5 (AREF/PB0)
- new net: IC3.9 (PWM2), U8.6 (PB1)
- new net: D33.2 (DOUT), D37.4 (DIN)
- new net: IC1.3 (ENB), R51.2
- new net: D50.2 (DOUT), D54.4 (DIN)
- new net: R87.1, U7.2 (XTAL1/PB3)
- new net: IC2.8 (PWM1), U7.5 (AREF/PB0)
- new net: IC2.9 (PWM2), U7.6 (PB1)
- new net: R86.1, U7.7 (PB2)
- new net: D47.2 (DOUT), D51.4 (DIN)
- new net: JP18.2 (C), U6.2 (A1)
- new net: JP18.3 (B), R122.1
- new net: D40.2 (DOUT), D44.4 (DIN)
- new net: R110.1, U8.2 (XTAL1/PB3)
- new net: SW1.1, U11.J3_20 (GPIO19)
- new net: D2.2 (A), Q2.2 (G), R83.2
- new net: D36.2 (DOUT), D40.4 (DIN)
- new net: JP23.1 (A), R128.1
- new net: JP23.2 (C), JP24.2 (C)
- new net: JP23.3 (B), R127.1
- new net: D41.2 (DOUT), D45.4 (DIN)
- new net: D37.2 (DOUT), D41.4 (DIN)
- new net: D45.2 (DOUT), D49.4 (DIN)
- new net: JP19.2 (C), U6.21 (A2)
- new net: D34.4 (DIN), D61.2 (DOUT)
- new net: D57.2 (DOUT), D61.4 (DIN)
- new net: C96.1, R104.1
- new net: C103.1, R113.1
- new net: IC1.5 (EN), R73.2
- new net: IC2.5 (EN), R87.2
- new net: D43.2 (DOUT), D47.4 (DIN)
- new net: IC2.3 (ENB), R86.2
- new net 12V: 3V3.3 (VCC), 3V3_conv1.3 (VIN), 5V1.3 (VCC), 5V_conv1.3 (VIN), BT1.1 (+), BT2.1 (+)
- new net 3V3: 3V3.1 (VOUT), 3V3_conv1.6 (VOUT)
- new net 5V: 5V1.1 (VOUT), 5V_conv1.6 (VOUT), C10.1, C11.1, C17.1, C23.1, C24.1, C25.1, C26.1, C27.1, C28.1, C29.1, C30.1, C31.1, C32.1, C33.1, C34.1, C35.1, C36.1, C59.1, C6.1, C60.1, C61.1, C62.1, C63.1, C64.1, C65.1, C7.1, C77.1, C78.1, C79.1, C8.1, C80.1, C9.1, D33.1 (VDD), D34.1 (VDD), D35.1 (VDD), D36.1 (VDD), D37.1 (VDD), D38.1 (VDD)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
- new net diag-m1: R77.1
- new net diag-m2: R89.1
- new net diag-m3: R112.1
- new net diag-m4: R121.1
- new net esp-rx: U11.J3_6 (U0TXD), teensy1.17 (25_A11_RX6_SDA2)
- new net esp-tx: U11.J3_5 (U0RXD), teensy1.16 (24_A10_TX6_SCL2)
- new net occ-m1: R78.1
- new net occ-m2: R85.1
- new net occ-m3: R108.1
- new net occ-m4: R117.1
- new net ocm-m1: C66.2, R74.1
- new net ocm-m2: C75.2, R82.1
- new net ocm-m3: C97.2, R105.1
- new net ocm-m4: C104.2, R114.1
- new net rx-cam: U1.5 (P4), teensy1.38 (16_A2_RX4_SCL1)
- new net rx-m1: U3.1 (~{RESET}/PB5), teensy1.2 (0_RX1_CRX2_CS1)
- new net rx-m2: U7.1 (~{RESET}/PB5), teensy1.9 (7_RX2_OUT1A)
- new net rx-m3: U8.1 (~{RESET}/PB5), teensy1.20 (28_RX7)
- new net rx-m4: U9.1 (~{RESET}/PB5), teensy1.26 (34_RX8)
- new net rx-proto: U2.4 (RX), teensy1.37 (15_A1_RX3_SPDIF_IN)
- new net tx-cam: U1.6 (P5), teensy1.39 (17_A3_TX4_SDA1)
- new net tx-m1: U3.3 (XTAL2/PB4), teensy1.3 (1_TX1_CTX2_MISO1)
- new net tx-m2: U7.3 (XTAL2/PB4), teensy1.10 (8_TX2_IN1)
- new net tx-m3: U8.3 (XTAL2/PB4), teensy1.21 (29_TX7)
- new net tx-m4: U9.3 (XTAL2/PB4), teensy1.27 (35_TX8)
- new net tx-proto: U2.3 (TX), teensy1.36 (14_A0_TX3_SPDIF_OUT)
- new net vout-m1: C67.1, C68.1, C69.1, C70.1, D1.1 (K), IC1.11 (VBAT_1), IC1.12 (VBAT_2), IC1.24 (VBAT_3), IC1.25 (VBAT_4), Q1.3 (S)
- new net vout-m2: C76.1, C92.1, C93.1, C94.1, D2.1 (K), IC2.11 (VBAT_1), IC2.12 (VBAT_2), IC2.24 (VBAT_3), IC2.25 (VBAT_4), Q2.3 (S)
- new net vout-m3: C100.1, C101.1, C98.1, C99.1, D3.1 (K), IC3.11 (VBAT_1), IC3.12 (VBAT_2), IC3.24 (VBAT_3), IC3.25 (VBAT_4), Q3.3 (S)
- new net vout-m4: C105.1, C106.1, C107.1, C108.1, D4.1 (K), IC4.11 (VBAT_1), IC4.12 (VBAT_2), IC4.24 (VBAT_3), IC4.25 (VBAT_4), Q4.3 (S)
- no-connect marks 1 -> 29
Other:
- note removed: "https://www.renesas.com/en/document/dst/isl29125-datasheet"
- moved on the sheet: C18, C19, C20, C21, C22, C48, C49, C50, C51, C52, C53, C54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

Commit message: Update Electronics.kicad_sch
Parts:
- added U13: ESP32-S3-DEVKITM-1-N8, ESP32-S3-DEVKITM-1-N8:MODULE_ESP32-S3-DEVKITM-1-N8, symbol ESP32-S3-DEVKITM-1-N8:ESP32-S3-DEVKITM-1-N8
Other:
- moved on the sheet: 3V3, 3V3_conv1, 5V1, 5V_conv1, BT1, BT2

Commit message: v1
Parts:
- added SW5: tacticle push button, 1825910-6:SW_1825910-6-4, symbol button:1825910-6
- added SW6: SW_DPST_x2, symbol Switch:SW_DPST_x2
Connections:
- net +3V3: no longer R10.2, R11.2, R12.2, R13.2, R14.2, R15.2, R16.2, R17.2, R2.2, R3.2, R4.2, R5.2, R6.2, R7.2, R8.2, R9.2
- net 12V: now also 3V3_conv1.2 (EN), 5V_conv1.2 (EN), SW6.2 (B); no longer BT1.1 (+), BT2.1 (+)
- net 3V3: now also R10.2, R11.2, R12.2, R13.2, R14.2, R15.2, R16.2, R17.2, R2.2, R3.2, R4.2, R5.2, R6.2, R7.2, R8.2, R9.2
- new net: BT1.1 (+), BT2.1 (+), SW6.1 (A)
- no-connect marks 29 -> 31
Other:
- moved on the sheet: BT1, BT2

Commit message: -motor driver -imu !!!need to check logic level converters!!!
Parts:
- removed C103, C74: 4.7uF, symbol Device:C
- removed D3, D4: 16.2v, symbol Device:D_Zener
- removed U3, U7, U8, U9: ATtiny85V-10P, Package_DIP:DIP-8_W7.62mm, symbol MCU_Microchip_ATtiny:ATtiny85V-10P
- removed U5: ~, Library:miniIMU, symbol TSSP4038:miniIMU
- added BZ1, BZ2: Buzzer, symbol Device:Buzzer
- added C103, C117, C124, C74: 4.7uF, symbol Device:C_Polarized
- added C109, C110, C120, C121, C130, C131: 20pF???, symbol Device:C
- added C111, C132: NP, symbol Device:C
- added C112, C133: 47uF, symbol Device:C
- added C113, C115, C127, C134, C136, C139, C140, C141: 0.1uF, symbol Device:C
- added C114, C116, C122, C123, C135, C142, C143: 100nF, symbol Device:C
- added C118, C119, C125, C126: 1uF, symbol Device:C
- added C128: 4.7uF, symbol Device:C
- added C129: 0.47uF, symbol Device:C
- added C137, C138: 22pF, symbol Device:C_Polarized
- added D10, D12, D16, D5: TX-LED, symbol Device:LED
- added D11, D15, D4, D9: RX-LED, symbol Device:LED
- added D13, D6: 16.2v, symbol Device:D_Zener
- added D14, D3, D7, D8: ????, symbol Device:LED
- added IC5: BNO086, BNO086, symbol SamacSys_Parts:BNO086
- added IR17, IR18: TSSP4038, OptoDevice:Vishay_MINICAST-3Pin, symbol Sensor_Proximity:TSSP58038
- added J1, J2, J3, J4, J6: shortable, symbol Connector:Conn_01x02_Socket
- added JP25: SolderJumper_3_Bridged12, symbol Jumper:SolderJumper_3_Bridged12
- added JP26, JP27: SolderJumper_2_Bridged, symbol Jumper:SolderJumper_2_Bridged
- added JP28: SolderJumper_3_Bridged12, Jumper:SolderJumper-3_P1.3mm_Open_RoundedPad1.0x1.5mm, symbol Jumper:SolderJumper_3_Bridged12
- added JP29: SolderJumper_2_Open, symbol Jumper:SolderJumper_2_Open
- added R129, R152, R165, R166: 10K, symbol Device:R_US
- added R130, R147, R153: 220, symbol Device:R_US
- added R131, R132, R133, R135, R136, R137, R138, R139, R140, R141, R142, R143, R144, R146, R148, R149, R150, R151, R154, R155, R156, R157, R158, R161, R162: 1K, symbol Device:R_US
- added R134: 1, symbol Device:R_US
- added R145: 100K, symbol Device:R_US
- added R159, R160: 2.2K, symbol Device:R_US
- added R163, R164: 4.7K, symbol Device:R_US
- added R167, R168: 100, symbol Device:R_US
- added U14, U16, U3, U8: ATmega328P-M, Package_DFN_QFN:QFN-32-1EP_5x5mm_P0.5mm_EP3.1x3.1mm, symbol MCU_Microchip_ATmega:ATmega328P-M
- added U15, U17, U7, U9: FT232RL, Package_SO:SSOP-28_5.3x10.2mm_P0.65mm, symbol Interface_USB:FT232RL
- added Y1, Y2, Y3, Y4: 16MHz, symbol Device:Crystal
- added Y5: 32.768, symbol Device:Crystal
- C100, C102, C73: value 0.1uF -> 100nF
- C104, C75: value 0.47uF -> 1uF
- C105, C76: value NP -> 1uF
- C106, C92, C99: value 47uF -> 0.1uF
- C107, C93: value 0.1uF -> 4.7uF
- C108, C94: value 0.1uF -> 0.47uF
- C95: value 0.1uF -> 20pF???
- C96: value 4.7uF -> 20pF???
- C97: value 0.47uF -> NP
- C98: value NP -> 47uF
- R104, R113: value 1 -> 1K
- R106: value 100K -> 10K
- R111: value 10K -> 1
- R112, R116, R121, R84, R89: value 220 -> 1K
- R117, R87: value 1K -> 220
- R120, R88: value 10K -> 1K
- R83: value 100K -> 1K
- R85: value 1K -> 100K
- U11: footprint ESP32-S3-DEVKITM-1-N8:MODULE_ESP32-S3-DEVKITM-1-N8 -> MODULE_ESP32-S3-DEVKITM-1-N8
- teensy1: footprint Library:Teensy41 -> teensy.pretty-master:Teensy41
Connections:
- net +3V3: now also C140.2, C141.2, IC5.28 (VDDIO), IC5.3 (VDD), R159.1, R160.1, R163.1, R164.1, R165.2, R166.1
- net +5V: now also C104.2, C105.2, C106.1, C75.2, C76.2, C92.1, R106.1, R111.2, R116.2, R86.2, C103.1, C117.1, C118.2, C119.2, C124.1, C125.2, C126.2, C127.1, C74.1, D10.2 (A), D11.2 (A), D12.2 (A), D15.2 (A), D16.2 (A), D4.2 (A), D5.2 (A), D9.2 (A), R129.1, R134.2, R139.2, R146.2, R152.1, R157.2, R161.2, U14.18 (AVCC), U14.4 (VCC), U14.6 (VCC), U15.20 (VCC), U15.4 (VCCIO), U16.18 (AVCC)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; no longer C102.1, C73.1, C95.1, R104.2, R111.1, R113.2, R120.1, R88.1
- net 3V3: now also R167.2, R168.2
- net GND: now also C102.1, C105.1, C108.1, C73.1, C76.1, C94.1, C97.2, R110.1, R110.2, R117.1, R85.1, R87.1, BZ1.2 (-), BZ2.2 (-), C103.2, C111.2, C112.2, C113.2, C115.2, C116.1, C117.2, C118.1, C119.1, C123.1, C124.2, C125.1, C126.1, C127.2, C128.2, C129.1, C132.2, C133.2, C134.2, C136.2, C137.2, C138.2, C139.1, C140.1, C141.1, C142.2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; no longer C100.2, C102.2, C105.2, C108.2, C73.2, C76.2, C94.2, C95.2, C96.2, C97.1, R106.1, R107.1, R116.1, R83.1, R84.1
- net SCL: now also IC5.19 (H_SCL/SCK/RX), JP27.2 (B)
- net SDA: now also IC5.20 (H_SDA/H_MISO/TX), JP26.2 (B)
- net diag-m2: now also R107.1; no longer R89.1
- net diag-m3: now also R130.1; no longer R112.1
- net diag-m4: now also R153.1; no longer R121.1
- net occ-m1: now also U8.12 (PB0)
- net occ-m2: now also R89.1, U3.12 (PB0); no longer R85.1
- net occ-m3: now also R119.1, U14.12 (PB0); no longer R108.1
- net occ-m4: now also R149.1, U16.12 (PB0); no longer R117.1
- net ocm-m1: now also U8.23 (PC0)
- net ocm-m2: now also C94.2, R84.1, U3.23 (PC0); no longer C75.2, R82.1
- net ocm-m3: now also C108.2, R114.1, U14.23 (PC0); no longer C97.2, R105.1
- net ocm-m4: now also C129.2, R144.1, U16.23 (PC0); no longer C104.2, R114.1
- net rx-m1: now also R137.2, U9.1 (TXD)
- net rx-m2: now also R82.2, U7.1 (TXD)
- net rx-m3: now also R112.2, U15.1 (TXD)
- net rx-m4: now also R135.2, U17.1 (TXD)
- net tx-m1: now also R138.2, U9.5 (RXD)
- net tx-m2: now also R83.2, U7.5 (RXD)
- net tx-m3: now also R113.2, U15.5 (RXD)
- net tx-m4: now also R143.2, U17.5 (RXD)
- net vout-m2: now also C101.1, C97.1, C98.1, C99.1; no longer C76.1, C92.1, C93.1, C94.1
- net vout-m3: now also C111.1, C112.1, C113.1, C115.1, D6.1 (K); no longer C100.1, C101.1, C98.1, C99.1
- net vout-m4: now also C132.1, C133.1, C134.1, C136.1, D13.1 (K); no longer C105.1, C106.1, C107.1, C108.1
- net at R81.1: now also C93.1
- net at Q4.2 (G): now also D13.2 (A), R145.2; no longer R115.2
- net at IC2.7 (OCM), R84.2: now also R87.2; no longer R82.2
- net at Q3.2 (G): now also R115.2, D6.2 (A); no longer R106.2
- net int-imu: now reaches teensy1.31 (39_MISO1_OUT1A)
- net int-imu: now also IC5.14 (H_INTN)
- net csn-imu: now reaches teensy1.32 (40_A16)
- net csn-imu: now also IC5.18 (H_CSN)
- net rst-imu: now reaches teensy1.33 (41_A17)
- net rst-imu: now also IC5.11 (NRST), J6.1 (Pin_1), R166.2
- net at teensy1.35 (13_SCK_LED): now also BZ1.1 (+)
- net at IC3.1 (OCC): now also R119.2; no longer R108.2
- net at R85.2: now also D2.2 (A), Q2.2 (G); no longer IC2.1 (OCC)
- net enAM1: now reaches R73.1
- net enAM1: now also U8.13 (PB1)
- net pwm1-m1: now reaches IC1.8 (PWM1)
- net pwm1-m1: now also U8.9 (PD5)
- net pwm2-m1: now reaches IC1.9 (PWM2)
- net pwm2-m1: now also U8.10 (PD6)
- net enBM1: now reaches R51.1
- net enBM1: now also U8.14 (PB2)
- net at R118.1: now also U14.17 (PB5)
- net at R118.2: now also D7.2 (A); no longer IC4.3 (ENB)
- net encA-m4: now reaches M3.5 (encA)
- net encA-m4: now also U16.24 (PC1)
- net encB-m4: now reaches M3.6 (encB)
- net encB-m4: now also U16.25 (PC2)
- net encA-m3: now reaches M2.5 (encA)
- net encA-m3: now also U14.24 (PC1)
- net encB-m3: now reaches M2.6 (encB)
- net encB-m3: now also U14.25 (PC2)
- net at R109.1: now also U7.22 (CBUS1)
- net at IC3.3 (ENB): now also R120.2; no longer R109.2
- net at R117.2: now also IC3.7 (OCM), R114.2; no longer IC4.1 (OCC)
- net at IC4.5 (EN): now also R151.2; no longer R119.2
- net pwm1-m4: now reaches IC4.8 (PWM1)
- net pwm1-m4: now also U16.9 (PD5)
- net pwm2-m4: now reaches IC4.9 (PWM2)
- net pwm2-m4: now also U16.10 (PD6)
- net at IC3.5 (EN): now also R121.2; no longer R110.2
- net pwm1-m3: now reaches IC3.8 (PWM1)
- net pwm1-m3: now also U14.9 (PD5)
- net pwm2-m3: now reaches IC3.9 (PWM2)
- net pwm2-m3: now also U14.10 (PD6)
- net pwm1-m2: now reaches IC2.8 (PWM1)
- net pwm1-m2: now also U3.9 (PD5)
- net pwm2-m2: now reaches IC2.9 (PWM2)
- net pwm2-m2: now also U3.10 (PD6)
- net at R86.1: now also J1.1 (Pin_1), U3.29 (~{RESET}/PC6)
- net at U11.J1_18 (GPIO16): now also IR17.1 (OUT)
- net at U11.J1_19 (GPIO17): now also IR18.1 (OUT)
- net at U11.J3_19 (GPIO20): now also BZ2.1 (+)
- net encA-m1: now reaches M4.5 (encA)
- net encA-m1: now also U8.24 (PC1)
- net encB-m1: now reaches M4.6 (encB)
- net encB-m1: now also U8.25 (PC2)
- net at C96.1: now also U3.8 (XTAL2/PB7); no longer R104.1
- net encA-m2: now reaches M1.5 (encA)
- net encA-m2: now also U3.24 (PC1)
- net encB-m2: now reaches M1.6 (encB)
- net encB-m2: now also U3.25 (PC2)
- net at R113.1: now also U14.31 (PD1)
- net at IC2.5 (EN): now also R105.2; no longer R87.2
- net at IC2.3 (ENB): now also R104.2; no longer R86.2
- new net: D15.1 (K), R154.2
- new net: J2.1 (Pin_1), R139.1, U8.29 (~{RESET}/PC6)
- new net: C114.1, U15.19 (~{RESET})
- new net: R132.1, U15.22 (CBUS1)
- new net: R131.1, U15.23 (CBUS0)
- new net: C107.1, R111.1
- new net: JP26.1 (A), R159.2
- new net: JP25.3 (B), R157.1
- new net: C128.1, R134.1
- new net: R143.1, U16.31 (PD1)
- new net: C110.1, U14.8 (XTAL2/PB7)
- new net: C110.2, Y3.1
- new net: R148.1, U16.17 (PB5)
- new net: C123.2, U16.20 (AREF)
- new net: J4.1 (Pin_1), R146.1, U16.29 (~{RESET}/PC6)
- new net: R135.1, U16.30 (PD0)
- new net: C130.1, U16.7 (XTAL1/PB6)
- new net: C131.1, U16.8 (XTAL2/PB7)
- new net: C102.2, U14.20 (AREF)
- new net: IC5.16 (ENV_SDA), R163.2
- new net: C142.1, IR17.3 (Vs), R167.1
- new net: J3.1 (Pin_1), R116.1, U14.29 (~{RESET}/PC6)
- new net: R112.1, U14.30 (PD0)
- new net: C109.1, U14.7 (XTAL1/PB6)
- new net: R137.1, U8.30 (PD0)
- new net: C100.1, U7.19 (~{RESET})
- new net: D14.2 (A), R148.2
- new net: C139.2, IC5.9 (CAP)
- new net: IC3.18 (DIAG), R129.2, R130.2
- new net: IC4.1 (OCC), R149.2
- new net: D5.1 (K), R109.2
- new net: R154.1, U17.23 (CBUS0)
- new net: C121.2, Y2.1
- new net: C120.2, Y2.2
- new net: IC4.7 (OCM), R144.2, R147.2
- new net: D10.1 (K), R141.2
- new net: C130.2, Y4.2
- new net: C135.1, U17.19 (~{RESET})
- new net: R155.1, U17.22 (CBUS1)
- new net: R136.1, U8.17 (PB5)
- new net: C116.2, U8.20 (AREF)
- new net: R138.1, U8.31 (PD1)
- new net: C120.1, U8.7 (XTAL1/PB6)
- new net: C121.1, U8.8 (XTAL2/PB7)
- new net: IC5.17 (SA0/H_MOSI), JP29.2 (B), R165.1
- new net: C131.2, Y4.1
- new net: JP28.1 (A), R162.2
- new net: C73.2, U3.20 (AREF)
- new net: D11.1 (K), R131.2
- new net: IC4.18 (DIAG), R152.2, R153.2
- new net: C137.1, IC5.27 (XIN32), Y5.1
- new net: IC2.18 (DIAG), R106.2, R107.2
- new net: R88.1, U3.17 (PB5)
- new net: R82.1, U3.30 (PD0)
- new net: R83.1, U3.31 (PD1)
- new net: C95.1, U3.7 (XTAL1/PB6)
- new net: D12.1 (K), R132.2
- new net: IC5.5 (PS1), JP28.2 (C)
- new net: JP28.3 (B), R161.1
- new net: D3.2 (A), R88.2
- new net: D9.1 (K), R140.2
- new net: C122.1, U9.19 (~{RESET})
- new net: R141.1, U9.22 (CBUS1)
- new net: R140.1, U9.23 (CBUS0)
- new net: D8.2 (A), R136.2
- new net: JP27.1 (A), R160.2
- new net: C95.2, Y1.2
- new net: JP25.1 (A), R158.2
- new net: IC5.6 (PS0/WAKE), JP25.2 (C)
- new net: C109.2, Y3.2
- new net: C96.2, Y1.1
- new net: C143.1, IR18.3 (Vs), R168.1
- new net: R108.1, U7.23 (CBUS0)
- new net: D4.1 (K), R108.2
- new net: IC4.3 (ENB), R150.2
- new net: IC2.1 (OCC), R89.2
- new net: D16.1 (K), R155.2
- new net: C138.1, IC5.26 (XOUT32/CLKSEL1), Y5.2
- new net: IC5.15 (ENV_SCL), R164.2
- new net enAM2: R105.1, U3.13 (PB1)
- new net enAM3: R121.1, U14.13 (PB1)
- new net enAM4: R151.1, U16.13 (PB1)
- new net enBM2: R104.1, U3.14 (PB2)
- new net enBM3: R120.1, U14.14 (PB2)
- new net enBM4: R150.1, U16.14 (PB2)
- new net reset-m1: C100.2, C122.2
- new net reset-m3: C114.2
- new net reset-m4: C135.2
- new net usb+m1: U9.15 (USBD+)
- new net usb+m2: U7.15 (USBD+)
- new net usb+m3: U15.15 (USBD+)
- new net usb+m4: U17.15 (USBD+)
- new net usb-m1: U9.16 (USBD-)
- new net usb-m2: U7.16 (USBD-)
- new net usb-m3: U15.16 (USBD-)
- new net usb-m4: U17.16 (USBD-)
- no-connect marks 31 -> 44
Other:
- moved on the sheet: 3V3, 3V3_conv1, 5V1, 5V_conv1, BT1, BT2, JP23, JP24, R127, R128, SW3, SW6A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

Commit message: Update Electronics.kicad_sch
Parts:
- removed U11: ESP32-S3-DEVKITM-1-N8, MODULE_ESP32-S3-DEVKITM-1-N8, symbol ESP32-S3-DEVKITM-1-N8:ESP32-S3-DEVKITM-1-N8
- removed U13: ESP32-S3-DEVKITM-1-N8, ESP32-S3-DEVKITM-1-N8:MODULE_ESP32-S3-DEVKITM-1-N8, symbol ESP32-S3-DEVKITM-1-N8:ESP32-S3-DEVKITM-1-N8
- added U5: ESP32-S3-DevKitC, PCM_Espressif:ESP32-S3-DevKitC, symbol Espressif:ESP32-S3-DevKitC
Connections:
- net +3V3: now also U5.1 (3V3), U5.2 (3V3)
- net GND: now also SW5.3, SW5.4, U5.22 (GND), U5.23 (GND), U5.24 (GND), U5.44 (GND)
- net esp-rx: now also U5.42 (GPIO44/U0RXD)
- net esp-tx: now also U5.43 (GPIO43/U0TXD)
- net at IR17.1 (OUT): now also U5.9 (GPIO16/ADC2_CH5/32K_N)
- net at SW5.1: now also U5.27 (GPIO21)
- net at IR14.1 (OUT): now also U5.20 (GPIO14/ADC2_CH3)
- net at SW2.1: now also U5.33 (GPIO36)
- net at SW4.1: now also U5.32 (GPIO35)
- net at IR12.1 (OUT): now also U5.18 (GPIO12/ADC2_CH1)
- net at IR7.1 (OUT): now also U5.7 (GPIO7/ADC1_CH6)
- net at IR4.1 (OUT): now also U5.4 (GPIO4/ADC1_CH3)
- net at IR15.1 (OUT): now also U5.10 (GPIO17/ADC2_CH6)
- net at SW1.1: now also U5.34 (GPIO37)
- net at IR3.1 (OUT): now also U5.13 (GPIO3/ADC1_CH2)
- net at IR9.1 (OUT): now also U5.15 (GPIO9/ADC1_CH8)
- net at IR10.1 (OUT): now also U5.16 (GPIO10/ADC1_CH9)
- net at IR11.1 (OUT): now also U5.17 (GPIO11/ADC2_CH0)
- net at IR13.1 (OUT): now also U5.19 (GPIO13/ADC2_CH2)
- net at IR16.1 (OUT): now also U5.11 (GPIO18/ADC2_CH7)
- net at IR18.1 (OUT): now also U5.8 (GPIO15/ADC2_CH4/32K_P)
- net at IR1.1 (OUT): now also U5.41 (GPIO1/ADC1_CH0)
- net at IR2.1 (OUT): now also U5.40 (GPIO2/ADC1_CH1)
- net at IR5.1 (OUT): now also U5.5 (GPIO5/ADC1_CH4)
- net at IR6.1 (OUT): now also U5.6 (GPIO6/ADC1_CH5)
- net at IR8.1 (OUT): now also U5.12 (GPIO8/ADC1_CH7)
- net at BZ2.1 (+): now also U5.35 (GPIO38)
- no-connect marks 44 -> 45
Other:
- moved on the sheet: BZ2, SW1, SW2, SW4, SW5

Commit message: pinnen toegevoegd en goede eps32
Parts:
- added J1, J2, J7: Conn_01x08_Pin, symbol Connector:Conn_01x08_Pin
- added J3, J4, J6: Conn_01x08_Socket, symbol Connector:Conn_01x08_Socket
- added J5: Conn_01x03_Socket, symbol Connector:Conn_01x03_Socket
- added J8: Conn_01x03_Pin, symbol Connector:Conn_01x03_Pin
- renumbered 3V3 to 3V1, BZ2 to BZ1, BZ1 to BZ2, C46 to C1, C45 to C10, C109 to C100, C110 to C101, C111 to C102, C68 to C103, C112 to C104, C69 to C105, C122 to C106, C113 to C107, C70 to C108, C114 to C109, C43 to C11, C115 to C110, C73 to C111, C74 to C112, C75 to C113, C76 to C114, C123 to C115, C92 to C116, C93 to C117, C124 to C118, C125 to C119, C41 to C12, C126 to C120, C94 to C121, C127 to C122, C95 to C123, C96 to C124, C128 to C125, C97 to C126, C129 to C127, C98 to C128, C99 to C129, C40 to C13, C100 to C133, C101 to C134, C139 to C135, C133 to C136, C141 to C137, C140 to C138, C134 to C139, C39 to C14, C135 to C140, C136 to C141, C137 to C142, C138 to C143, C38 to C15, C37 to C16, C81 to C17, C1 to C18, C2 to C19, C44 to C2, C3 to C20, C4 to C21, C5 to C22, C82 to C23, C83 to C24, C84 to C25, C85 to C26, C86 to C27, C87 to C28, C88 to C29, C42 to C3, C89 to C30, C90 to C31, C91 to C32, C142 to C33, C143 to C34, C48 to C35, C49 to C36, C50 to C37, C18 to C38, C19 to C39, C16 to C4, C20 to C40, C21 to C41, C22 to C42, C51 to C43, C52 to C44, C53 to C45, C54 to C46, C55 to C47, C56 to C48, C57 to C49, C15 to C5, C58 to C50, C17 to C51, C6 to C52, C7 to C53, C8 to C54, C9 to C55, C10 to C56, C11 to C57, C65 to C58, C23 to C59, C14 to C6, C24 to C60, C25 to C61, C26 to C62, C27 to C63, C28 to C64, C29 to C65, C30 to C66, C31 to C67, C32 to C68, C33 to C69, C13 to C7, C77 to C70, C34 to C71, C35 to C72, C36 to C73, C78 to C74, C59 to C75, C60 to C76, C61 to C77, C79 to C78, C62 to C79, C12 to C8, C63 to C80, C64 to C81, C80 to C82, C116 to C83, C102 to C84, C117 to C85, C118 to C86, C119 to C87, C103 to C88, C104 to C89, C47 to C9, C105 to C90, C71 to C91, C106 to C92, C72 to C93, C66 to C94, C107 to C95, C108 to C96, C120 to C97, C121 to C98, C67 to C99, D33 to D1, D42 to D10, D43 to D11, D44 to D12, D45 to D13, D46 to D14, D47 to D15, D48 to D16, D49 to D17, D50 to D18, D51 to D19, D34 to D2, D52 to D20, D53 to D21, D54 to D22, D55 to D23, D56 to D24, D57 to D25, D58 to D26, D59 to D27, D60 to D28, D61 to D29, D35 to D3, D62 to D30, D63 to D31, D64 to D32, D1 to D33, D8 to D34, D6 to D35, D7 to D36, D9 to D37, D10 to D38, D11 to D39, D36 to D4, D12 to D40, D2 to D41, D3 to D42, D13 to D43, D14 to D44, D4 to D45, D5 to D46, D15 to D47, D16 to D48, D37 to D5, D38 to D6, D39 to D7, D40 to D8, D41 to D9, IC3 to IC2, IC2 to IC3, J3 to J10, J1 to J11, J6 to J12, J4 to J13, J2 to J9, JP8 to JP1, JP21 to JP10, JP22 to JP11, JP9 to JP12, JP10 to JP13, JP11 to JP14, JP12 to JP15, JP13 to JP16, JP14 to JP17, JP15 to JP18, JP16 to JP19, JP7 to JP2, JP19 to JP20, JP18 to JP21, JP17 to JP22, JP24 to JP23, JP23 to JP24, JP28 to JP26, JP29 to JP27, JP27 to JP28, JP26 to JP29, JP6 to JP3, JP5 to JP4, JP4 to JP5, JP3 to JP6, JP2 to JP7, JP1 to JP8, JP20 to JP9, M4 to M1, M1 to M3, M3 to M4, Q3 to Q2, Q2 to Q3, R18 to R1, R3 to R10, R79 to R100, R139 to R101, R75 to R102, R114 to R103, R136 to R104, R115 to R105, R116 to R106, R117 to R107, R118 to R108, R78 to R109, R4 to R11, R51 to R110, R73 to R111, R119 to R112, R120 to R113, R121 to R114, R76 to R115, R77 to R116, R129 to R117, R130 to R118, R140 to R119, R5 to R12, R141 to R120, R131 to R121, R132 to R122, R142 to R123, R133 to R124, R127 to R125, R128 to R126, R81 to R127, R82 to R128, R83 to R129, R6 to R13, R84 to R130, R85 to R131, R86 to R132, R87 to R133, R88 to R134, R134 to R135, R135 to R136, R143 to R137, R89 to R138, R104 to R139, R7 to R14, R105 to R140, R144 to R141, R145 to R142, R146 to R143, R147 to R144, R148 to R145, R166 to R146, R157 to R147, R158 to R148, R8 to R15, R164 to R152, R162 to R153, R165 to R154, R106 to R155, R163 to R156, R107 to R157, R161 to R158, R108 to R159, R9 to R16, R109 to R160, R160 to R161, R152 to R162, R153 to R163, R110 to R164, R159 to R165, R154 to R166, R155 to R167, R156 to R168, R10 to R17, R11 to R18, R12 to R19, R22 to R2, R13 to R20, R14 to R21, R15 to R22, R16 to R23, R17 to R24, R167 to R25, R168 to R26, R96 to R27, R19 to R28, R95 to R29, R26 to R3, R94 to R30, R93 to R31, R92 to R32, R91 to R33, R90 to R34, R41 to R35, R20 to R36, R24 to R37, R30 to R38, R31 to R39, R27 to R4, R42 to R40, R43 to R41, R44 to R42, R45 to R43, R21 to R44, R25 to R45, R32 to R46, R33 to R47, R46 to R48, R47 to R49, R34 to R5, R48 to R50, R49 to R51, R50 to R52, R124 to R53, R125 to R54, R126 to R55, R23 to R56, R28 to R57, R29 to R58, R38 to R59, R35 to R6, R39 to R60, R40 to R61, R52 to R62, R53 to R63, R97 to R64, R54 to R65, R98 to R66, R99 to R67, R100 to R68, R101 to R69, R36 to R7, R102 to R70, R103 to R71, R55 to R72, R56 to R73, R57 to R74, R58 to R75, R59 to R76, R60 to R77, R61 to R78, R62 to R79, R37 to R8, R63 to R80, R64 to R81, R65 to R82, R66 to R83, R67 to R84, R68 to R85, R69 to R86, R70 to R87, R71 to R88, R72 to R89, R2 to R9, R123 to R90, R1 to R91, R122 to R92, R80 to R93, R137 to R94, R138 to R95, R74 to R96, R111 to R97, R112 to R98, R113 to R99, SW4 to SW3, SW5 to SW4, SW3 to SW5, U5 to U1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
Connections:
- net 3V3: now also J1.1 (Pin_1), J2.1 (Pin_1), J3.1 (Pin_1), J5.1 (Pin_1), J6.1 (Pin_1), J8.3 (Pin_3)
- net 5V: now also J1.3 (Pin_3), J2.3 (Pin_3), J3.3 (Pin_3), J5.3 (Pin_3), J6.3 (Pin_3), J8.1 (Pin_1)
- net GND: now also J1.2 (Pin_2), J2.2 (Pin_2), J3.2 (Pin_2), J5.2 (Pin_2), J6.2 (Pin_2), J8.2 (Pin_2)
- net LED: now also J1.4 (Pin_4), J2.4 (Pin_4), J3.4 (Pin_4), J6.4 (Pin_4)
- net SCL: now also J2.6 (Pin_6), J6.6 (Pin_6)
- net SDA: now also J2.5 (Pin_5), J6.5 (Pin_5)
- net esp-rx: now also J1.6 (Pin_6), J3.6 (Pin_6)
- net esp-tx: now also J1.5 (Pin_5), J3.5 (Pin_5)
- net rx-cam: now also J1.7 (Pin_7), J3.7 (Pin_7)
- net rx-m1: now also J4.2 (Pin_2), J7.2 (Pin_2)
- net rx-m2: now also J4.4 (Pin_4), J7.4 (Pin_4)
- net rx-m3: now also J4.6 (Pin_6), J7.6 (Pin_6)
- net rx-m4: now also J4.8 (Pin_8), J7.8 (Pin_8)
- net tx-cam: now also J1.8 (Pin_8), J3.8 (Pin_8)
- net tx-m1: now also J4.1 (Pin_1), J7.1 (Pin_1)
- net tx-m2: now also J4.3 (Pin_3), J7.3 (Pin_3)
- net tx-m3: now also J4.5 (Pin_5), J7.5 (Pin_5)
- net tx-m4: now also J4.7 (Pin_7), J7.7 (Pin_7)
Other:
- moved on the sheet: U5

Commit message: boven pcb best ver af
Other:
- moved on the sheet: J1
Changed lines of the file:
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@@
 	(wire
 		(pts
-			(xy 240.03 153.67) (xy 243.84 153.67)
+			(xy 491.49 295.91) (xy 495.3 295.91)
 		)
 		(stroke
@@
 	(wire
 		(pts
-			(xy 240.03 140.97) (xy 243.84 140.97)
+			(xy 491.49 283.21) (xy 495.3 283.21)
 		)
 		(stroke
@@
 	(wire
 		(pts
-			(xy 240.03 146.05) (xy 243.84 146.05)
+			(xy 491.49 288.29) (xy 495.3 288.29)
 		)
 		(stroke
@@
 	(wire
 		(pts
-			(xy 240.03 135.89) (xy 243.84 135.89)
+			(xy 491.49 278.13) (xy 495.3 278.13)
 		)
 		(stroke
@@
 	(wire
 		(pts
-			(xy 240.03 148.59) (xy 243.84 148.59)
+			(xy 491.49 290.83) (xy 495.3 290.83)
 		)
 		(stroke
@@
 	(wire
 		(pts
-			(xy 240.03 143.51) (xy 243.84 143.51)
+			(xy 491.49 285.75) (xy 495.3 285.75)
 		)
 		(stroke
@@
 	(wire
 		(pts
-			(xy 240.03 138.43) (xy 243.84 138.43)
+			(xy 491.49 280.67) (xy 495.3 280.67)
 		)
 		(stroke
@@
 	(wire
 		(pts
-			(xy 240.03 151.13) (xy 243.84 151.13)
+			(xy 491.49 293.37) (xy 495.3 293.37)
 		)
 		(stroke
@@
 	)
 	(label "esp-rx"
-		(at 240.03 148.59 180)
+		(at 491.49 290.83 180)
 		(effects
 			(font
@@
 	)
 	(label "3V3"
-		(at 240.03 135.89 180)
+		(at 491.49 278.13 180)
 		(effects
 			(font
@@
 	)
 	(label "GND"
-		(at 240.03 138.43 180)
+		(at 491.49 280.67 180)
 		(effects
 			(font
@@
 	)
 	(label "tx-cam"
-		(at 240.03 153.67 180)
+		(at 491.49 295.91 180)
 		(effects
 			(font
@@
 	)
 	(label "LED"
-		(at 240.03 143.51 180)
+		(at 491.49 285.75 180)
 		(effects
 			(font
@@
 	)
 	(label "rx-cam"
-		(at 240.03 151.13 180)
+		(at 491.49 293.37 180)
 		(effects
 			(font
@@
 	)
 	(label "5V"
-		(at 240.03 140.97 180)
+		(at 491.49 283.21 180)
 		(effects
 			(font
@@
 	)
 	(label "esp-tx"
-		(at 240.03 146.05 180)
+		(at 491.49 288.29 180)
 		(effects
 			(font
@@
 	(symbol
 		(lib_id "Connector:Conn_01x08_Pin")
-		(at 248.92 143.51 0)
+		(at 500.38 285.75 0)
 		(mirror y)
 		(unit 1)
@@
 		(dnp no)
 		(property "Reference" "J1"
-			(at 238.506 126.238 0)
+			(at 489.966 268.478 0)
 			(effects
 				(font
@@
 		)
 		(property "Value" "Conn_01x08_Pin"
-			(at 239.268 129.794 0)
+			(at 490.728 272.034 0)
 			(effects
 				(font
@@
 		)
 		(property "Footprint" ""
-			(at 248.92 143.51 0)
+			(at 500.38 285.75 0)
 			(effects
 				(font
@@
 		)
 		(property "Datasheet" "~"
-			(at 248.92 143.51 0)
+			(at 500.38 285.75 0)
 			(effects
 				(font
@@
 		)
 		(property "Description" "Generic connector, single row, 01x08, script generated"
-			(at 248.92 143.51 0)
+			(at 500.38 285.75 0)
 			(effects
 				(font

Commit message: some final adjustments.
Parts:
- added R169, R170, R171, R172, R173, R174, R175, R176, R177, R178, R179, R180, R181, R182, R183, R184, R185, R186, R187, R188, R189, R190, R191, R192, R193, R194, R195, R196, R197, R198, R199, R200, R201, R202, R203, R204, R205, R206, R207, R208, R209, R210, R211, R212, R213, R214, R215, R216, R217, R218, R219, R220, R221, R222, R223, R224: 10K, symbol Device:R_US
- added SW10, SW7, SW8, SW9: SW_DIP_x04, symbol Switch:SW_DIP_x04
Connections:
- net GND: now also R169.1, R170.1, R171.1, R172.1, R173.1, R174.1, R175.1, R176.1, R177.1, R178.1, R179.1, R181.1, R183.1, R184.1, R185.1, R186.1, R187.1, R188.1, R190.1, R192.1, R193.1, R194.1, R195.1, R196.1, R197.1, R199.1, R201.1, R202.1, R203.1, R204.1, R205.1, R206.1, R207.1, R208.1, R209.1, R210.1, R211.1, R212.1, R213.1, R214.1, R215.1, R216.1, R217.1, R218.1, R219.1, R220.1, R221.1, R222.1, R223.1, R224.1
- net rx-m1: now also SW7.8; no longer R94.2, U9.1 (TXD)
- net rx-m2: now also SW8.8; no longer R128.2, U13.1 (TXD)
- net rx-m3: now also SW9.8; no longer R98.2, U10.1 (TXD)
- net rx-m4: now also SW10.8; no longer R136.2, U14.1 (TXD)
- net tx-m1: now also SW7.7; no longer R95.2, U9.5 (RXD)
- net tx-m2: now also SW8.7; no longer R129.2, U13.5 (RXD)
- net tx-m3: now also SW9.7; no longer R99.2, U10.5 (RXD)
- net tx-m4: now also SW10.7; no longer R137.2, U14.5 (RXD)
- net at U12.1 (PD3): now also R202.2
- net at U12.11 (PD7): now also R204.2
- net at U12.15 (PB3): now also R196.2
- net at U12.16 (PB4): now also R197.2
- net at U12.19 (ADC6): now also R223.2
- net at U12.2 (PD4): now also R203.2
- net at U12.22 (ADC7): now also R224.2
- net at U12.26 (PC3): now also R198.2
- net at U12.27 (PC4): now also R199.2
- net at U12.28 (PC5): now also R200.2
- net at U12.32 (PD2): now also R201.2
- net at U7.1 (PD3): now also R193.2
- net at U7.11 (PD7): now also R195.2
- net at U7.15 (PB3): now also R187.2
- net at U7.16 (PB4): now also R188.2
- net at U7.19 (ADC6): now also R221.2
- net at U7.2 (PD4): now also R194.2
- net at U7.22 (ADC7): now also R222.2
- net at U7.26 (PC3): now also R189.2
- net at U7.27 (PC4): now also R190.2
- net at U7.28 (PC5): now also R191.2
- net at U7.32 (PD2): now also R192.2
- net at IC2.10 (NC_2): now also R212.2
- net at IC2.26 (NC_3): now also R211.2
- net at IC2.6 (NC_1): now also R213.2
- net at U6.1 (PD3): now also R175.2
- net at U6.11 (PD7): now also R177.2
- net at U6.15 (PB3): now also R169.2
- net at U6.16 (PB4): now also R170.2
- net at U6.19 (ADC6): now also R219.2
- net at U6.2 (PD4): now also R174.2
- net at U6.22 (ADC7): now also R220.2
- net at U6.26 (PC3): now also R171.2
- net at U6.27 (PC4): now also R172.2
- net at U6.28 (PC5): now also R173.2
- net at U6.32 (PD2): now also R176.2
- net at U11.1 (PD3): now also R184.2
- net at U11.11 (PD7): now also R186.2
- net at U11.15 (PB3): now also R178.2
- net at U11.16 (PB4): now also R179.2
- net at U11.19 (ADC6): now also R217.2
- net at U11.2 (PD4): now also R185.2
- net at U11.22 (ADC7): now also R218.2
- net at U11.26 (PC3): now also R180.2
- net at U11.27 (PC4): now also R181.2
- net at U11.28 (PC5): now also R182.2
- net at U11.32 (PD2): now also R183.2
- net at IC4.10 (NC_2): now also R215.2
- net at IC4.26 (NC_3): now also R214.2
- net at IC4.6 (NC_1): now also R216.2
- net at IC3.10 (NC_2): now also R209.2
- net at IC3.26 (NC_3): now also R210.2
- net at IC3.6 (NC_1): now also R208.2
- net at IC1.10 (NC_2): now also R206.2
- net at IC1.26 (NC_3): now also R207.2
- net at IC1.6 (NC_1): now also R205.2
- new net: R128.2, SW8.1, SW8.3
- new net: R129.2, SW8.2, SW8.4
- new net: R137.2, SW10.2, SW10.4
- new net: R94.2, SW7.1, SW7.3
- new net: R98.2, SW9.1, SW9.3
- new net: R136.2, SW10.1, SW10.3
- new net: R99.2, SW9.2, SW9.4
- new net: R95.2, SW7.2, SW7.4
- new net rx-m10: SW7.6, U9.1 (TXD)
- new net rx-m20: SW8.6, U13.1 (TXD)
- new net rx-m30: SW9.6, U10.1 (TXD)
- new net rx-m40: SW10.6, U14.1 (TXD)
- new net tx-m10: SW7.5, U9.5 (RXD)
- new net tx-m20: SW8.5, U13.5 (RXD)
- new net tx-m30: SW9.5, U10.5 (RXD)
- new net tx-m40: SW10.5, U14.5 (RXD)
- no-connect marks 45 -> 77
