File: PCB/Electronics/Electronics.kicad_sch (KiCad schematic)
At the start: 542 parts, among them IC1 TB9051FTG, IC2 TB9051FTG, IC3 TB9051FTG, IC4 TB9051FTG, IC5 BNO086, J1 Conn_01x08_Pin, J10 shortable, J11 shortable, J12 shortable, J13 shortable, J2 Conn_01x08_Pin, J3 Conn_01x08_Socket, J4 Conn_01x08_Socket, J5 Conn_01x03_Socket, J6 Conn_01x08_Socket, J7 Conn_01x08_Pin, J8 Conn_01x03_Pin, J9 shortable, Q1 Q_PMOS_DGS, Q2 Q_PMOS_DGS, Q3 Q_PMOS_DGS, Q4 Q_PMOS_DGS, SW1 tacticle push button, SW10 SW_DIP_x04, SW2 tacticle push button, SW3 tacticle push button, SW4 tacticle push button, SW5 SW_DIP_x03, SW6 SW_DPST_x2, SW7 SW_DIP_x04, SW8 SW_DIP_x04, SW9 SW_DIP_x04, U1 ESP32-S3-DevKitC, U10 FT232RL, U11 ATmega328P-M, U12 ATmega328P-M, U13 FT232RL, U14 FT232RL, U2 TCA9548APWR, U3 TCA9548APWR, U4 74AHCT125, U6 ATmega328P-M, U7 ATmega328P-M, U9 FT232RL, Y1 16MHz, Y2 16MHz, Y3 16MHz, Y4 16MHz, Y5 32.768

Commit message: fsdgal;nk
Parts:
- added J14: Conn_02x04_Row_Letter_Last, symbol Connector_Generic:Conn_02x04_Row_Letter_Last
Connections:
- net GND: now also R180.1, R182.1, R189.1, R191.1, R198.1, R200.1
- net usb+m1: now also J14.1a (Pin_1a)
- net usb+m2: now also J14.2a (Pin_2a)
- net usb+m3: now also J14.3a (Pin_3a)
- net usb+m4: now also J14.4a (Pin_4a)
- net usb-m1: now also J14.1b (Pin_1b)
- net usb-m2: now also J14.2b (Pin_2b)
- net usb-m3: now also J14.3b (Pin_3b)
- net usb-m4: now also J14.4b (Pin_4b)
