File: PCB/Electronics/Electronics.kicad_pcb (KiCad board)
At the start: 2 copper layers, 63 parts, among them IC1 TB9051FTG, IC2 TB9051FTG, IC3 TB9051FTG, IC4 TB9051FTG, U3 ATtiny85V-10P, U4 TCA9548APWR, U6 TCA9548APWR, U7 ATtiny85V-10P, U8 ATtiny85V-10P, U9 ATtiny85V-10P

Commit message: v2
Parts:
- moved IC1 0.51 mm to (204.6, 74.7)
- moved M1 0.25 mm to (170.5, 114.0)
Changed lines of the file:
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@@
 	(footprint "Connector_JST:JST_XH_B6B-XH-AM_1x06_P2.50mm_Vertical"
 		(layer "F.Cu")
-		(at 170.75 114.025)
+		(at 170.5 114)
 		(descr "JST XH series connector, B6B-XH-AM, with boss (http://www.jst-mfg.com/product/pdf/eng/eXH.pdf), generated with kicad-footprint-generator")
 		(tags "connector JST XH vertical boss")
@@
 	(footprint "SamacSys_Parts:TB9051FTG"
 		(layer "F.Cu")
-		(at 204.505 74.15)
+		(at 204.6 74.65)
 		(descr "TB9051FTG-6")
 		(tags "Integrated Circuit")

Commit message: -motor driver -imu !!!need to check logic level converters!!!
Parts:
- added IC5: BNO086, SamacSys_Parts:BNO086, F.Cu at (81.0, 101.7)
- added IR17: TSSP4038, OptoDevice:Vishay_MINICAST-3Pin, F.Cu at (113.0, 59.1)
- added IR18: TSSP4038, OptoDevice:Vishay_MINICAST-3Pin, F.Cu at (113.0, 65.5)
- added JP28: SolderJumper_3_Bridged12, Jumper:SolderJumper-3_P1.3mm_Open_RoundedPad1.0x1.5mm, F.Cu at (88.9, 108.0)
- added U11: ESP32-S3-DEVKITM-1-N8, esp32devk:MODULE_ESP32-S3-DEVKITM-1-N8, F.Cu at (31.6, 55.5)
- added U14: ATmega328P-M, Package_DFN_QFN:QFN-32-1EP_5x5mm_P0.5mm_EP3.1x3.1mm, F.Cu at (115.4, 37.0)
- added U15: FT232RL, Package_SO:SSOP-28_5.3x10.2mm_P0.65mm, F.Cu at (104.0, 82.1)
- added U16: ATmega328P-M, Package_DFN_QFN:QFN-32-1EP_5x5mm_P0.5mm_EP3.1x3.1mm, F.Cu at (115.4, 44.3)
- added U17: FT232RL, Package_SO:SSOP-28_5.3x10.2mm_P0.65mm, F.Cu at (114.5, 82.1)
- added teensy1: Teensy4.1, teensy.pretty-master:Teensy41, F.Cu at (156.8, 31.1)
- U3, U8: value ATtiny85V-10P -> ATmega328P-M; footprint Package_DIP:DIP-8_W7.62mm -> Package_DFN_QFN:QFN-32-1EP_5x5mm_P0.5mm_EP3.1x3.1mm
- U7, U9: value ATtiny85V-10P -> FT232RL; footprint Package_DIP:DIP-8_W7.62mm -> Package_SO:SSOP-28_5.3x10.2mm_P0.65mm
- moved U9 142.0 mm to (93.4, 82.1)
- moved IR1 141.1 mm to (79.3, 52.7)
- moved IR11 141.1 mm to (96.1, 65.5)
- moved IR12 141.1 mm to (96.1, 71.9)
- moved IR13 141.1 mm to (104.5, 52.7)
- moved IR14 141.1 mm to (104.5, 59.1)
- moved IR15 141.1 mm to (104.5, 65.5)
- moved IR16 141.1 mm to (104.5, 71.9)
- moved IR2 141.1 mm to (79.3, 59.1)
- moved IR3 141.1 mm to (79.3, 65.5)
- moved IR4 141.1 mm to (79.3, 71.9)
- moved IR5 141.1 mm to (87.7, 52.7)
- moved IR6 141.1 mm to (87.7, 59.1)
- moved IR7 141.1 mm to (87.7, 65.5)
- moved IR8 141.1 mm to (87.7, 71.9)
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Connections:
- IC1 pad 8: Net-(IC1-PWM1) -> /pwm1-m1
- IC1 pad 9: Net-(IC1-PWM2) -> /pwm2-m1
- IC2 pad 8: Net-(IC2-PWM1) -> /pwm1-m2
- IC2 pad 9: Net-(IC2-PWM2) -> /pwm2-m2
- IC3 pad 8: Net-(IC3-PWM1) -> /pwm1-m3
- IC3 pad 9: Net-(IC3-PWM2) -> /pwm2-m3
- IC4 pad 8: Net-(IC4-PWM1) -> /pwm1-m4
- IC4 pad 9: Net-(IC4-PWM2) -> /pwm2-m4
- M1 pad 5: unconnected-(M1-encA-Pad5) -> /encA-m2
- M1 pad 6: unconnected-(M1-encB-Pad6) -> /encB-m2
- M2 pad 5: unconnected-(M2-encA-Pad5) -> /encA-m3
- M2 pad 6: unconnected-(M2-encB-Pad6) -> /encB-m3
- M3 pad 5: unconnected-(M3-encA-Pad5) -> /encA-m4
- M3 pad 6: unconnected-(M3-encB-Pad6) -> /encB-m4
- M4 pad 5: unconnected-(M4-encA-Pad5) -> /encA-m1
- M4 pad 6: unconnected-(M4-encB-Pad6) -> /encB-m1
- U3 pad 1: /rx-m1 -> unconnected-(U3-PD3-Pad1)
- U3 pad 2: Net-(U3-XTAL1/PB3) -> unconnected-(U3-PD4-Pad2)
- U3 pad 3: /tx-m1 -> GND
- U3 pad 4: GND -> +5V
- U3 pad 5: Net-(IC1-PWM1) -> GND
- U3 pad 6: Net-(IC1-PWM2) -> +5V
- U3 pad 8: +5V -> Net-(U3-XTAL2/PB7)
- U7 pad 2: Net-(U7-XTAL1/PB3) -> unconnected-(U7-DTR-Pad2)
- U7 pad 3: /tx-m2 -> unconnected-(U7-RTS-Pad3)
- U7 pad 4: GND -> +5V
- U7 pad 5: Net-(IC2-PWM1) -> /tx-m2
- U7 pad 6: Net-(IC2-PWM2) -> unconnected-(U7-RI-Pad6)
- U7 pad 7: Net-(U7-PB2) -> GND
- U7 pad 8: +5V -> (no net)
- U8 pad 1: /rx-m3 -> unconnected-(U8-PD3-Pad1)
- U8 pad 2: Net-(U8-XTAL1/PB3) -> unconnected-(U8-PD4-Pad2)
- U8 pad 3: /tx-m3 -> GND
- U8 pad 4: GND -> +5V
- U8 pad 5: Net-(IC3-PWM1) -> GND
- U8 pad 6: Net-(IC3-PWM2) -> +5V
- U8 pad 8: +5V -> Net-(U8-XTAL2/PB7)
- U9 pad 1: /rx-m4 -> /rx-m1
- U9 pad 2: Net-(U9-XTAL1/PB3) -> unconnected-(U9-DTR-Pad2)
- U9 pad 3: /tx-m4 -> unconnected-(U9-RTS-Pad3)
- U9 pad 4: GND -> +5V
- U9 pad 5: Net-(IC4-PWM1) -> /tx-m1
- U9 pad 6: Net-(IC4-PWM2) -> unconnected-(U9-RI-Pad6)
- U9 pad 7: Net-(U9-PB2) -> GND
- U9 pad 8: +5V -> (no net)

Commit message: pinnen toegevoegd en goede eps32
Parts:
- moved U11 9.46 mm to (26.9, 63.7)
Changed lines of the file:
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@@
 	(footprint "esp32devk:MODULE_ESP32-S3-DEVKITM-1-N8"
 		(layer "F.Cu")
-		(at 31.635 55.508)
+		(at 26.93 63.71)
 		(property "Reference" "U11"
 			(at -9.575 -37.015 0)

Commit message: boven pcb af
Parts:
- moved U15 3.04 mm to (104.0, 85.2)
- moved M2 0.38 mm to (48.4, 83.2)
Changed lines of the file:
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@@
 	(footprint "Package_SO:SSOP-28_5.3x10.2mm_P0.65mm"
 		(layer "F.Cu")
-		(at 103.96 82.135)
+		(at 103.96 85.175)
 		(descr "28-Lead Plastic Shrink Small Outline (SS)-5.30 mm Body [SSOP] (see Microchip Packaging Specification 00000049BS.pdf)")
 		(tags "SSOP 0.65")
@@
 	(footprint "Connector_JST:JST_XH_B6B-XH-AM_1x06_P2.50mm_Vertical"
 		(layer "F.Cu")
-		(at 48.58 82.865)
+		(at 48.4 83.2)
 		(descr "JST XH series connector, B6B-XH-AM, with boss (http://www.jst-mfg.com/product/pdf/eng/eXH.pdf), generated with kicad-footprint-generator")
 		(tags "connector JST XH vertical boss")
