File: PCB/Boven PCB/Boven PCB.kicad_sch (KiCad schematic)
At the start: 55 parts, among them J2 Conn_01x08_Pin, SW1 tacticle push button, SW2 tacticle push button, SW4 tacticle push button, SW5 tacticle push button, U11 ESP32-S3-DEVKITM-1-N8

Commit message: v2
Parts:
- removed U11: ESP32-S3-DEVKITM-1-N8, button:test, symbol ESP32-S3-DEVKITM-1-N8:ESP32-S3-DEVKITM-1-N8
- added C6, C7: 100nF, Capacitor_SMD:C_0603_1608Metric_Pad1.08x0.95mm_HandSolder, symbol Device:C
- added IR17, IR18: TSSP4038, OptoDevice:Vishay_MINICAST-3Pin, symbol Sensor_Proximity:TSSP58038
- added R1, R18: 100, Resistor_SMD:R_0603_1608Metric_Pad0.98x0.95mm_HandSolder, symbol Device:R_US
- added U2: ESP32-S3-DevKitC, PCM_Espressif:ESP32-S3-DevKitC, symbol Espressif:ESP32-S3-DevKitC
- renumbered C84 to C10, C85 to C11, C86 to C12, C87 to C13, C88 to C14, C89 to C15, C90 to C16, C91 to C17, C81 to C18, C82 to C8, C83 to C9
Connections:
- net 3V3: now also R1.2, R18.2, U2.1 (3V3), U2.2 (3V3)
- net 5V: now also U2.21 (5V)
- net GND: now also SW5.3, SW5.4, C6.2, C7.2, IR17.2 (GND), IR18.2 (GND)
- net esp-rx: now also U2.43 (GPIO43/U0TXD)
- net esp-tx: now also U2.42 (GPIO44/U0RXD)
- net at SW5.1: now also U2.34 (GPIO37)
- net at IR14.1 (OUT): now also U2.20 (GPIO14/ADC2_CH3)
- net at SW2.1: now also U2.32 (GPIO35)
- net at SW4.1: now also U2.33 (GPIO36)
- net at IR12.1 (OUT): now also U2.18 (GPIO12/ADC2_CH1)
- net at IR7.1 (OUT): now also U2.7 (GPIO7/ADC1_CH6)
- net at IR4.1 (OUT): now also U2.4 (GPIO4/ADC1_CH3)
- net at IR15.1 (OUT): now also U2.10 (GPIO17/ADC2_CH6)
- net at SW1.1: now also U2.27 (GPIO21)
- net at IR3.1 (OUT): now also U2.13 (GPIO3/ADC1_CH2)
- net at IR9.1 (OUT): now also U2.15 (GPIO9/ADC1_CH8)
- net at IR10.1 (OUT): now also U2.16 (GPIO10/ADC1_CH9)
- net at IR11.1 (OUT): now also U2.17 (GPIO11/ADC2_CH0)
- net at IR13.1 (OUT): now also U2.19 (GPIO13/ADC2_CH2)
- net at IR16.1 (OUT): now also U2.11 (GPIO18/ADC2_CH7)
- net at IR1.1 (OUT): now also U2.41 (GPIO1/ADC1_CH0)
- net at IR2.1 (OUT): now also U2.40 (GPIO2/ADC1_CH1)
- net at IR5.1 (OUT): now also U2.5 (GPIO5/ADC1_CH4)
- net at IR6.1 (OUT): now also U2.6 (GPIO6/ADC1_CH5)
- net at IR8.1 (OUT): now also U2.12 (GPIO8/ADC1_CH7)
- new net: C7.1, IR18.3 (Vs), R18.1
- new net: C6.1, IR17.3 (Vs), R1.1
- new net: IR18.1 (OUT), U2.9 (GPIO16/ADC2_CH5/32K_N)
- new net: U2.22 (GND), U2.23 (GND), U2.24 (GND), U2.44 (GND)
- new net: IR17.1 (OUT), U2.8 (GPIO15/ADC2_CH4/32K_P)
Other:
- moved on the sheet: SW1, SW2, SW4, SW5, U1

Commit message: boven pcb best ver af
Parts:
- added H1, H2, H3: MountingHole, MountingHole:MountingHole_4mm, symbol Mechanical:MountingHole
Changed lines of the file:
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@@
 	)
 	(symbol
+		(lib_id "Mechanical:MountingHole")
+		(at 200.66 43.18 0)
+		(unit 1)
+		(exclude_from_sim no)
+		(in_bom no)
+		(on_board yes)
+		(dnp no)
+		(fields_autoplaced yes)
+		(property "Reference" "H3"
+			(at 203.2 41.9099 0)
+			(effects
+				(font
+					(size 1.27 1.27)
+				)
+				(justify left)
+			)
+		)
+		(property "Value" "MountingHole"
+			(at 203.2 44.4499 0)
+			(effects
+				(font
+					(size 1.27 1.27)
+				)
+				(justify left)
+			)
+		)
+		(property "Footprint" "MountingHole:MountingHole_4mm"
+			(at 200.66 43.18 0)
+			(effects
+				(font
+					(size 1.27 1.27)
+				)
+				(hide yes)
+			)
+		)
+		(property "Datasheet" "~"
+			(at 200.66 43.18 0)
+			(effects
+				(font
+					(size 1.27 1.27)
+				)
+				(hide yes)
+			)
+		)
+		(property "Description" "Mounting Hole without connection"
+			(at 200.66 43.18 0)
+			(effects
+				(font
+					(size 1.27 1.27)
+				)
+				(hide yes)
+			)
+		)
+		(instances
+			(project "Boven PCB"
+				(path "/0a17e4c7-bbfc-4caa-a863-5ceb97e156cc"
+					(reference "H3")
+					(unit 1)
+				)
+			)
+		)
+	)
+	(symbol
 		(lib_id "button:1825910-6")
 		(at 166.37 181.61 90)
@@
 	)
 	(symbol
+		(lib_id "Mechanical:MountingHole")
+		(at 200.66 38.1 0)
+		(unit 1)
+		(exclude_from_sim no)
+		(in_bom no)
+		(on_board yes)
+		(dnp no)
+		(fields_autoplaced yes)
+		(property "Reference" "H2"
+			(at 203.2 36.8299 0)
+			(effects
+				(font
+					(size 1.27 1.27)
+				)
+				(justify left)
+			)
+		)
+		(property "Value" "MountingHole"
+			(at 203.2 39.3699 0)
+			(effects
+				(font
+					(size 1.27 1.27)
+				)
+				(justify left)
+			)
+		)
+		(property "Footprint" "MountingHole:MountingHole_4mm"
+			(at 200.66 38.1 0)
+			(effects
+				(font
+					(size 1.27 1.27)
+				)
+				(hide yes)
+			)
+		)
+		(property "Datasheet" "~"
+			(at 200.66 38.1 0)
+			(effects
+				(font
+					(size 1.27 1.27)
+				)
+				(hide yes)
+			)
+		)
+		(property "Description" "Mounting Hole without connection"
+			(at 200.66 38.1 0)
+			(effects
+				(font
+					(size 1.27 1.27)
+				)
+				(hide yes)
+			)
+		)
+		(instances
+			(project "Boven PCB"
+				(path "/0a17e4c7-bbfc-4caa-a863-5ceb97e156cc"
+					(reference "H2")
+					(unit 1)
+				)
+			)
+		)
+	)
+	(symbol
 		(lib_id "power:GND")
 		(at 205.74 204.47 0)
@@
 					(unit 1)
 				)
+			)
+		)
+	)
+	(symbol
+		(lib_id "Mechanical:MountingHole")
+		(at 200.66 33.02 0)
+		(unit 1)
+		(exclude_from_sim no)
+		(in_bom no)
+		(on_board yes)
+		(dnp no)
+		(fields_autoplaced yes)
+		(property "Reference" "H1"
+			(at 203.2 31.7499 0)
+			(effects
+				(font
+					(size 1.27 1.27)
+				)
+				(justify left)
+			)
+		)
+		(property "Value" "MountingHole"
+			(at 203.2 34.2899 0)
+			(effects
+				(font
+					(size 1.27 1.27)
+				)
+				(justify left)
+			)
+		)
+		(property "Footprint" "MountingHole:MountingHole_4mm"
+			(at 200.66 33.02 0)
+			(effects
+				(font
+					(size 1.27 1.27)
+				)
+				(hide yes)
+			)
+		)
+		(property "Datasheet" "~"
+			(at 200.66 33.02 0)
+			(effects
+				(font
+					(size 1.27 1.27)
+				)
+				(hide yes)
+			)
+		)
+		(property "Description" "Mounting Hole without connection"
+			(at 200.66 33.02 0)
+			(effects
+				(font
+					(size 1.27 1.27)
+				)
+				(hide yes)
+			)
+		)
+		(instances
+			(project ""
+				(path "/0a17e4c7-bbfc-4caa-a863-5ceb97e156cc"
+					(reference "H1")
+					(unit 1)
+				)
