File: PCB/Boven PCB/Boven PCB.kicad_pcb (KiCad board)
At the start: 2 copper layers, 54 parts, among them J2 Conn_01x08_Pin, SW1 tacticle push button, SW2 tacticle push button, SW4 tacticle push button, SW5 tacticle push button, U11 ESP32-S3-DEVKITM-1-N8

Commit message: v2
Parts:
- added C6: 100nF, Capacitor_SMD:C_0603_1608Metric_Pad1.08x0.95mm_HandSolder, B.Cu at (71.6, 80.3)
- added C7: 100nF, Capacitor_SMD:C_0603_1608Metric_Pad1.08x0.95mm_HandSolder, B.Cu at (85.2, 71.3)
- added IR17: TSSP4038, OptoDevice:Vishay_MINICAST-3Pin, F.Cu at (73.3, 76.6)
- added IR18: TSSP4038, OptoDevice:Vishay_MINICAST-3Pin, F.Cu at (87.7, 68.2)
- added R1: 100, Resistor_SMD:R_0603_1608Metric_Pad0.98x0.95mm_HandSolder, B.Cu at (72.6, 82.8)
- added R18: 100, Resistor_SMD:R_0603_1608Metric_Pad0.98x0.95mm_HandSolder, B.Cu at (85.2, 73.9)
- C1, C2, C3, C4, C5, R10, R11, R12, R13, R14, R15, R16, R17, R2, R3, R4, R5, R6, R7, R8, R9: moved to B.Cu
- C10: renamed from C84; moved to B.Cu
- C11: renamed from C85; moved to B.Cu
- C12: renamed from C86; moved to B.Cu
- C13: renamed from C87; moved to B.Cu
- C14: renamed from C88; moved to B.Cu
- C15: renamed from C89; moved to B.Cu
- C16: renamed from C90; moved to B.Cu
- C17: renamed from C91; moved to B.Cu
- C18: renamed from C81; moved to B.Cu
- C8: renamed from C82; moved to B.Cu
- C9: renamed from C83; moved to B.Cu
- SW1, SW2, SW4, SW5: footprint Button_Switch_THT:KSA_Tactile_SPST -> Button_Switch_THT:SW_Push_2P1T_Toggle_CK_PVA1xxH4xxxxxxV2
- moved R2 132.3 mm to (99.3, 69.5), turned to -90 degrees
- moved R17 130.6 mm to (63.9, 95.5), turned to -30 degrees
- moved C17 130.6 mm to (62.1, 93.5), turned to 60 degrees
- moved R3 128.5 mm to (114.7, 70.4), turned to -110 degrees
- moved C18 127.9 mm to (100.2, 67.0)
- moved R16 122.6 mm to (60.2, 110.2), turned to -10 degrees
- moved C16 121.4 mm to (58.0, 108.8), turned to 80 degrees
- moved IR16 115.8 mm to (62.6, 89.3), turned to -120 degrees
- moved R15 111.9 mm to (61.9, 125.5), turned to 10 degrees
- moved C1 109.4 mm to (116.3, 68.5), turned to -20 degrees
- moved C15 109.3 mm to (59.4, 125.0), turned to 100 degrees
- moved IR15 106.9 mm to (56.9, 105.0), turned to -100 degrees
- moved C2 101.9 mm to (131.0, 75.4), turned to -40 degrees
- moved R4 100.6 mm to (128.8, 76.5), turned to -130 degrees
- moved R14 97.9 mm to (69.8, 139.0), turned to 30 degrees
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Connections:
- SW5 pad 1: unconnected-(SW5-Pad1) -> Net-(U2-GPIO37)
- SW5 pad 3: unconnected-(SW5-Pad3) -> GND
- SW5 pad 4: unconnected-(SW5-Pad4) -> GND
Routing:
- net /3V3: track 0.00 -> 342.8 mm
- net Net-(IR1-OUT): track 0.00 -> 111.1 mm
- net Net-(IR18-OUT): track 0.00 -> 107.1 mm, vias 0 -> 1
- net Net-(IR17-OUT): track 0.00 -> 90.5 mm, vias 0 -> 1
- net Net-(IR15-OUT): track 0.00 -> 88.3 mm
- net Net-(IR12-OUT): track 0.00 -> 87.4 mm, vias 0 -> 1
- net Net-(IR5-OUT): track 0.00 -> 84.5 mm, vias 0 -> 1
- net Net-(IR11-OUT): track 0.00 -> 74.3 mm, vias 0 -> 1
- net Net-(IR6-OUT): track 0.00 -> 71.4 mm, vias 0 -> 1
- net Net-(IR16-OUT): track 0.00 -> 71.0 mm, vias 0 -> 1
- net Net-(IR4-OUT): track 0.00 -> 70.7 mm, vias 0 -> 1
- net Net-(IR14-OUT): track 0.00 -> 70.1 mm
- net Net-(IR3-OUT): track 0.00 -> 64.2 mm
- net Net-(IR10-OUT): track 0.00 -> 63.9 mm, vias 0 -> 1
- net Net-(IR2-OUT): track 0.00 -> 60.2 mm
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- added copper zone on B.Cu, net GND
Other:
- board outline added: 100.5 x 100.5 mm

Commit message: boven pcb best ver af
Parts:
- added H1: MountingHole, MountingHole:MountingHole_4mm, F.Cu at (149.9, 113.0)
- added H2: MountingHole, MountingHole:MountingHole_4mm, F.Cu at (81.1, 152.8)
- added H3: MountingHole, MountingHole:MountingHole_4mm, F.Cu at (81.1, 73.3)
- moved SW4 61.9 mm to (72.3, 99.5)
- moved SW1 58.8 mm to (130.4, 98.9)
- moved SW2 9.58 mm to (72.3, 89.8)
- moved SW5 9.52 mm to (130.4, 89.1)
- moved C10 0.75 mm to (123.6, 154.8)
- moved R10 0.68 mm to (123.3, 152.3)
- moved IR12 0.56 mm to (73.7, 149.7)
- moved C13 0.56 mm to (77.9, 150.4)
- moved R13 0.56 mm to (80.1, 149.2)
- moved IR11 0.55 mm to (88.0, 157.9)
- moved C12 0.55 mm to (92.1, 157.8)
- moved R12 0.55 mm to (93.8, 155.9)
- moved C11 0.50 mm to (107.8, 159.3)
- moved IR10 0.50 mm to (104.1, 160.8)
- moved R11 0.50 mm to (108.8, 156.8)
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Connections:
- U11 pad 24: (no net) -> GND
- U11 pad J1_22: (no net) -> GND
- U11 pad J3_1: (no net) -> GND
- U11 pad J3_12: (no net) -> Net-(U2-GPIO37)
- U11 pad J3_13: (no net) -> Net-(U2-GPIO36)
- U11 pad J3_14: (no net) -> Net-(U2-GPIO35)
- U11 pad J3_18: (no net) -> Net-(U2-GPIO21)
- U11 pad J3_5: (no net) -> /esp-rx
- U11 pad J3_6: (no net) -> /esp-tx
Routing:
- net /esp-rx: track 0.00 -> 54.5 mm
- net /esp-tx: track 0.00 -> 53.4 mm
- net Net-(U2-GPIO35): track 0.00 -> 50.7 mm, vias 0 -> 1
- net Net-(U2-GPIO37): track 0.00 -> 45.4 mm
- net Net-(U2-GPIO36): track 0.00 -> 38.8 mm, vias 0 -> 1
- net Net-(U2-GPIO21): track 0.00 -> 18.5 mm
- net /3V3: track 342.8 -> 345.3 mm, vias 0 -> 19
- net GND: track 0.74 -> 2.53 mm

Commit message: alleen nog cxampera
Parts:
- moved R8 0.76 mm to (143.7, 130.4)
- moved C5 0.65 mm to (149.7, 117.5)
- moved C8 0.64 mm to (145.6, 132.4)
- moved C4 0.61 mm to (148.5, 101.4)
- moved R6 0.61 mm to (146.0, 100.9)
- moved R7 0.60 mm to (147.5, 116.0)
- moved C9 0.54 mm to (136.5, 145.9)
- moved IR5 0.49 mm to (150.9, 105.1)
- moved R9 0.42 mm to (135.7, 143.4)
- moved IR7 0.42 mm to (145.4, 137.1)
- moved IR6 0.35 mm to (151.1, 121.5)
- moved IR8 0.33 mm to (134.6, 149.6)
Routing:
- net GND: track 2.53 -> 19.3 mm
- net Net-(IR1-OUT): track 111.1 -> 125.8 mm, vias 0 -> 1
- net Net-(IR4-OUT): track 70.7 -> 75.7 mm
- net Net-(IR3-OUT): track 64.2 -> 69.1 mm
- net /3V3: track 345.3 -> 349.4 mm, vias 19 -> 21
- net Net-(IR12-OUT): track 87.4 -> 84.1 mm
- net Net-(IR13-OUT): track 58.0 -> 60.0 mm
- net Net-(IR5-OUT): track 84.5 -> 86.4 mm
- net Net-(IR6-OUT): track 71.4 -> 73.2 mm
- net Net-(IR7-Vs): track 3.80 -> 5.41 mm
- net Net-(IR11-OUT): track 74.3 -> 73.0 mm
- net Net-(IR10-OUT): track 63.7 -> 62.4 mm
- net Net-(IR8-OUT): track 55.9 -> 54.7 mm, vias 1 -> 2
- net Net-(IR17-OUT): track 90.5 -> 89.5 mm
- net Net-(IR16-OUT): track 71.0 -> 71.6 mm
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
Commit message: boven pcb af
Parts:
- added U1: ~, Lib:openMV_H7, F.Cu at (103.4, 93.2)
Routing:
- net /5V: track 0.00 -> 105.0 mm, vias 0 -> 1
- net /rx-cam: track 0.00 -> 59.3 mm, vias 0 -> 1
- net /tx-cam: track 0.00 -> 58.3 mm, vias 0 -> 1
- net /esp-rx: track 54.5 -> 46.1 mm
- net /esp-tx: track 53.4 -> 46.1 mm
- net Net-(U2-GPIO37): track 45.4 -> 39.9 mm, vias 0 -> 1
- net Net-(IR8-OUT): track 54.7 -> 56.5 mm
- net Net-(IR2-OUT): track 60.5 -> 60.0 mm
