File: PCB/Midden pcb Motoren+power/Midden pcb Motoren+power.kicad_sch (KiCad schematic)
At the start: 267 parts, among them IC1 TB9051FTG, IC2 TB9051FTG, IC3 TB9051FTG, IC4 TB9051FTG, IC5 BNO086, J10 shortable, J11 shortable, J12 shortable, J13 shortable, J4 Conn_01x08_Socket, J5 Conn_01x03_Socket, J6 Conn_01x08_Socket, J7 Conn_01x08_Pin, J8 Conn_01x03_Pin, J9 shortable, Q1 Q_PMOS_DGS, Q2 Q_PMOS_DGS, Q3 Q_PMOS_DGS, Q4 Q_PMOS_DGS, SW10 SW_DIP_x04, SW5 SW_DIP_x03, SW6 SW_DPST_x2, SW7 SW_DIP_x04, SW8 SW_DIP_x04, SW9 SW_DIP_x04, U10 FT232RL, U11 ATmega328P-M, U12 ATmega328P-M, U13 FT232RL, U14 FT232RL, U6 ATmega328P-M, U7 ATmega328P-M, U9 FT232RL, Y1 16MHz, Y2 16MHz, Y3 16MHz, Y4 16MHz, Y5 32.768

Commit message: M1 is af
Parts:
- removed J5: Conn_01x03_Socket, Connector_JST:JST_EH_S3B-EH_1x03_P2.50mm_Horizontal, symbol Connector:Conn_01x03_Socket
- removed J8: Conn_01x03_Pin, Connector_JST:JST_EH_S3B-EH_1x03_P2.50mm_Horizontal, symbol Connector:Conn_01x03_Pin
- added J1: Conn_01x04_Pin, symbol Connector:Conn_01x04_Pin
- added J2: Conn_01x04_Socket, symbol Connector:Conn_01x04_Socket
- added J3: Conn_01x08_Socket, Connector_JST:JST_EH_S8B-EH_1x08_P2.50mm_Horizontal, symbol Connector:Conn_01x08_Socket
Connections:
- net 12V is gone; now on net +12V: 3V1.3 (VCC), 3V3_conv1.2 (EN), 3V3_conv1.3 (VIN), 5V1.3 (VCC), 5V_conv1.2 (EN), 5V_conv1.3 (VIN), SW6.2 (B)
- net +12V: now also J1.1 (Pin_1), J2.1 (Pin_1)
- net GND: now also J1.3 (Pin_3), J2.3 (Pin_3), J3.2 (Pin_2); no longer 3V1.1 (VOUT), 3V3_conv1.6 (VOUT), 5V1.1 (VOUT), 5V_conv1.6 (VOUT), IC5.19 (H_SCL/SCK/RX), IC5.20 (H_SDA/H_MISO/TX), J6.1 (Pin_1), J6.2 (Pin_2), J6.3 (Pin_3), J6.4 (Pin_4), J6.5 (Pin_5), J6.6 (Pin_6), J6.8 (Pin_8), JP28.2 (B), JP29.2 (B), R125.2, R126.2, U8.1 (SCL), teensy1.4 (2_OUT2), teensy1.40 (18_A4_SDA), teensy1.41 (19_A5_SCL)
- net esp-rx: now also J3.6 (Pin_6)
- net esp-tx: now also J3.5 (Pin_5)
- net rx-cam: now also J3.7 (Pin_7)
- net tx-cam: now also J3.8 (Pin_8)
- new net 3V3: 3V1.1 (VOUT), 3V3_conv1.6 (VOUT), J1.4 (Pin_4), J2.4 (Pin_4), J3.1 (Pin_1), J6.8 (Pin_8)
- new net 5V: 5V1.1 (VOUT), 5V_conv1.6 (VOUT), J1.2 (Pin_2), J2.2 (Pin_2), J3.3 (Pin_3), J6.6 (Pin_6)
- new net LED: J3.4 (Pin_4), J6.5 (Pin_5), teensy1.4 (2_OUT2)
- new net SCL: IC5.19 (H_SCL/SCK/RX), J6.3 (Pin_3), JP28.2 (B), R126.2, U8.1 (SCL), teensy1.41 (19_A5_SCL)
- new net SDA: IC5.20 (H_SDA/H_MISO/TX), J6.4 (Pin_4), JP29.2 (B), R125.2, U8.1 (SCL), teensy1.40 (18_A4_SDA)
Other:
- moved on the sheet: J6

Commit message: m2
Changed lines of the file:
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@@
 	)
 	(label "pwm1-m3"
-		(at 447.04 199.39 0)
+		(at 447.04 199.39 180)
 		(effects
 			(font
 				(size 1.27 1.27)
 			)
-			(justify left bottom)
+			(justify right bottom)
 		)
 	)

Commit message: motor driver symbol changed
Parts:
- IC1, IC2, IC3, IC4: footprint Lib:TB9051FTG -> SamacSys_Parts:TB9051FTG
Changed lines of the file:
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@@
 			)
 		)
-		(property "Footprint" "Lib:TB9051FTG"
+		(property "Footprint" "SamacSys_Parts:TB9051FTG"
 			(at 514.35 171.12 0)
 			(effects
@@
 			)
 		)
-		(property "Footprint" "Lib:TB9051FTG"
+		(property "Footprint" "SamacSys_Parts:TB9051FTG"
 			(at 755.65 164.77 0)
 			(effects
@@
 			)
 		)
-		(property "Footprint" "Lib:TB9051FTG"
+		(property "Footprint" "SamacSys_Parts:TB9051FTG"
 			(at 289.56 525.45 0)
 			(effects
@@
 			)
 		)
-		(property "Footprint" "Lib:TB9051FTG"
+		(property "Footprint" "SamacSys_Parts:TB9051FTG"
 			(at 193.04 247.32 0)
 			(effects
